Commit message: Added Lirad Sensor
Closin #54

File: leobot_description/urdf/sensors/hokuyo.urdf.xacro (robot description, xacro)
@@ -1,5 +1,5 @@
 <?xml version="1.0"?>
 <robot xmlns:xacro="http://ros.org/wiki/xacro">
-     <xacro:property name="hokuyo_width" value="0.1"/>
+     <xacro:property name="hokuyo_width" value="0.001"/>
      <xacro:property name="hokuyo_height" value="0.05"/>
      <xacro:property name="hokuyo_depth" value="0.06"/>
@@ -12,5 +12,5 @@
       </visual>
       <xacro:box_collision width="${hokuyo_width}" height="${hokuyo_height}" depth="${hokuyo_depth}"/>
-      <xacro:box_inertia mass="0.01" width="${hokuyo_width}" height="${hokuyo_height}" depth="${hokuyo_depth}"/>
+      <xacro:box_inertia mass="0.001" width="${hokuyo_width}" height="${hokuyo_height}" depth="${hokuyo_depth}"/>
     </link>
     <joint name="laser_base_joint" type="fixed">

Commit message: The Laser is rotated to the front PID added to the diff drive controller AMCL test pathed. Please, smb verify.

File: leobot_description/urdf/sensors/hokuyo.urdf.xacro (robot description, xacro)
@@ -14,5 +14,5 @@
             </link>
             <joint name="laser_base_joint" type="fixed">
-              <origin xyz="${(base_radius - 0.0001)} 0.0 ${-base_height/2 + 0.01}" rpy="0.0 ${pi} 0.0" />
+              <origin xyz="${(base_radius - 0.0001)} 0.0 ${-base_height/2 + 0.01}" rpy="0.0 0.0 0.0" />
               <parent link="base_link" />
               <child link="laser_link" />
