Commit message: Attach the cameras to rotating camera stick in simulation
For task: Create rotational stereo camera URDF #130

File: leobot_description/urdf/materials.urdf.xacro (robot description, xacro)
@@ -31,3 +31,8 @@
     </material>
   </xacro:macro>
+    <xacro:macro name="yellow_material">
+        <material name="yellow">
+            <color rgba="1.0 1.0 0.0 1.0"/>
+        </material>
+    </xacro:macro>
 </robot>

File: leobot_description/urdf/sensors/camera.urdf.xacro (robot description, xacro)
@@ -2,5 +2,5 @@
 <robot xmlns:xacro="http://ros.org/wiki/xacro">
     <xacro:property name="camera_radius" value="0.025"/>
-    <xacro:property name="camera_mass" value="0.1"/>
+    <xacro:property name="camera_mass"   value="0.1"/>
     <xacro:macro name="fish_camera" params="prefix parent_link_name parent_height side parent_width">
         <link name="${prefix}_camera_link">
@@ -12,8 +12,9 @@
             <xacro:sphere_inertia mass="${camera_mass}" radius="${camera_radius}"/>
         </link>
-        <joint name="head_${prefix}_camera_joint" type="fixed">
-            <origin xyz="${side*(camera_radius + parent_width/2) - side*0.005} ${-parent_height/2 + camera_radius} 0" rpy="${pi/2 + side * pi/2 } ${pi/2 + side * pi/2 } 0"/>
-            <parent link="${parent_link_name}" />
-            <child link="${prefix}_camera_link" />
+        <joint name="${prefix}_camera_joint" type="fixed">
+            <origin xyz="${-camera_radius - parent_width/2} ${side*(-camera_radius/2 + parent_height/2)} 0"
+                    rpy="${pi/2 + side * pi/2} ${pi/2 + side * pi/2} 0"/>
+            <parent link="${parent_link_name}"/>
+            <child link="${prefix}_camera_link"/>
         </joint>
     </xacro:macro>
