Commit message: Added whells to udrf. No result on visual presentation. [ERROR] [1518718664.102881522]: Could not parse visual element for Link [caster_wheel_link] [ERROR] [1518718664.102986561]: Could not parse visual element for Link [left_bearing_link] [ERROR] [1518718664.103117951]: Could not parse visual element for Link [right_bearing_link]

File: leobot_description/urdf/wheels.urdf.xacro (robot description, xacro)
@@ -4,5 +4,5 @@
         <link name="${prefix}_bearing_link">>
             <visual>
-                <xacro:sphere_geometry radius="${bearing_radius}"/>
+                <mesh filename="package://leobot_description/meshes/wheel.stl" scale="0.001 0.001 0.001"/>
                 <xacro:blue_material/>
             </visual>
@@ -17,5 +17,5 @@
         <link name="${prefix}_wheel_link">
             <visual>
-                <xacro:cylinder_geometry radius="${radius}" height="${width}"/>
+                 <xacro:cylinder_geometry radius="${radius}" height="${width}"/>
                 <xacro:red_material/>
             </visual>
@@ -44,5 +44,5 @@
         <link name="caster_wheel_link">
             <visual>
-                <xacro:sphere_geometry radius="${radius}"/>
+                <mesh filename="package://leobot_description/meshes/wheel-2-with-ball.stl" scale="0.001 0.001 0.001"/>
                 <xacro:red_material/>
             </visual>

Commit message: Wheels were placed correctly.Think about refactoring wheel macros.

File: leobot_description/urdf/wheels.urdf.xacro (robot description, xacro)
@@ -4,8 +4,8 @@
         <link name="${prefix}_bearing_link">>
             <visual>
-                <geometry>
+<!--                <geometry>
                     <mesh filename="package://leobot_description/meshes/wheel.stl" scale="0.001 0.001 0.001"/>
                     <xacro:blue_material/>
-                </geometry>
+                </geometry>-->
             </visual>
             <xacro:sphere_collision radius="${bearing_radius}"/>
@@ -13,5 +13,5 @@
         </link>
         <joint name="${prefix}_bearing_base_joint" type="fixed">
-            <origin rpy="0 0 0" xyz="0.0 ${direction * (base_radius + bearing_radius - 0.0001)} ${-(base_height/2 - bearing_radius)}"/>
+            <origin rpy="0 0 0" xyz="0.35 ${direction * (base_radius + bearing_radius - 0.0001)} 0.04"/>
             <parent link="base_link"/>
             <child link="${prefix}_bearing_link"/>
@@ -19,5 +19,10 @@
         <link name="${prefix}_wheel_link">
             <visual>
-                 <xacro:cylinder_geometry radius="${radius}" height="${width}"/>
+                 <!--<xacro:cylinder_geometry radius="${radius}" height="${width}"/>-->
+                <origin rpy="${pi / 2} 0  0 " xyz ="0 0 0"/>
+              <geometry>
+                    <mesh filename="package://leobot_description/meshes/wheel.stl" scale="0.001 0.001 0.001"/>
+                    <xacro:blue_material/>
+                </geometry>
                 <xacro:red_material/>
             </visual>
@@ -27,4 +32,5 @@
         <joint name="${prefix}_wheel_bearing_joint" type="continuous">
             <origin rpy="${pi / 2} 0 0" xyz="0.0 ${direction * (bearing_radius + width/2 - 0.0001)} 0.0"/>
+            <!--<origin rpy="0 0 0" xyz="0.0 ${direction * (bearing_radius + width/2 - 0.0001)} 0.0"/>-->
             <parent link="${prefix}_bearing_link"/>
             <child link="${prefix}_wheel_link"/>
@@ -57,5 +63,5 @@
             <parent link="base_link"/>
             <child link="caster_wheel_link"/>
-            <origin rpy="0 0 0" xyz="${base_radius - radius - 0.01} 0.0 ${-(base_height/2 + radius - 0.01)}"/>
+            <origin rpy="0 0 0" xyz="1 0.0 -0.04"/>
         </joint>
     </xacro:macro>

Commit message: Corrected back and front of the robot First attempt to build a map. ToDo: built map properly

File: leobot_description/urdf/wheels.urdf.xacro (robot description, xacro)
@@ -53,5 +53,5 @@
             <parent link="base_link"/>
             <child link="caster_wheel_link"/>
-            <origin rpy="0 0 0" xyz="${base_radius - radius - 0.01} 0.0 ${-(base_height/2 + radius - 0.01)}"/>
+            <origin rpy="0 0 0" xyz="${-(base_radius - radius - 0.01)} 0.0 ${-(base_height/2 + radius - 0.01)}"/>
         </joint>
     </xacro:macro>

Commit message: Fix the XML structure in wheels.urdf.xacro
For task: Fix the XML structure in wheels.urdf.xacro #140

File: leobot_description/urdf/wheels.urdf.xacro (robot description, xacro)
@@ -8,5 +8,5 @@
     <xacro:macro name="mecanum_wheel"
                  params="prefix wheel_type side position parent_length parent_height parent_width">
-        <link name="${prefix}_motor_holder">>
+        <link name="${prefix}_motor_holder">
             <visual>
                 <xacro:cylinder_geometry radius="${motor_holder_radius}" height="${motor_holder_height}"/>
