Commit message: LeoBotUrdf

File: leobot_description/robot/robot.urdf.xacro (robot description, xacro)
@@ -57,4 +57,5 @@
     <parent link="body_link"/>
     <child link="left_wheel_link"/>
+    <axis xyz="0 0 1" />
   </joint>
        <!-- Leo_right_wheel -->
@@ -72,4 +73,5 @@
     <parent link="body_link"/>
     <child link="right_wheel_link"/>
+    <axis xyz="0 0 1" />
   </joint>
        <!-- Leo_caster_wheel -->

Commit message: Create URDF for stereo camera rotation

File: leobot_description/robot/robot.urdf.xacro (robot description, xacro)
@@ -13,4 +13,22 @@
     <xacro:cylinder_inertia mass="10" radius="0.25" height="1.0"/>
   </link>
+  <!-- Head link -->
+  <link name="head_link">
+    <visual>
+      <xacro:cylinder_geometry radius="0.15" height="0.1"/>
+      <xacro:navajo_white_material/>
+    </visual>
+    <xacro:cylinder_collision radius="0.15" height="0.1"/>
+    <xacro:cylinder_inertia mass="1" radius="0.15" height="0.1"/>
+  </link>
+  <joint name="head_link_joint" type="revolute">
+    <origin rpy="0 0 0" xyz="0 0 0.525"/>
+    <axis xyz="0 0 1" />
+    <parent link="base_link"/>
+    <child link="head_link"/>
+    <limit effort="10" velocity="10" lower="-1.57" upper="1.57" />
+    <dynamics damping="10" friction="1" />
+  </joint>
+  <!-- Left camera link -->
   <link name="camera_left_link">
     <visual>
@@ -22,8 +40,9 @@
   </link>
   <joint name="camera_left_link_joint" type="fixed">
-    <origin rpy="0 0 0" xyz="0 0.075 0.525"/>
-    <parent link="base_link"/>
+    <origin rpy="0 0 0" xyz="0 0.075 0.1"/>
+    <parent link="head_link"/>
     <child link="camera_left_link"/>
   </joint>
+  <!-- Right camera link-->
   <link name="camera_right_link">
     <visual>
@@ -35,6 +54,6 @@
   </link>
   <joint name="camera_right_link_joint" type="fixed">
-    <origin rpy="0 0 0" xyz="0 -0.075 0.525"/>
-    <parent link="base_link"/>
+    <origin rpy="0 0 0" xyz="0 -0.075 0.1"/>
+    <parent link="head_link"/>
     <child link="camera_right_link"/>
   </joint>

Commit message: Fix expressions for pi and delete comment

File: leobot_description/robot/robot.urdf.xacro (robot description, xacro)
@@ -13,5 +13,4 @@
     <xacro:cylinder_inertia mass="10" radius="0.25" height="1.0"/>
   </link>
-  <!-- Head link -->
   <link name="head_link">
     <visual>
@@ -27,8 +26,7 @@
     <parent link="base_link"/>
     <child link="head_link"/>
-    <limit effort="10" velocity="10" lower="-1.57" upper="1.57" />
+    <limit effort="10" velocity="10" lower="${90/180*pi}" upper="${90/180*pi}" />
     <dynamics damping="10" friction="1" />
   </joint>
-  <!-- Left camera link -->
   <link name="camera_left_link">
     <visual>
@@ -44,5 +42,4 @@
     <child link="camera_left_link"/>
   </joint>
-  <!-- Right camera link-->
   <link name="camera_right_link">
     <visual>

Commit message: Change 90/180*pi on pi/2

File: leobot_description/robot/robot.urdf.xacro (robot description, xacro)
@@ -26,5 +26,5 @@
     <parent link="base_link"/>
     <child link="head_link"/>
-    <limit effort="10" velocity="10" lower="${90/180*pi}" upper="${90/180*pi}" />
+    <limit effort="10" velocity="10" lower="${-pi/2}" upper="${pi/2}" />
     <dynamics damping="10" friction="1" />
   </joint>

Commit message: Add transmission tag

File: leobot_description/robot/robot.urdf.xacro (robot description, xacro)
@@ -29,4 +29,14 @@
     <dynamics damping="10" friction="1" />
   </joint>
+  <transmission name="head_transmission">
+     <type>transmission_interface/SimpleTransmission</type>
+     <joint name="head_link_joint">
+       <hardwareInterface>EffortJointInterface</hardwareInterface>
+     </joint>
+     <actuator name="head_motor">
+       <hardwareInterface>EffortJointInterface</hardwareInterface>
+       <mechanicalReduction>1</mechanicalReduction>
+     </actuator>
+  </transmission>
   <link name="camera_left_link">
     <visual>

Commit message: remove dynamics tag and add hardware_interface

File: leobot_description/robot/robot.urdf.xacro (robot description, xacro)
@@ -27,10 +27,9 @@
     <child link="head_link"/>
     <limit effort="10" velocity="10" lower="${-pi/2}" upper="${pi/2}" />
-    <dynamics damping="10" friction="1" />
   </joint>
   <transmission name="head_transmission">
      <type>transmission_interface/SimpleTransmission</type>
      <joint name="head_link_joint">
-       <hardwareInterface>EffortJointInterface</hardwareInterface>
+       <hardwareInterface>hardware_interface/EffortJointInterface</hardwareInterface>
      </joint>
      <actuator name="head_motor">

Commit message: Small fixes of formatting. Added nodejs-legacy dependency

File: leobot_description/robot/robot.urdf.xacro (robot description, xacro)
@@ -5,5 +5,5 @@
   <xacro:include filename="$(find leobot_description)/urdf/common.urdf.xacro"/>
   <xacro:include filename="$(find leobot_description)/urdf/wheels.urdf.xacro"/>
-    <!-- Robot properties -->
+  <!-- Robot properties -->
   <xacro:property name="base_radius" value="0.25"/>
   <xacro:property name="base_height" value="1.0"/>
@@ -42,12 +42,12 @@
   </joint>
   <transmission name="head_transmission">
-     <type>transmission_interface/SimpleTransmission</type>
-     <joint name="head_link_joint">
-       <hardwareInterface>hardware_interface/EffortJointInterface</hardwareInterface>
-     </joint>
-     <actuator name="head_motor">
-       <hardwareInterface>EffortJointInterface</hardwareInterface>
-       <mechanicalReduction>1</mechanicalReduction>
-     </actuator>
+    <type>transmission_interface/SimpleTransmission</type>
+    <joint name="head_link_joint">
+      <hardwareInterface>hardware_interface/EffortJointInterface</hardwareInterface>
+    </joint>
+    <actuator name="head_motor">
+      <hardwareInterface>EffortJointInterface</hardwareInterface>
+      <mechanicalReduction>1</mechanicalReduction>
+    </actuator>
   </transmission>
   <link name="camera_left_link">

File: leobot_description/urdf/wheels.urdf.xacro (robot description, xacro)
@@ -4,9 +4,9 @@
         <link name="${prefix}_bearing_link">>
             <visual>
-              <xacro:sphere_geometry radius="${bearing_radius}"/>
-              <xacro:blue_material/>
+                <xacro:sphere_geometry radius="${bearing_radius}"/>
+                <xacro:blue_material/>
             </visual>
-        <xacro:sphere_collision radius="${bearing_radius}"/>
-        <xacro:sphere_inertia mass="0.1" radius="${bearing_radius}"/>
+            <xacro:sphere_collision radius="${bearing_radius}"/>
+            <xacro:sphere_inertia mass="0.1" radius="${bearing_radius}"/>
         </link>
         <joint name="${prefix}_bearing_base_joint" type="fixed">
@@ -17,6 +17,6 @@
         <link name="${prefix}_wheel_link">
             <visual>
-              <xacro:cylinder_geometry radius="${radius}" height="${width}"/>
-              <xacro:red_material/>
+                <xacro:cylinder_geometry radius="${radius}" height="${width}"/>
+                <xacro:red_material/>
             </visual>
             <xacro:cylinder_collision radius="${radius}" height="${width}"/>

Commit message: base.stl model added to udrf

File: leobot_description/robot/robot.urdf.xacro (robot description, xacro)
@@ -17,9 +17,10 @@
   <link name="base_link">
     <visual>
-      <xacro:cylinder_geometry radius="${base_radius}" height="${base_height}"/>
+      <origin xyz="0 0 0" rpy="0 0 0"/>
+      <geometry>
+          <mesh filename="package://leobot_description/meshes/base.stl" scale="0.001 0.001 0.001"/>
+      </geometry>
       <xacro:navajo_white_material/>
     </visual>
-    <xacro:cylinder_collision radius="${base_radius}" height="${base_height}"/>
-    <xacro:cylinder_inertia mass="10" radius="${base_radius}" height="${base_height}"/>
   </link>
   <xacro:caster_wheel radius="${caster_radius}" mass="${caster_mass}" base_radius="${base_radius}" base_height="${base_height}"/>

Commit message: Base was moved and rotated. Wheels are visible now.

File: leobot_description/robot/robot.urdf.xacro (robot description, xacro)
@@ -17,5 +17,5 @@
   <link name="base_link">
     <visual>
-      <origin xyz="0 0 0" rpy="0 0 0"/>
+      <origin xyz="0 -0.25 -0.4" rpy="0 0 ${pi}"/>
       <geometry>
           <mesh filename="package://leobot_description/meshes/base.stl" scale="0.001 0.001 0.001"/>

File: leobot_description/urdf/wheels.urdf.xacro (robot description, xacro)
@@ -4,6 +4,8 @@
         <link name="${prefix}_bearing_link">>
             <visual>
-                <mesh filename="package://leobot_description/meshes/wheel.stl" scale="0.001 0.001 0.001"/>
-                <xacro:blue_material/>
+                <geometry>
+                    <mesh filename="package://leobot_description/meshes/wheel.stl" scale="0.001 0.001 0.001"/>
+                    <xacro:blue_material/>
+                </geometry>
             </visual>
             <xacro:sphere_collision radius="${bearing_radius}"/>
@@ -44,6 +46,8 @@
         <link name="caster_wheel_link">
             <visual>
-                <mesh filename="package://leobot_description/meshes/wheel-2-with-ball.stl" scale="0.001 0.001 0.001"/>
-                <xacro:red_material/>
+                <geometry>
+                    <mesh filename="package://leobot_description/meshes/wheel-2-with-ball.stl" scale="0.001 0.001 0.001"/>
+                    <xacro:red_material/>
+                </geometry>
             </visual>
             <xacro:sphere_collision radius="${radius}"/>

Commit message: Base and tower placed correctly. Problem with wheels and head

File: leobot_description/robot/robot.urdf.xacro (robot description, xacro)
@@ -6,6 +6,9 @@
   <xacro:include filename="$(find leobot_description)/urdf/wheels.urdf.xacro"/>
   <!-- Robot properties -->
+  <xacro:property name="base_width" value="0.7"/>
+  <xacro:property name="base_length" value="1.132"/>
+  <xacro:property name="base_height" value="0.4"/>
   <xacro:property name="base_radius" value="0.25"/>
-  <xacro:property name="base_height" value="1.0"/>
+  <xacro:property name="tower_height" value="1.225"/>
   <xacro:property name="caster_radius" value="0.05"/>
   <xacro:property name="caster_mass" value="10"/>
@@ -17,5 +20,5 @@
   <link name="base_link">
     <visual>
-      <origin xyz="0 -0.25 -0.4" rpy="0 0 ${pi}"/>
+      <origin xyz="0 -0.25 0" rpy="0 0 ${pi}"/>
       <geometry>
           <mesh filename="package://leobot_description/meshes/base.stl" scale="0.001 0.001 0.001"/>
@@ -24,7 +27,30 @@
     </visual>
   </link>
+   <link name="base_link_inertia">
+    <xacro:box_collision width="${base_width + 0.05}" depth="${base_length+0.05}" height="${base_height + 0.05}"/>
+    <xacro:box_inertia mass="3.0" width="${base_length}" depth="${base_height}" height="${base_width}"/>
+  </link>
+  <joint name="base_link_inertia_joint" type="fixed">
+    <origin xyz="0 0 0" rpy="0 0 0"/>
+    <parent link="base_link"/>
+    <child link="base_link_inertia"/>
+  </joint>
   <xacro:caster_wheel radius="${caster_radius}" mass="${caster_mass}" base_radius="${base_radius}" base_height="${base_height}"/>
   <xacro:standard_wheel prefix="left" direction="1.0" bearing_radius="${bearing_radius}" radius="${wheel_radius}" width="${wheel_width}" mass="${wheel_mass}" base_radius="${base_radius}"/>
   <xacro:standard_wheel prefix="right" direction="-1.0" bearing_radius="${bearing_radius}" radius="${wheel_radius}" width="${wheel_width}" mass="${wheel_mass}" base_radius="${base_radius}"/>
+    <link name="tower_link">
+        <visual>
+          <origin xyz="0 -0.25 0" rpy="0 0 ${pi}"/>
+          <geometry>
+              <mesh filename="package://leobot_description/meshes/tower.stl" scale="0.001 0.001 0.001"/>
+          </geometry>
+          <xacro:navajo_white_material/>
+        </visual>
+      </link>
+       <joint name="tower_link_joint" type="fixed">
+        <origin xyz="0 0 0" rpy="0 0 0"/>
+        <parent link="base_link_inertia"/>
+        <child link="tower_link"/>
+      </joint>
   <link name="head_link">
     <visual>
@@ -36,7 +62,7 @@
   </link>
   <joint name="head_link_joint" type="revolute">
-    <origin rpy="0 0 0" xyz="0 0 0.525"/>
+    <origin rpy="0 0 0" xyz="0 0 0"/>
     <axis xyz="0 0 1" />
-    <parent link="base_link"/>
+    <parent link="tower_link"/>
     <child link="head_link"/>
     <limit effort="10" velocity="10" lower="${-pi/2}" upper="${pi/2}" />

Commit message: Wheel parameters update

File: leobot_description/robot/robot.urdf.xacro (robot description, xacro)
@@ -13,5 +13,5 @@
   <xacro:property name="caster_radius" value="0.05"/>
   <xacro:property name="caster_mass" value="10"/>
-  <xacro:property name="wheel_width" value="0.005"/>
+  <xacro:property name="wheel_width" value="0.035"/>
   <xacro:property name="wheel_radius" value="0.1"/>
   <xacro:property name="wheel_mass" value="10"/>

Commit message: Base and tower stls were replaced on similar with centered start of coordionates. Head is movable and was placed in correct position on tower. Wheels require reposotioning.

File: leobot_description/robot/robot.urdf.xacro (robot description, xacro)
@@ -11,4 +11,5 @@
   <xacro:property name="base_radius" value="0.25"/>
   <xacro:property name="tower_height" value="1.225"/>
+  <xacro:property name="head_height" value="0.1"/>
   <xacro:property name="caster_radius" value="0.05"/>
   <xacro:property name="caster_mass" value="10"/>
@@ -20,5 +21,5 @@
   <link name="base_link">
     <visual>
-      <origin xyz="0 -0.25 0" rpy="0 0 ${pi}"/>
+      <origin xyz="0 0 0" rpy="0 0 ${-pi}"/>
       <geometry>
           <mesh filename="package://leobot_description/meshes/base.stl" scale="0.001 0.001 0.001"/>
@@ -41,5 +42,5 @@
     <link name="tower_link">
         <visual>
-          <origin xyz="0 -0.25 0" rpy="0 0 ${pi}"/>
+          <origin xyz="0 0 0" rpy="0 0 ${-pi}"/>
           <geometry>
               <mesh filename="package://leobot_description/meshes/tower.stl" scale="0.001 0.001 0.001"/>
@@ -55,5 +56,5 @@
   <link name="head_link">
     <visual>
-      <xacro:cylinder_geometry radius="0.15" height="0.1"/>
+      <xacro:cylinder_geometry radius="0.15" height="${head_height}"/>
       <xacro:navajo_white_material/>
     </visual>
@@ -62,5 +63,5 @@
   </link>
   <joint name="head_link_joint" type="revolute">
-    <origin rpy="0 0 0" xyz="0 0 0"/>
+    <origin rpy="0 0 0" xyz="0.75 0 ${base_height+tower_height+head_height/2}"/>
     <axis xyz="0 0 1" />
     <parent link="tower_link"/>

Commit message: Added new stl geometry for robot head

File: leobot_description/robot/robot.urdf.xacro (robot description, xacro)
@@ -10,5 +10,5 @@
   <xacro:property name="base_height" value="0.4"/>
   <xacro:property name="base_radius" value="0.25"/>
-  <xacro:property name="tower_height" value="1.225"/>
+  <xacro:property name="tower_height" value="1.125"/>
   <xacro:property name="head_height" value="0.1"/>
   <xacro:property name="caster_radius" value="0.05"/>
@@ -56,5 +56,9 @@
   <link name="head_link">
     <visual>
-      <xacro:cylinder_geometry radius="0.15" height="${head_height}"/>
+      <origin xyz="-0.75 0 -${base_height+tower_height+head_height/2}" rpy="0 0 ${-pi}"/>
+          <geometry>
+              <mesh filename="package://leobot_description/meshes/head.stl" scale="0.001 0.001 0.001"/>
+          </geometry>
+      <!--<xacro:cylinder_geometry radius="0.15" height="${head_height}"/>-->
       <xacro:navajo_white_material/>
     </visual>

Commit message: Fixed rViz errors.

File: leobot_description/robot/robot.urdf.xacro (robot description, xacro)
@@ -60,5 +60,4 @@
               <mesh filename="package://leobot_description/meshes/head.stl" scale="0.001 0.001 0.001"/>
           </geometry>
-      <!--<xacro:cylinder_geometry radius="0.15" height="${head_height}"/>-->
       <xacro:navajo_white_material/>
     </visual>

File: leobot_description/urdf/wheels.urdf.xacro (robot description, xacro)
@@ -4,8 +4,6 @@
         <link name="${prefix}_bearing_link">>
             <visual>
-<!--                <geometry>
-                    <mesh filename="package://leobot_description/meshes/wheel.stl" scale="0.001 0.001 0.001"/>
-                    <xacro:blue_material/>
-                </geometry>-->
+                <xacro:sphere_geometry radius="${bearing_radius}"/>
+                <xacro:blue_material/>
             </visual>
             <xacro:sphere_collision radius="${bearing_radius}"/>
@@ -19,5 +17,4 @@
         <link name="${prefix}_wheel_link">
             <visual>
-                 <!--<xacro:cylinder_geometry radius="${radius}" height="${width}"/>-->
                 <origin rpy="${pi / 2} 0  0 " xyz ="0 0 0"/>
               <geometry>
@@ -32,5 +29,4 @@
         <joint name="${prefix}_wheel_bearing_joint" type="continuous">
             <origin rpy="${pi / 2} 0 0" xyz="0.0 ${direction * (bearing_radius + width/2 - 0.0001)} 0.0"/>
-            <!--<origin rpy="0 0 0" xyz="0.0 ${direction * (bearing_radius + width/2 - 0.0001)} 0.0"/>-->
             <parent link="${prefix}_bearing_link"/>
             <child link="${prefix}_wheel_link"/>

Commit message: Attempt to change base collision position by adding origin tag.

File: leobot_description/robot/robot.urdf.xacro (robot description, xacro)
@@ -29,7 +29,8 @@
   </link>
    <link name="base_link_inertia">
-    <xacro:box_collision width="${base_width + 0.05}" depth="${base_length+0.05}" height="${base_height + 0.05}"/>
+    <origin xyz="${-base_length/2} 0 ${base_height/2}" rpy="0 0 ${-pi}"/>
+    <xacro:box_collision width="${base_width + 0.05}" depth="${base_length+0.05}" height="${base_height + 0.05}" />
     <xacro:box_inertia mass="3.0" width="${base_length}" depth="${base_height}" height="${base_width}"/>
-  </link>
+   </link>
   <joint name="base_link_inertia_joint" type="fixed">
     <origin xyz="0 0 0" rpy="0 0 0"/>

Commit message: Added collisions for base_inertia, tower and head links.

File: leobot_description/robot/robot.urdf.xacro (robot description, xacro)
@@ -29,6 +29,10 @@
   </link>
    <link name="base_link_inertia">
-    <origin xyz="${-base_length/2} 0 ${base_height/2}" rpy="0 0 ${-pi}"/>
-    <xacro:box_collision width="${base_width + 0.05}" depth="${base_length+0.05}" height="${base_height + 0.05}" />
+     <collision>
+       <origin xyz="${base_length/2} 0 ${base_height/2} " rpy="0 0 0"/>
+       <geometry>
+         <box size="${base_length+0.05} ${base_width + 0.05}  ${base_height + 0.05}"/>
+       </geometry>
+      </collision>
     <xacro:box_inertia mass="3.0" width="${base_length}" depth="${base_height}" height="${base_width}"/>
    </link>
@@ -49,4 +53,10 @@
           <xacro:navajo_white_material/>
         </visual>
+        <collision>
+            <origin xyz="${base_length/2} 0 ${base_height+tower_height/2} " rpy="0 0 0"/>
+            <geometry>
+              <box size="${base_length+0.05} ${base_width + 0.05}  ${tower_height + 0.05}"/>
+            </geometry>
+        </collision>
       </link>
        <joint name="tower_link_joint" type="fixed">
@@ -63,6 +73,10 @@
       <xacro:navajo_white_material/>
     </visual>
-    <xacro:cylinder_collision radius="0.15" height="0.1"/>
-    <xacro:cylinder_inertia mass="1" radius="0.15" height="0.1"/>
+    <collision>
+      <geometry>
+        <cylinder length="0.2" radius="0.35"/>
+      </geometry>
+    </collision>
+    <xacro:cylinder_inertia mass="1" radius="0.35" height="0.1"/>
   </link>
   <joint name="head_link_joint" type="revolute">

Commit message: Added collisions for base_inertia, tower and head links.

File: leobot_description/robot/robot.urdf.xacro (robot description, xacro)
@@ -59,4 +59,5 @@
             </geometry>
         </collision>
+        <xacro:box_inertia mass="3.0" width="${base_width}" depth="${base_length}" height="${tower_height}"/>
       </link>
        <joint name="tower_link_joint" type="fixed">
@@ -75,8 +76,8 @@
     <collision>
       <geometry>
-        <cylinder length="0.2" radius="0.35"/>
+        <cylinder length="${head_height*2}" radius="${base_width/2}"/>
       </geometry>
     </collision>
-    <xacro:cylinder_inertia mass="1" radius="0.35" height="0.1"/>
+    <xacro:cylinder_inertia mass="1" radius="${base_width/2}" height="${head_height*2}"/>
   </link>
   <joint name="head_link_joint" type="revolute">
