Commit message: Wheels macroses were refactored according to suggestions of AndriyPt

File: leobot_description/robot/robot.urdf.xacro (robot description, xacro)
@@ -9,5 +9,5 @@
   <xacro:property name="base_length" value="1.132"/>
   <xacro:property name="base_height" value="0.4"/>
-  <xacro:property name="base_radius" value="0.25"/>
+  <xacro:property name="distance_between_wheels" value="0.55"/>
   <xacro:property name="tower_height" value="1.125"/>
   <xacro:property name="head_height" value="0.1"/>
@@ -17,4 +17,8 @@
   <xacro:property name="wheel_radius" value="0.1"/>
   <xacro:property name="wheel_mass" value="10"/>
+  <xacro:property name="wheel_position_x" value="0.35"/>
+  <xacro:property name="wheel_position_z" value="0.04"/>
+  <xacro:property name="caster_wheel_position_x" value="1"/>
+  <xacro:property name="caster_wheel_position_z" value="-0.04"/>
   <xacro:property name="bearing_radius" value="0.01"/>
   <!-- Robot links -->
@@ -42,7 +46,7 @@
     <child link="base_link_inertia"/>
   </joint>
-  <xacro:caster_wheel radius="${caster_radius}" mass="${caster_mass}" base_radius="${base_radius}" base_height="${base_height}"/>
-  <xacro:standard_wheel prefix="left" direction="-1.0" bearing_radius="${bearing_radius}" radius="${wheel_radius}" width="${wheel_width}" mass="${wheel_mass}" base_radius="${base_radius}"/>
-  <xacro:standard_wheel prefix="right" direction="1.0" bearing_radius="${bearing_radius}" radius="${wheel_radius}" width="${wheel_width}" mass="${wheel_mass}" base_radius="${base_radius}"/>
+  <xacro:caster_wheel radius="${caster_radius}" mass="${caster_mass}" position_x="${caster_wheel_position_x}" position_z="${caster_wheel_position_z}"/>
+  <xacro:standard_wheel prefix="left" direction="-1.0" bearing_radius="${bearing_radius}" radius="${wheel_radius}" width="${wheel_width}" mass="${wheel_mass}" distance_between_wheels="${distance_between_wheels}" position_x="${wheel_position_x}" position_z="${wheel_position_z}"/>
+  <xacro:standard_wheel prefix="right" direction="1.0" bearing_radius="${bearing_radius}" radius="${wheel_radius}" width="${wheel_width}" mass="${wheel_mass}" distance_between_wheels="${distance_between_wheels}" position_x="${wheel_position_x}" position_z="${wheel_position_z}"/>
     <link name="tower_link">
         <visual>

File: leobot_description/urdf/wheels.urdf.xacro (robot description, xacro)
@@ -1,5 +1,5 @@
 <?xml version="1.0"?>
 <robot xmlns:xacro="http://ros.org/wiki/xacro">
-    <xacro:macro name="standard_wheel" params="prefix direction bearing_radius radius width mass base_radius">
+    <xacro:macro name="standard_wheel" params="prefix direction bearing_radius radius width mass distance_between_wheels position_x position_z">
         <link name="${prefix}_bearing_link">>
             <visual>
@@ -11,5 +11,5 @@
         </link>
         <joint name="${prefix}_bearing_base_joint" type="fixed">
-            <origin rpy="0 0 0" xyz="0.35 ${direction * (base_radius + bearing_radius - 0.0001)} 0.04"/>
+            <origin rpy="0 0 0" xyz="${position_x} ${direction * (distance_between_wheels/2 + bearing_radius - 0.0001)} ${position_z}"/>
             <parent link="base_link"/>
             <child link="${prefix}_bearing_link"/>
@@ -28,5 +28,5 @@
         </link>
         <joint name="${prefix}_wheel_bearing_joint" type="continuous">
-            <origin rpy="${pi / 2} 0 0" xyz="0.0 ${direction * (bearing_radius + width/2 - 0.0001)} 0.0"/>
+            <origin rpy="${pi / 2} 0 0" xyz="0.0 0.0 0.0"/>
             <parent link="${prefix}_bearing_link"/>
             <child link="${prefix}_wheel_link"/>
@@ -45,5 +45,5 @@
         </transmission>
     </xacro:macro>
-    <xacro:macro name="caster_wheel" params="radius mass base_radius base_height">
+    <xacro:macro name="caster_wheel" params="radius mass position_x position_z">
         <link name="caster_wheel_link">
             <visual>
@@ -59,5 +59,5 @@
             <parent link="base_link"/>
             <child link="caster_wheel_link"/>
-            <origin rpy="0 0 0" xyz="1 0.0 -0.04"/>
+            <origin rpy="0 0 0" xyz="${position_x} 0.0 ${position_z}"/>
         </joint>
     </xacro:macro>

Commit message: Fixed frames orientation and direction of movement for diff drive controller

File: leobot_description/robot/robot.urdf.xacro (robot description, xacro)
@@ -1,12 +1,11 @@
 <?xml version="1.0"?>
 <robot name="leobot" xmlns:xacro="http://ros.org/wiki/xacro">
-  <!-- Included files -->
   <xacro:include filename="$(find leobot_description)/urdf/materials.urdf.xacro"/>
   <xacro:include filename="$(find leobot_description)/urdf/common.urdf.xacro"/>
   <xacro:include filename="$(find leobot_description)/urdf/wheels.urdf.xacro"/>
-  <!-- Robot properties -->
   <xacro:property name="base_width" value="0.7"/>
   <xacro:property name="base_length" value="1.132"/>
   <xacro:property name="base_height" value="0.4"/>
+  <xacro:property name="safety_width" value="0.03"/>
   <xacro:property name="distance_between_wheels" value="0.55"/>
   <xacro:property name="tower_height" value="1.125"/>
@@ -17,63 +16,73 @@
   <xacro:property name="wheel_radius" value="0.1"/>
   <xacro:property name="wheel_mass" value="10"/>
-  <xacro:property name="wheel_position_x" value="0.35"/>
-  <xacro:property name="wheel_position_z" value="0.04"/>
-  <xacro:property name="caster_wheel_position_x" value="1"/>
+  <xacro:property name="wheel_position_x" value="-0.35"/>
+  <xacro:property name="wheel_position_z" value="0.02"/>
+  <xacro:property name="caster_wheel_position_x" value="-1.0"/>
   <xacro:property name="caster_wheel_position_z" value="-0.04"/>
   <xacro:property name="bearing_radius" value="0.01"/>
-  <!-- Robot links -->
-  <link name="base_link">
+  <link name="base_link"/>
+  <link name="chassis">
     <visual>
-      <origin xyz="0 0 0" rpy="0 0 ${-pi}"/>
       <geometry>
-          <mesh filename="package://leobot_description/meshes/base.stl" scale="0.001 0.001 0.001"/>
+        <mesh filename="package://leobot_description/meshes/base.stl" scale="0.001 0.001 0.001"/>
       </geometry>
       <xacro:navajo_white_material/>
     </visual>
   </link>
-   <link name="base_link_inertia">
-     <collision>
-       <origin xyz="${base_length/2} 0 ${base_height/2} " rpy="0 0 0"/>
-       <geometry>
-         <box size="${base_length+0.05} ${base_width + 0.05}  ${base_height + 0.05}"/>
-       </geometry>
-      </collision>
-    <xacro:box_inertia mass="3.0" width="${base_length}" depth="${base_height}" height="${base_width}"/>
-   </link>
-  <joint name="base_link_inertia_joint" type="fixed">
+  <joint name="base_link_joint" type="fixed">
+    <origin xyz="0 0 0.05" rpy="0 0 0" />
+    <parent link="base_link" />
+    <child link="chassis" />
+  </joint>
+  <link name="chassis_inertia">
+    <collision>
+      <origin xyz="${-base_length/2} 0 ${base_height/2 - safety_width}" rpy="0 0 0"/>
+      <geometry>
+        <box size="${base_length + safety_width} ${base_width + safety_width} ${base_height + safety_width}"/>
+      </geometry>
+    </collision>
+    <xacro:box_inertia mass="10.0" width="${base_width}" depth="${base_length}" height="${base_height}"
+                       x="${-base_length/2}" z="${base_height/2}"/>
+  </link>
+  <joint name="chassis_inertia_joint" type="fixed">
+    <origin xyz="0 0 0" rpy="0 0 0" />
+    <parent link="chassis" />
+    <child link="chassis_inertia" />
+  </joint>
+  <xacro:caster_wheel radius="${caster_radius}" mass="${caster_mass}" x="${caster_wheel_position_x}"
+                      z="${caster_wheel_position_z}"/>
+  <xacro:standard_wheel prefix="left" direction="1.0" bearing_radius="${bearing_radius}" radius="${wheel_radius}"
+                        width="${wheel_width}" mass="${wheel_mass}" distance_between_wheels="${distance_between_wheels}"
+                        x="${wheel_position_x}" z="${wheel_position_z}"/>
+  <xacro:standard_wheel prefix="right" direction="-1.0" bearing_radius="${bearing_radius}" radius="${wheel_radius}"
+                        width="${wheel_width}" mass="${wheel_mass}" distance_between_wheels="${distance_between_wheels}"
+                        x="${wheel_position_x}" z="${wheel_position_z}"/>
+  <link name="tower_link">
+    <visual>
+      <origin xyz="0 0 0" rpy="0 0 0"/>
+      <geometry>
+        <mesh filename="package://leobot_description/meshes/tower.stl" scale="0.001 0.001 0.001"/>
+      </geometry>
+      <xacro:navajo_white_material/>
+    </visual>
+    <collision>
+      <origin xyz="${-base_length/2} 0 ${base_height + tower_height/2} " rpy="0 0 0"/>
+      <geometry>
+        <box size="${base_length + safety_width} ${base_width + safety_width} ${tower_height + safety_width}"/>
+      </geometry>
+    </collision>
+    <xacro:box_inertia mass="3.0" width="${base_width}" depth="${base_length}" height="${tower_height}"/>
+  </link>
+  <joint name="tower_link_joint" type="fixed">
     <origin xyz="0 0 0" rpy="0 0 0"/>
-    <parent link="base_link"/>
-    <child link="base_link_inertia"/>
+    <parent link="chassis"/>
+    <child link="tower_link"/>
   </joint>
-  <xacro:caster_wheel radius="${caster_radius}" mass="${caster_mass}" position_x="${caster_wheel_position_x}" position_z="${caster_wheel_position_z}"/>
-  <xacro:standard_wheel prefix="left" direction="-1.0" bearing_radius="${bearing_radius}" radius="${wheel_radius}" width="${wheel_width}" mass="${wheel_mass}" distance_between_wheels="${distance_between_wheels}" position_x="${wheel_position_x}" position_z="${wheel_position_z}"/>
-  <xacro:standard_wheel prefix="right" direction="1.0" bearing_radius="${bearing_radius}" radius="${wheel_radius}" width="${wheel_width}" mass="${wheel_mass}" distance_between_wheels="${distance_between_wheels}" position_x="${wheel_position_x}" position_z="${wheel_position_z}"/>
-    <link name="tower_link">
-        <visual>
-          <origin xyz="0 0 0" rpy="0 0 ${-pi}"/>
-          <geometry>
-              <mesh filename="package://leobot_description/meshes/tower.stl" scale="0.001 0.001 0.001"/>
-          </geometry>
-          <xacro:navajo_white_material/>
-        </visual>
-        <collision>
-            <origin xyz="${base_length/2} 0 ${base_height+tower_height/2} " rpy="0 0 0"/>
-            <geometry>
-              <box size="${base_length+0.05} ${base_width + 0.05}  ${tower_height + 0.05}"/>
-            </geometry>
-        </collision>
-        <xacro:box_inertia mass="3.0" width="${base_width}" depth="${base_length}" height="${tower_height}"/>
-      </link>
-       <joint name="tower_link_joint" type="fixed">
-        <origin xyz="0 0 0" rpy="0 0 0"/>
-        <parent link="base_link_inertia"/>
-        <child link="tower_link"/>
-      </joint>
   <link name="head_link">
     <visual>
-      <origin xyz="-0.75 0 -${base_height+tower_height+head_height/2}" rpy="0 0 ${-pi}"/>
-          <geometry>
-              <mesh filename="package://leobot_description/meshes/head.stl" scale="0.001 0.001 0.001"/>
-          </geometry>
+      <origin xyz="0.75 0 -${base_height+tower_height+head_height/2}" rpy="0 0 0"/>
+      <geometry>
+        <mesh filename="package://leobot_description/meshes/head.stl" scale="0.001 0.001 0.001"/>
+      </geometry>
       <xacro:navajo_white_material/>
     </visual>
@@ -86,5 +95,5 @@
   </link>
   <joint name="head_link_joint" type="revolute">
-    <origin rpy="0 0 0" xyz="0.75 0 ${base_height+tower_height+head_height/2}"/>
+    <origin rpy="0 0 0" xyz="-0.75 0 ${base_height+tower_height+head_height/2}"/>
     <axis xyz="0 0 1" />
     <parent link="tower_link"/>

File: leobot_description/urdf/common.urdf.xacro (robot description, xacro)
@@ -59,8 +59,8 @@
     </collision>
   </xacro:macro>
-  <xacro:macro name="box_inertia" params="mass width height depth">
+  <xacro:macro name="box_inertia" params="mass width height depth x:=0 y:=0 z:=0 roll:=0 pitch:=0 yaw:=0">
     <inertial>
+      <origin xyz="${x} ${y} ${z}" rpy="${roll} ${pitch} ${yaw}"/>
       <mass value="${mass}"/>
-      <origin xyz="0 0 0"/>
       <inertia ixx="${(depth*depth + height*height)*mass/12}" ixy="0.0" ixz="0.0"
                iyy="${(depth*depth + width*width)*mass/12}" iyz="0.0"

File: leobot_description/urdf/wheels.urdf.xacro (robot description, xacro)
@@ -1,22 +1,24 @@
 <?xml version="1.0"?>
 <robot xmlns:xacro="http://ros.org/wiki/xacro">
-    <xacro:macro name="standard_wheel" params="prefix direction bearing_radius radius width mass distance_between_wheels position_x position_z">
+    <xacro:macro name="standard_wheel"
+                 params="prefix direction bearing_radius radius width mass distance_between_wheels x z">
         <link name="${prefix}_bearing_link">>
             <visual>
-                <xacro:sphere_geometry radius="${bearing_radius}"/>
+                <xacro:cylinder_geometry radius="${bearing_radius}" height="${2 * wheel_width}"/>
                 <xacro:blue_material/>
             </visual>
-            <xacro:sphere_collision radius="${bearing_radius}"/>
-            <xacro:sphere_inertia mass="0.1" radius="${bearing_radius}"/>
+            <xacro:cylinder_collision radius="${bearing_radius}" height="${2 * wheel_width}"/>
+            <xacro:cylinder_inertia mass="0.01" radius="${bearing_radius}" height="${2 * wheel_width}"/>
         </link>
         <joint name="${prefix}_bearing_base_joint" type="fixed">
-            <origin rpy="0 0 0" xyz="${position_x} ${direction * (distance_between_wheels/2 + bearing_radius - 0.0001)} ${position_z}"/>
-            <parent link="base_link"/>
+            <origin rpy="${-pi / 2} 0 0"
+                    xyz="${x} ${direction * (distance_between_wheels/2 + wheel_width)} ${z}"/>
+            <parent link="chassis"/>
             <child link="${prefix}_bearing_link"/>
         </joint>
         <link name="${prefix}_wheel_link">
             <visual>
-                <origin rpy="${pi / 2} 0  0 " xyz ="0 0 0"/>
-              <geometry>
+                <origin rpy="${pi / 2} 0  0 " xyz="0 0 0"/>
+                <geometry>
                     <mesh filename="package://leobot_description/meshes/wheel.stl" scale="0.001 0.001 0.001"/>
                     <xacro:blue_material/>
@@ -28,8 +30,8 @@
         </link>
         <joint name="${prefix}_wheel_bearing_joint" type="continuous">
-            <origin rpy="${pi / 2} 0 0" xyz="0.0 0.0 0.0"/>
+            <origin rpy="0 0 0" xyz="0 0 ${direction * wheel_width/2}"/>
             <parent link="${prefix}_bearing_link"/>
             <child link="${prefix}_wheel_link"/>
-            <axis xyz="0 0 1" />
+            <axis xyz="0 0 1"/>
         </joint>
         <transmission name="${prefix}_wheel_transmission">
@@ -45,9 +47,10 @@
         </transmission>
     </xacro:macro>
-    <xacro:macro name="caster_wheel" params="radius mass position_x position_z">
+    <xacro:macro name="caster_wheel" params="radius mass x z">
         <link name="caster_wheel_link">
             <visual>
                 <geometry>
-                    <mesh filename="package://leobot_description/meshes/wheel-2-with-ball.stl" scale="0.001 0.001 0.001"/>
+                    <mesh filename="package://leobot_description/meshes/wheel-2-with-ball.stl"
+                          scale="0.001 0.001 0.001"/>
                     <xacro:red_material/>
                 </geometry>
@@ -57,7 +60,7 @@
         </link>
         <joint name="caster_wheel_base_joint" type="fixed">
-            <parent link="base_link"/>
+            <parent link="chassis"/>
             <child link="caster_wheel_link"/>
-            <origin rpy="0 0 0" xyz="${position_x} 0.0 ${position_z}"/>
+            <origin rpy="0 0 0" xyz="${x} 0.0 ${z}"/>
         </joint>
     </xacro:macro>

Commit message: Added LIDAR to new robot URDF

File: leobot_description/robot/robot.urdf.xacro (robot description, xacro)
@@ -3,4 +3,5 @@
   <xacro:include filename="$(find leobot_description)/urdf/materials.urdf.xacro"/>
   <xacro:include filename="$(find leobot_description)/urdf/common.urdf.xacro"/>
+  <xacro:include filename="$(find leobot_description)/urdf/sensors/hokuyo.urdf.xacro"/>
   <xacro:include filename="$(find leobot_description)/urdf/wheels.urdf.xacro"/>
   <xacro:property name="base_width" value="0.7"/>
@@ -58,4 +59,5 @@
                         width="${wheel_width}" mass="${wheel_mass}" distance_between_wheels="${distance_between_wheels}"
                         x="${wheel_position_x}" z="${wheel_position_z}"/>
+  <xacro:lidar_hokuyo parent_link_name="chassis"/>
   <link name="tower_link">
     <visual>

File: leobot_description/urdf/sensors/hokuyo.urdf.xacro (robot description, xacro)
@@ -1,21 +1,21 @@
 <?xml version="1.0"?>
-    <robot xmlns:xacro="http://ros.org/wiki/xacro">
-        <xacro:property name="hokuyo_width" value="0.001"/>
-        <xacro:property name="hokuyo_height" value="0.05"/>
-        <xacro:property name="hokuyo_depth" value="0.06"/>
-        <xacro:macro name="lidar_hokuyo" params="base_radius base_height">
-            <link name="laser_link">
-              <visual>
-                  <xacro:box_geometry width="${hokuyo_width}" height="${hokuyo_height}" depth="${hokuyo_depth}"/>
-                  <xacro:green_material/>
-              </visual>
-              <xacro:box_collision width="${hokuyo_width}" height="${hokuyo_height}" depth="${hokuyo_depth}"/>
-              <xacro:box_inertia mass="0.001" width="${hokuyo_width}" height="${hokuyo_height}" depth="${hokuyo_depth}"/>
-            </link>
-            <joint name="laser_base_joint" type="fixed">
-              <origin xyz="${(base_radius - 0.0001)} 0.0 ${-base_height/2 + 0.01}" rpy="0.0 0.0 0.0" />
-              <parent link="base_link" />
-              <child link="laser_link" />
-            </joint>
-        </xacro:macro>
-    </robot>
+<robot xmlns:xacro="http://ros.org/wiki/xacro">
+    <xacro:property name="hokuyo_width" value="0.001"/>
+    <xacro:property name="hokuyo_height" value="0.05"/>
+    <xacro:property name="hokuyo_depth" value="0.06"/>
+    <xacro:macro name="lidar_hokuyo" params="parent_link_name">
+        <link name="laser_link">
+            <visual>
+                <xacro:box_geometry width="${hokuyo_width}" height="${hokuyo_height}" depth="${hokuyo_depth}"/>
+                <xacro:green_material/>
+            </visual>
+            <xacro:box_collision width="${hokuyo_width}" height="${hokuyo_height}" depth="${hokuyo_depth}"/>
+            <xacro:box_inertia mass="0.001" width="${hokuyo_width}" height="${hokuyo_height}" depth="${hokuyo_depth}"/>
+        </link>
+        <joint name="laser_base_joint" type="fixed">
+            <origin xyz="0 0 ${hokuyo_height}" rpy="0 0 0"/>
+            <parent link="${parent_link_name}" />
+            <child link="laser_link" />
+        </joint>
+    </xacro:macro>
+</robot>
