Commit message: Adding CAD Models Accidentally adding lots of errors to the design

File: leobot_description/robot/robot.urdf.xacro (robot description, xacro)
@@ -5,4 +5,5 @@
   <xacro:include filename="$(find leobot_description)/urdf/sensors/hokuyo.urdf.xacro"/>
   <xacro:include filename="$(find leobot_description)/urdf/wheels.urdf.xacro"/>
+   <xacro:property name="base_radius" value="0.25"/>
   <xacro:property name="base_width" value="0.7"/>
   <xacro:property name="base_length" value="1.132"/>
@@ -22,47 +23,17 @@
   <xacro:property name="caster_wheel_position_z" value="-0.04"/>
   <xacro:property name="bearing_radius" value="0.01"/>
-  <link name="base_link"/>
-  <link name="chassis">
+ <link name="base_link">
     <visual>
-      <geometry>
-        <mesh filename="package://leobot_description/meshes/base.stl" scale="0.001 0.001 0.001"/>
-      </geometry>
+      <xacro:box_geometry width="1" height="1" depth="1"/>
       <xacro:navajo_white_material/>
     </visual>
-  </link>
-  <joint name="base_link_joint" type="fixed">
-    <origin xyz="0 0 0.05" rpy="0 0 0" />
-    <parent link="base_link" />
-    <child link="chassis" />
-  </joint>
-  <link name="chassis_inertia">
-    <collision>
-      <origin xyz="${-base_length/2} 0 ${base_height/2 - safety_width}" rpy="0 0 0"/>
-      <geometry>
-        <box size="${base_length + safety_width} ${base_width + safety_width} ${base_height + safety_width}"/>
-      </geometry>
-    </collision>
-    <xacro:box_inertia mass="10.0" width="${base_width}" depth="${base_length}" height="${base_height}"
-                       x="${-base_length/2}" z="${base_height/2}"/>
-  </link>
-  <joint name="chassis_inertia_joint" type="fixed">
-    <origin xyz="0 0 0" rpy="0 0 0" />
-    <parent link="chassis" />
-    <child link="chassis_inertia" />
-  </joint>
-  <xacro:caster_wheel radius="${caster_radius}" mass="${caster_mass}" x="${caster_wheel_position_x}"
-                      z="${caster_wheel_position_z}"/>
-  <xacro:standard_wheel prefix="left" direction="1.0" bearing_radius="${bearing_radius}" radius="${wheel_radius}"
-                        width="${wheel_width}" mass="${wheel_mass}" distance_between_wheels="${distance_between_wheels}"
-                        x="${wheel_position_x}" z="${wheel_position_z}"/>
-  <xacro:standard_wheel prefix="right" direction="-1.0" bearing_radius="${bearing_radius}" radius="${wheel_radius}"
-                        width="${wheel_width}" mass="${wheel_mass}" distance_between_wheels="${distance_between_wheels}"
-                        x="${wheel_position_x}" z="${wheel_position_z}"/>
-  <xacro:lidar_hokuyo parent_link_name="chassis"/>
-  <link name="tower_link">
+    <xacro:box_collision width="1" height="1" depth="1"/>
+    <xacro:box_inertia mass="10" width="1" height="1" depth="1"/>
+</link>
+  <link name="wheel_FR">
     <visual>
       <origin xyz="0 0 0" rpy="0 0 0"/>
       <geometry>
-        <mesh filename="package://leobot_description/meshes/tower.stl" scale="0.001 0.001 0.001"/>
+        <mesh filename="package://leobot_description/meshes/Mecanum_Wheel_01.STL" scale="1 1 1"/>
       </geometry>
       <xacro:navajo_white_material/>
@@ -71,46 +42,77 @@
       <origin xyz="${-base_length/2} 0 ${base_height + tower_height/2} " rpy="0 0 0"/>
       <geometry>
-        <box size="${base_length + safety_width} ${base_width + safety_width} ${tower_height + safety_width}"/>
+        <cylinder length="${base_height}" radius="${base_radius}"/>
       </geometry>
     </collision>
-    <xacro:box_inertia mass="3.0" width="${base_width}" depth="${base_length}" height="${tower_height}"/>
+    <xacro:cylinder_inertia mass="10" radius="${base_radius}" height="${base_height}"/>
   </link>
-  <joint name="tower_link_joint" type="fixed">
-    <origin xyz="0 0 0" rpy="0 0 0"/>
-    <parent link="chassis"/>
-    <child link="tower_link"/>
-  </joint>
-  <link name="head_link">
+    <link name="wheel_FL">
     <visual>
-      <origin xyz="0.75 0 -${base_height+tower_height+head_height/2}" rpy="0 0 0"/>
+      <origin xyz="0 0 0" rpy="0 0 0"/>
       <geometry>
-        <mesh filename="package://leobot_description/meshes/head.stl" scale="0.001 0.001 0.001"/>
+        <mesh filename="package://leobot_description/meshes/Mecanum_Wheel_01.STL" scale="1 1 1"/>
       </geometry>
       <xacro:navajo_white_material/>
     </visual>
     <collision>
+      <origin xyz="${-base_length/2} 0 ${base_height + tower_height/2} " rpy="0 0 0"/>
       <geometry>
-        <cylinder length="${head_height*2}" radius="${base_width/2}"/>
+        <cylinder length="${base_height}" radius="${base_radius}"/>
       </geometry>
     </collision>
-    <xacro:cylinder_inertia mass="1" radius="${base_width/2}" height="${head_height*2}"/>
+    <xacro:cylinder_inertia mass="10" radius="${base_radius}" height="${base_height}"/>
   </link>
-  <joint name="head_link_joint" type="revolute">
-    <origin rpy="0 0 0" xyz="-0.75 0 ${base_height+tower_height+head_height/2}"/>
-    <axis xyz="0 0 1" />
-    <parent link="tower_link"/>
-    <child link="head_link"/>
-    <limit effort="10" velocity="10" lower="${-pi/2}" upper="${pi/2}" />
+    <link name="wheel_RL">
+    <visual>
+      <origin xyz="0 0 0" rpy="0 0 0"/>
+      <geometry>
+        <mesh filename="package://leobot_description/meshes/Mecanum_Wheel_02.STL" scale="1 1 1"/>
+      </geometry>
+      <xacro:navajo_white_material/>
+    </visual>
+    <collision>
+      <origin xyz="${-base_length/2} 0 ${base_height + tower_height/2} " rpy="0 0 0"/>
+      <geometry>
+        <cylinder length="${base_height}" radius="${base_radius}"/>
+      </geometry>
+    </collision>
+    <xacro:cylinder_inertia mass="10" radius="${base_radius}" height="${base_height}"/>
+  </link>
+    <link name="wheel_RR">
+    <visual>
+      <origin xyz="0 0 0" rpy="0 0 0"/>
+      <geometry>
+        <mesh filename="package://leobot_description/meshes/Mecanum_Wheel_02.STL" scale="1 1 1"/>
+      </geometry>
+      <xacro:navajo_white_material/>
+    </visual>
+    <collision>
+      <origin xyz="${-base_length/2} 0 ${base_height + tower_height/2} " rpy="0 0 0"/>
+      <geometry>
+        <cylinder length="${base_height}" radius="${base_radius}"/>
+      </geometry>
+    </collision>
+    <xacro:cylinder_inertia mass="10" radius="${base_radius}" height="${base_height}"/>
+  </link>
+  <joint name="base_link_wheel_FR_joint" type="continuous">
+    <origin xyz="0 0 0.05" rpy="0 0 0" />
+    <parent link="base_link" />
+    <child link="wheel_FL" />
   </joint>
-  <transmission name="head_transmission">
-    <type>transmission_interface/SimpleTransmission</type>
-    <joint name="head_link_joint">
-      <hardwareInterface>hardware_interface/EffortJointInterface</hardwareInterface>
-    </joint>
-    <actuator name="head_motor">
-      <hardwareInterface>EffortJointInterface</hardwareInterface>
-      <mechanicalReduction>1</mechanicalReduction>
-    </actuator>
-  </transmission>
+  <joint name="base_link_joint_wheel_FL_joint" type="continuous">
+    <origin xyz="0 0 0.05" rpy="0 0 0" />
+    <parent link="base_link" />
+    <child link="wheel_FR" />
+  </joint>
+  <joint name="base_link_joint_wheel_RL_joint" type="continuous">
+    <origin xyz="0 0 0" rpy="0 0 0" />
+    <parent link="base_link" />
+    <child link="wheel_RL" />
+  </joint>
+  <joint name="base_link_joint_wheel_RR_joint" type="continuous">
+    <origin xyz="0 0 0" rpy="0 0 0" />
+    <parent link="base_link" />
+    <child link="wheel_RR" />
+  </joint>
   <link name="camera_left_link">
     <visual>
@@ -123,5 +125,5 @@
   <joint name="camera_left_link_joint" type="fixed">
     <origin rpy="0 0 0" xyz="0 0.075 0.075"/>
-    <parent link="head_link"/>
+    <parent link="base_link"/>
     <child link="camera_left_link"/>
   </joint>
@@ -136,5 +138,5 @@
   <joint name="camera_right_link_joint" type="fixed">
     <origin rpy="0 0 0" xyz="0 -0.075 0.075"/>
-    <parent link="head_link"/>
+    <parent link="base_link"/>
     <child link="camera_right_link"/>
   </joint>

Commit message: Indent and clean up the XML markup

File: leobot_description/robot/robot.urdf.xacro (robot description, xacro)
@@ -1,3 +1,2 @@
-<?xml version="1.0"?>
 <robot name="leobot" xmlns:xacro="http://ros.org/wiki/xacro">
   <xacro:include filename="$(find leobot_description)/urdf/materials.urdf.xacro"/>
@@ -5,5 +4,5 @@
   <xacro:include filename="$(find leobot_description)/urdf/sensors/hokuyo.urdf.xacro"/>
   <xacro:include filename="$(find leobot_description)/urdf/wheels.urdf.xacro"/>
-   <xacro:property name="base_radius" value="0.25"/>
+  <xacro:property name="base_radius" value="0.25"/>
   <xacro:property name="base_width" value="0.7"/>
   <xacro:property name="base_length" value="1.132"/>
@@ -23,5 +22,5 @@
   <xacro:property name="caster_wheel_position_z" value="-0.04"/>
   <xacro:property name="bearing_radius" value="0.01"/>
- <link name="base_link">
+  <link name="base_link">
     <visual>
       <xacro:box_geometry width="1" height="1" depth="1"/>
@@ -30,5 +29,5 @@
     <xacro:box_collision width="1" height="1" depth="1"/>
     <xacro:box_inertia mass="10" width="1" height="1" depth="1"/>
-</link>
+  </link>
   <link name="wheel_FR">
     <visual>
@@ -47,5 +46,5 @@
     <xacro:cylinder_inertia mass="10" radius="${base_radius}" height="${base_height}"/>
   </link>
-    <link name="wheel_FL">
+  <link name="wheel_FL">
     <visual>
       <origin xyz="0 0 0" rpy="0 0 0"/>
@@ -63,5 +62,5 @@
     <xacro:cylinder_inertia mass="10" radius="${base_radius}" height="${base_height}"/>
   </link>
-    <link name="wheel_RL">
+  <link name="wheel_RL">
     <visual>
       <origin xyz="0 0 0" rpy="0 0 0"/>
@@ -79,5 +78,5 @@
     <xacro:cylinder_inertia mass="10" radius="${base_radius}" height="${base_height}"/>
   </link>
-    <link name="wheel_RR">
+  <link name="wheel_RR">
     <visual>
       <origin xyz="0 0 0" rpy="0 0 0"/>

Commit message: Comment out the unused properties

File: leobot_description/robot/robot.urdf.xacro (robot description, xacro)
@@ -5,20 +5,20 @@
   <!--<xacro:include filename="$(find leobot_description)/urdf/wheels.urdf.xacro"/>-->
   <xacro:property name="base_radius" value="0.25"/>
-  <xacro:property name="base_width" value="0.7"/>
+  <!--<xacro:property name="base_width" value="0.7"/>-->
   <xacro:property name="base_length" value="1.132"/>
   <xacro:property name="base_height" value="0.4"/>
-  <xacro:property name="safety_width" value="0.03"/>
-  <xacro:property name="distance_between_wheels" value="0.55"/>
+  <!--<xacro:property name="safety_width" value="0.03"/>-->
+  <!--<xacro:property name="distance_between_wheels" value="0.55"/>-->
   <xacro:property name="tower_height" value="1.125"/>
-  <xacro:property name="head_height" value="0.1"/>
-  <xacro:property name="caster_radius" value="0.05"/>
-  <xacro:property name="caster_mass" value="10"/>
-  <xacro:property name="wheel_width" value="0.035"/>
-  <xacro:property name="wheel_radius" value="0.1"/>
-  <xacro:property name="wheel_mass" value="10"/>
-  <xacro:property name="wheel_position_x" value="-0.35"/>
-  <xacro:property name="wheel_position_z" value="0.02"/>
-  <xacro:property name="caster_wheel_position_x" value="-1.0"/>
-  <xacro:property name="caster_wheel_position_z" value="-0.04"/>
+  <!--<xacro:property name="head_height" value="0.1"/>-->
+  <!--<xacro:property name="caster_radius" value="0.05"/>-->
+  <!--<xacro:property name="caster_mass" value="10"/>-->
+  <!--<xacro:property name="wheel_width" value="0.035"/>-->
+  <!--<xacro:property name="wheel_radius" value="0.1"/>-->
+  <!--<xacro:property name="wheel_mass" value="10"/>-->
+  <!--<xacro:property name="wheel_position_x" value="-0.35"/>-->
+  <!--<xacro:property name="wheel_position_z" value="0.02"/>-->
+  <!--<xacro:property name="caster_wheel_position_x" value="-1.0"/>-->
+  <!--<xacro:property name="caster_wheel_position_z" value="-0.04"/>-->
   <xacro:property name="bearing_radius" value="0.01"/>
   <link name="base_link">

Commit message: Comment out the unused property

File: leobot_description/robot/robot.urdf.xacro (robot description, xacro)
@@ -21,5 +21,5 @@
   <!--<xacro:property name="caster_wheel_position_x" value="-1.0"/>-->
   <!--<xacro:property name="caster_wheel_position_z" value="-0.04"/>-->
-  <xacro:property name="bearing_radius" value="0.01"/>
+  <!--<xacro:property name="bearing_radius" value="0.01"/>-->
   <link name="base_link">
     <visual>

Commit message: Create macroses for mecanum wheels

File: leobot_description/robot/robot.urdf.xacro (robot description, xacro)
@@ -30,68 +30,30 @@
     <xacro:box_inertia mass="10" width="1" height="1" depth="1"/>
   </link>
-  <link name="wheel_FR">
-    <visual>
-      <origin xyz="0 0 0" rpy="0 0 0"/>
-      <geometry>
-        <mesh filename="package://leobot_description/meshes/Mecanum_Wheel_01.STL" scale="1 1 1"/>
-      </geometry>
-      <xacro:navajo_white_material/>
-    </visual>
-    <collision>
-      <origin xyz="${-base_length/2} 0 ${base_height + tower_height/2} " rpy="0 0 0"/>
-      <geometry>
-        <cylinder length="${base_height}" radius="${base_radius}"/>
-      </geometry>
-    </collision>
-    <xacro:cylinder_inertia mass="10" radius="${base_radius}" height="${base_height}"/>
-  </link>
-  <link name="wheel_FL">
-    <visual>
-      <origin xyz="0 0 0" rpy="0 0 0"/>
-      <geometry>
-        <mesh filename="package://leobot_description/meshes/Mecanum_Wheel_01.STL" scale="1 1 1"/>
-      </geometry>
-      <xacro:navajo_white_material/>
-    </visual>
-    <collision>
-      <origin xyz="${-base_length/2} 0 ${base_height + tower_height/2} " rpy="0 0 0"/>
-      <geometry>
-        <cylinder length="${base_height}" radius="${base_radius}"/>
-      </geometry>
-    </collision>
-    <xacro:cylinder_inertia mass="10" radius="${base_radius}" height="${base_height}"/>
-  </link>
-  <link name="wheel_RL">
-    <visual>
-      <origin xyz="0 0 0" rpy="0 0 0"/>
-      <geometry>
-        <mesh filename="package://leobot_description/meshes/Mecanum_Wheel_02.STL" scale="1 1 1"/>
-      </geometry>
-      <xacro:navajo_white_material/>
-    </visual>
-    <collision>
-      <origin xyz="${-base_length/2} 0 ${base_height + tower_height/2} " rpy="0 0 0"/>
-      <geometry>
-        <cylinder length="${base_height}" radius="${base_radius}"/>
-      </geometry>
-    </collision>
-    <xacro:cylinder_inertia mass="10" radius="${base_radius}" height="${base_height}"/>
-  </link>
-  <link name="wheel_RR">
-    <visual>
-      <origin xyz="0 0 0" rpy="0 0 0"/>
-      <geometry>
-        <mesh filename="package://leobot_description/meshes/Mecanum_Wheel_02.STL" scale="1 1 1"/>
-      </geometry>
-      <xacro:navajo_white_material/>
-    </visual>
-    <collision>
-      <origin xyz="${-base_length/2} 0 ${base_height + tower_height/2} " rpy="0 0 0"/>
-      <geometry>
-        <cylinder length="${base_height}" radius="${base_radius}"/>
-      </geometry>
-    </collision>
-    <xacro:cylinder_inertia mass="10" radius="${base_radius}" height="${base_height}"/>
-  </link>
+  <xacro:macro name="mecanum_wheel" params="link_name mesh_file">
+    <link name="${link_name}">
+      <visual>
+        <origin xyz="0 0 0" rpy="0 0 0"/>
+        <geometry>
+          <mesh filename="${mesh_file}" scale="1 1 1"/>
+        </geometry>
+        <xacro:navajo_white_material/>
+      </visual>
+      <collision>
+        <origin xyz="${-base_length/2} 0 ${base_height + tower_height/2} " rpy="0 0 0"/>
+        <geometry>
+          <cylinder length="${base_height}" radius="${base_radius}"/>
+        </geometry>
+      </collision>
+      <xacro:cylinder_inertia mass="10" radius="${base_radius}" height="${base_height}"/>
+    </link>
+  </xacro:macro>
+  <xacro:macro name="leobot_mecanum_wheel" params="name variant">
+    <xacro:mecanum_wheel link_name="wheel_${name}"
+                         mesh_file="package://leobot_description/meshes/Mecanum_Wheel_0${variant}.STL"/>
+  </xacro:macro>
+  <xacro:leobot_mecanum_wheel name="FR" variant="1"/>
+  <xacro:leobot_mecanum_wheel name="FL" variant="1"/>
+  <xacro:leobot_mecanum_wheel name="RL" variant="2"/>
+  <xacro:leobot_mecanum_wheel name="RR" variant="2"/>
   <joint name="base_link_wheel_FR_joint" type="continuous">
     <origin xyz="0 0 0.05" rpy="0 0 0" />

Commit message: Implement approximate positioning and geometry of wheels

File: leobot_description/robot/robot.urdf.xacro (robot description, xacro)
@@ -4,16 +4,17 @@
   <!--<xacro:include filename="$(find leobot_description)/urdf/sensors/hokuyo.urdf.xacro"/>-->
   <!--<xacro:include filename="$(find leobot_description)/urdf/wheels.urdf.xacro"/>-->
-  <xacro:property name="base_radius" value="0.25"/>
-  <!--<xacro:property name="base_width" value="0.7"/>-->
-  <xacro:property name="base_length" value="1.132"/>
-  <xacro:property name="base_height" value="0.4"/>
+  <xacro:property name="pi" value="3.1416"/>
+  <!--<xacro:property name="base_radius" value="0.25"/>-->
+  <xacro:property name="base_width" value="0.5"/>
+  <xacro:property name="base_length" value="0.5"/>
+  <!--<xacro:property name="base_height" value="0.4"/>-->
   <!--<xacro:property name="safety_width" value="0.03"/>-->
   <!--<xacro:property name="distance_between_wheels" value="0.55"/>-->
-  <xacro:property name="tower_height" value="1.125"/>
+  <!--<xacro:property name="tower_height" value="1.125"/>-->
   <!--<xacro:property name="head_height" value="0.1"/>-->
   <!--<xacro:property name="caster_radius" value="0.05"/>-->
   <!--<xacro:property name="caster_mass" value="10"/>-->
-  <!--<xacro:property name="wheel_width" value="0.035"/>-->
-  <!--<xacro:property name="wheel_radius" value="0.1"/>-->
+  <xacro:property name="wheel_width" value="0.06"/>
+  <xacro:property name="wheel_radius" value="0.05"/>
   <!--<xacro:property name="wheel_mass" value="10"/>-->
   <!--<xacro:property name="wheel_position_x" value="-0.35"/>-->
@@ -30,8 +31,8 @@
     <xacro:box_inertia mass="10" width="1" height="1" depth="1"/>
   </link>
-  <xacro:macro name="mecanum_wheel" params="link_name mesh_file">
+  <xacro:macro name="mecanum_wheel" params="link_name mesh_file radius width x:=0 y:=0">
     <link name="${link_name}">
       <visual>
-        <origin xyz="0 0 0" rpy="0 0 0"/>
+        <origin xyz="${x} ${y} ${-radius}" rpy="${pi/2} 0 0"/>
         <geometry>
           <mesh filename="${mesh_file}" scale="1 1 1"/>
@@ -40,20 +41,23 @@
       </visual>
       <collision>
-        <origin xyz="${-base_length/2} 0 ${base_height + tower_height/2} " rpy="0 0 0"/>
+        <origin xyz="${x} ${y} ${-radius}" rpy="${pi/2} 0 0"/>
         <geometry>
-          <cylinder length="${base_height}" radius="${base_radius}"/>
+          <cylinder length="${width}" radius="${radius}"/>
         </geometry>
       </collision>
-      <xacro:cylinder_inertia mass="10" radius="${base_radius}" height="${base_height}"/>
+      <xacro:cylinder_inertia mass="10" radius="${radius}" height="${width}"/>
     </link>
   </xacro:macro>
-  <xacro:macro name="leobot_mecanum_wheel" params="name variant">
+  <xacro:macro name="leobot_mecanum_wheel" params="name variant origin_x origin_y">
     <xacro:mecanum_wheel link_name="wheel_${name}"
-                         mesh_file="package://leobot_description/meshes/Mecanum_Wheel_0${variant}.STL"/>
+                         mesh_file="package://leobot_description/meshes/Mecanum_Wheel_0${variant}.STL"
+                         radius="${wheel_radius}" width="${wheel_width}"
+                         x="${origin_x * base_width/2}"
+                         y="${origin_y * base_length/2}"/>
   </xacro:macro>
-  <xacro:leobot_mecanum_wheel name="FR" variant="1"/>
-  <xacro:leobot_mecanum_wheel name="FL" variant="1"/>
-  <xacro:leobot_mecanum_wheel name="RL" variant="2"/>
-  <xacro:leobot_mecanum_wheel name="RR" variant="2"/>
+  <xacro:leobot_mecanum_wheel name="FR" variant="1" origin_x="1"  origin_y="1"/>
+  <xacro:leobot_mecanum_wheel name="FL" variant="1" origin_x="-1" origin_y="1"/>
+  <xacro:leobot_mecanum_wheel name="RL" variant="2" origin_x="1"  origin_y="-1"/>
+  <xacro:leobot_mecanum_wheel name="RR" variant="2" origin_x="-1" origin_y="-1"/>
   <joint name="base_link_wheel_FR_joint" type="continuous">
     <origin xyz="0 0 0.05" rpy="0 0 0" />

Commit message: Adjust the size of the base

File: leobot_description/robot/robot.urdf.xacro (robot description, xacro)
@@ -8,6 +8,7 @@
   <xacro:property name="base_width" value="0.5"/>
   <xacro:property name="base_length" value="0.5"/>
-  <!--<xacro:property name="base_height" value="0.4"/>-->
+  <xacro:property name="base_height" value="0.3"/>
   <!--<xacro:property name="safety_width" value="0.03"/>-->
+  <xacro:property name="base_mass" value="10"/>
   <!--<xacro:property name="distance_between_wheels" value="0.55"/>-->
   <!--<xacro:property name="tower_height" value="1.125"/>-->
@@ -25,9 +26,9 @@
   <link name="base_link">
     <visual>
-      <xacro:box_geometry width="1" height="1" depth="1"/>
+      <xacro:box_geometry width="${base_width}" height="${base_length}" depth="${base_height}"/>
       <xacro:navajo_white_material/>
     </visual>
-    <xacro:box_collision width="1" height="1" depth="1"/>
-    <xacro:box_inertia mass="10" width="1" height="1" depth="1"/>
+    <xacro:box_collision width="${base_width}" height="${base_length}" depth="${base_height}"/>
+    <xacro:box_inertia   width="${base_width}" height="${base_length}" depth="${base_height}" mass="${base_mass}"/>
   </link>
   <xacro:macro name="mecanum_wheel" params="link_name mesh_file radius width x:=0 y:=0">
