Commit message: Elevate the robot base above wheels, refactor generation of boxes, optimize the positioning

File: leobot_description/robot/robot.urdf.xacro (robot description, xacro)
@@ -24,16 +24,24 @@
   <!--<xacro:property name="caster_wheel_position_z" value="-0.04"/>-->
   <!--<xacro:property name="bearing_radius" value="0.01"/>-->
-  <link name="base_link">
-    <visual>
-      <xacro:box_geometry width="${base_width}" height="${base_length}" depth="${base_height}"/>
-      <xacro:navajo_white_material/>
-    </visual>
-    <xacro:box_collision width="${base_width}" height="${base_length}" depth="${base_height}"/>
-    <xacro:box_inertia   width="${base_width}" height="${base_length}" depth="${base_height}" mass="${base_mass}"/>
-  </link>
-  <xacro:macro name="mecanum_wheel" params="link_name mesh_file radius width x:=0 y:=0">
+  <xacro:macro name="leobot_base" params="*origin">
+    <link name="base_link">
+      <visual>
+        <xacro:insert_block name="origin"/>
+        <xacro:box_geometry width="${base_width}" height="${base_length}" depth="${base_height}"/>
+        <xacro:navajo_white_material/>
+      </visual>
+      <xacro:box_collision width="${base_width}" height="${base_length}" depth="${base_height}">
+        <xacro:insert_block name="origin"/>
+      </xacro:box_collision>
+      <xacro:box_inertia width="${base_width}" height="${base_length}" depth="${base_height}" mass="${base_mass}"/>
+    </link>
+  </xacro:macro>
+  <xacro:leobot_base>
+    <origin xyz="0 0 ${base_height/2 + wheel_radius}"/>
+  </xacro:leobot_base>
+  <xacro:macro name="mecanum_wheel" params="link_name mesh_file radius width *origin">
     <link name="${link_name}">
       <visual>
-        <origin xyz="${x} ${y} ${-radius}" rpy="${pi/2} 0 0"/>
+        <xacro:insert_block name="origin"/>
         <geometry>
           <mesh filename="${mesh_file}" scale="1 1 1"/>
@@ -42,5 +50,5 @@
       </visual>
       <collision>
-        <origin xyz="${x} ${y} ${-radius}" rpy="${pi/2} 0 0"/>
+        <xacro:insert_block name="origin"/>
         <geometry>
           <cylinder length="${width}" radius="${radius}"/>
@@ -53,12 +61,13 @@
     <xacro:mecanum_wheel link_name="wheel_${name}"
                          mesh_file="package://leobot_description/meshes/Mecanum_Wheel_0${variant}.STL"
-                         radius="${wheel_radius}" width="${wheel_width}"
-                         x="${origin_x * base_width/2}"
-                         y="${origin_y * base_length/2}"/>
+                         radius="${wheel_radius}" width="${wheel_width}">
+      <origin xyz="${origin_x * base_width/2} ${origin_y * base_length/2}"
+              rpy="${pi/2} 0 0"/>
+    </xacro:mecanum_wheel>
   </xacro:macro>
   <xacro:leobot_mecanum_wheel name="FR" variant="1" origin_x="1"  origin_y="1"/>
   <xacro:leobot_mecanum_wheel name="FL" variant="1" origin_x="-1" origin_y="1"/>
-  <xacro:leobot_mecanum_wheel name="RL" variant="2" origin_x="1"  origin_y="-1"/>
-  <xacro:leobot_mecanum_wheel name="RR" variant="2" origin_x="-1" origin_y="-1"/>
+  <xacro:leobot_mecanum_wheel name="RL" variant="2" origin_x="-1" origin_y="-1"/>
+  <xacro:leobot_mecanum_wheel name="RR" variant="2" origin_x="1"  origin_y="-1"/>
   <joint name="base_link_wheel_FR_joint" type="continuous">
     <origin xyz="0 0 0.05" rpy="0 0 0" />
@@ -86,5 +95,7 @@
       <xacro:green_material/>
     </visual>
-    <xacro:box_collision width="0.05" height="0.05" depth="0.05"/>
+    <xacro:box_collision width="0.05" height="0.05" depth="0.05">
+      <origin/>
+    </xacro:box_collision>
     <xacro:box_inertia mass="0.1" width="0.05" height="0.05" depth="0.05"/>
   </link>
@@ -99,5 +110,7 @@
       <xacro:green_material/>
     </visual>
-    <xacro:box_collision width="0.05" height="0.05" depth="0.05"/>
+    <xacro:box_collision width="0.05" height="0.05" depth="0.05">
+      <origin/>
+    </xacro:box_collision>
     <xacro:box_inertia mass="0.1" width="0.05" height="0.05" depth="0.05"/>
   </link>

File: leobot_description/urdf/common.urdf.xacro (robot description, xacro)
@@ -73,6 +73,7 @@
     </geometry>
   </xacro:macro>
-  <xacro:macro name="box_collision" params="width height depth">
+  <xacro:macro name="box_collision" params="width height depth *origin">
     <collision>
+      <xacro:insert_block name="origin"/>
       <xacro:box_geometry width="${width}" height="${height}" depth="${depth}"/>
     </collision>

Commit message: Added base link Added neck Added head Added cameras Added LIDAR Initial preparation for adding the wheels and motors

File: leobot_description/robot/robot.urdf.xacro (robot description, xacro)
@@ -2,43 +2,58 @@
   <xacro:include filename="$(find leobot_description)/urdf/materials.urdf.xacro"/>
   <xacro:include filename="$(find leobot_description)/urdf/common.urdf.xacro"/>
-  <!--<xacro:include filename="$(find leobot_description)/urdf/sensors/hokuyo.urdf.xacro"/>-->
-  <!--<xacro:include filename="$(find leobot_description)/urdf/wheels.urdf.xacro"/>-->
-  <xacro:property name="pi" value="3.1416"/>
-  <!--<xacro:property name="base_radius" value="0.25"/>-->
+  <xacro:include filename="$(find leobot_description)/urdf/sensors/camera.urdf.xacro"/>
+  <xacro:include filename="$(find leobot_description)/urdf/sensors/hokuyo.urdf.xacro"/>
+  <xacro:include filename="$(find leobot_description)/urdf/wheels.urdf.xacro"/>
   <xacro:property name="base_width" value="0.5"/>
-  <xacro:property name="base_length" value="0.5"/>
-  <xacro:property name="base_height" value="0.3"/>
-  <!--<xacro:property name="safety_width" value="0.03"/>-->
+  <xacro:property name="base_length" value="0.3"/>
+  <xacro:property name="base_height" value="0.54"/>
   <xacro:property name="base_mass" value="10"/>
-  <!--<xacro:property name="distance_between_wheels" value="0.55"/>-->
-  <!--<xacro:property name="tower_height" value="1.125"/>-->
-  <!--<xacro:property name="head_height" value="0.1"/>-->
-  <!--<xacro:property name="caster_radius" value="0.05"/>-->
-  <!--<xacro:property name="caster_mass" value="10"/>-->
-  <xacro:property name="wheel_width" value="0.06"/>
-  <xacro:property name="wheel_radius" value="0.05"/>
-  <!--<xacro:property name="wheel_mass" value="10"/>-->
-  <!--<xacro:property name="wheel_position_x" value="-0.35"/>-->
-  <!--<xacro:property name="wheel_position_z" value="0.02"/>-->
-  <!--<xacro:property name="caster_wheel_position_x" value="-1.0"/>-->
-  <!--<xacro:property name="caster_wheel_position_z" value="-0.04"/>-->
-  <!--<xacro:property name="bearing_radius" value="0.01"/>-->
-  <xacro:macro name="leobot_base" params="*origin">
-    <link name="base_link">
-      <visual>
-        <xacro:insert_block name="origin"/>
-        <xacro:box_geometry width="${base_width}" height="${base_length}" depth="${base_height}"/>
-        <xacro:navajo_white_material/>
-      </visual>
-      <xacro:box_collision width="${base_width}" height="${base_length}" depth="${base_height}">
-        <xacro:insert_block name="origin"/>
-      </xacro:box_collision>
-      <xacro:box_inertia width="${base_width}" height="${base_length}" depth="${base_height}" mass="${base_mass}"/>
-    </link>
-  </xacro:macro>
-  <xacro:leobot_base>
-    <origin xyz="0 0 ${base_height/2 + wheel_radius}"/>
-  </xacro:leobot_base>
-  <xacro:macro name="mecanum_wheel" params="link_name mesh_file radius width *origin">
+  <xacro:property name="neck_width" value="0.04"/>
+  <xacro:property name="neck_length" value="0.04"/>
+  <xacro:property name="neck_height" value="1.45"/>
+  <xacro:property name="neck_mass" value="1.0"/>
+  <xacro:property name="head_width" value="0.04"/>
+  <xacro:property name="head_length" value="0.04"/>
+  <xacro:property name="head_height" value="0.29"/>
+  <xacro:property name="head_mass" value="0.5"/>
+  <link name="base_link">
+    <visual>
+      <xacro:box_geometry width="${base_width}" height="${base_height}" depth="${base_length}"/>
+      <xacro:green_material/>
+    </visual>
+    <xacro:box_collision width="${base_width}" height="${base_height}" depth="${base_length}"/>
+    <xacro:box_inertia width="${base_width}" height="${base_height}" depth="${base_length}" mass="${base_mass}"/>
+  </link>
+  <link name="neck_link">
+    <visual>
+      <xacro:box_geometry width="${neck_width}" height="${neck_height}" depth="${neck_length}"/>
+      <xacro:red_material/>
+    </visual>
+    <xacro:box_collision width="${neck_width}" height="${neck_height}" depth="${neck_length}"/>
+    <xacro:box_inertia width="${neck_width}" height="${neck_height}" depth="${neck_length}" mass="${head_mass}"/>
+  </link>
+  <joint name="base_neck_joint" type="fixed">
+    <origin rpy="${pi/2} 0  0" xyz="0 ${-base_width/2 - neck_width} ${-base_length/2 + neck_height / 2 }"/>
+    <parent link="base_link"/>
+    <child link="neck_link"/>
+  </joint>
+  <link name="head_link">
+    <visual>
+      <xacro:box_geometry width="${head_width}" height="${head_height}" depth="${head_length}"/>
+      <xacro:blue_material/>
+    </visual>
+    <xacro:box_collision width="${head_width}" height="${head_height}" depth="${head_length}"/>
+    <xacro:box_inertia width="${head_width}" height="${head_height}" depth="${head_length}" mass="${head_mass}"/>
+  </link>
+  <joint name="neck_head_joint" type="fixed">
+    <origin rpy="${pi/2} 0  0" xyz="0 ${neck_height/2 + head_width/2} ${neck_length/2 - head_height/2}"/>
+    <parent link="neck_link"/>
+    <child link="head_link"/>
+  </joint>
+  <xacro:fish_camera prefix = "left" parent_link_name="head_link" parent_height="${head_height}" parent_width = "${head_width}" side="1"/>
+  <xacro:fish_camera prefix = "right" parent_link_name="head_link" parent_height="${head_height}"  parent_width = "${head_width}" side="-1"/>
+  <xacro:lidar_hokuyo parent_link_name="base_link" parent_height="${base_length}"/>
+  <xacro:mecanum_wheel prefix="FR" wheel_type="1" side="1" position="1" parent_length="${base_width}" parent_height="${base_height}" parent_width="${base_length}"/>
+<!--  <xacro:macro name="mecanum_wheel" params="link_name mesh_file radius width *origin">
     <link name="${link_name}">
       <visual>
@@ -57,6 +72,6 @@
       <xacro:cylinder_inertia mass="10" radius="${radius}" height="${width}"/>
     </link>
-  </xacro:macro>
-  <xacro:macro name="leobot_mecanum_wheel" params="name variant origin_x origin_y">
+  </xacro:macro>-->
+  <!--<xacro:macro name="leobot_mecanum_wheel" params="name variant origin_x origin_y">
     <xacro:mecanum_wheel link_name="wheel_${name}"
                          mesh_file="package://leobot_description/meshes/Mecanum_Wheel_0${variant}.STL"
@@ -90,33 +105,4 @@
     <child link="wheel_RR" />
   </joint>
-  <link name="camera_left_link">
-    <visual>
-      <xacro:box_geometry width="0.05" height="0.05" depth="0.05"/>
-      <xacro:green_material/>
-    </visual>
-    <xacro:box_collision width="0.05" height="0.05" depth="0.05">
-      <origin/>
-    </xacro:box_collision>
-    <xacro:box_inertia mass="0.1" width="0.05" height="0.05" depth="0.05"/>
-  </link>
-  <joint name="camera_left_link_joint" type="fixed">
-    <origin rpy="0 0 0" xyz="0 0.075 0.075"/>
-    <parent link="base_link"/>
-    <child link="camera_left_link"/>
-  </joint>
-  <link name="camera_right_link">
-    <visual>
-      <xacro:box_geometry width="0.05" height="0.05" depth="0.05"/>
-      <xacro:green_material/>
-    </visual>
-    <xacro:box_collision width="0.05" height="0.05" depth="0.05">
-      <origin/>
-    </xacro:box_collision>
-    <xacro:box_inertia mass="0.1" width="0.05" height="0.05" depth="0.05"/>
-  </link>
-  <joint name="camera_right_link_joint" type="fixed">
-    <origin rpy="0 0 0" xyz="0 -0.075 0.075"/>
-    <parent link="base_link"/>
-    <child link="camera_right_link"/>
-  </joint>
+-->
 </robot>

File: leobot_description/urdf/common.urdf.xacro (robot description, xacro)
@@ -73,7 +73,6 @@
     </geometry>
   </xacro:macro>
-  <xacro:macro name="box_collision" params="width height depth *origin">
+  <xacro:macro name="box_collision" params="width height depth">
     <collision>
-      <xacro:insert_block name="origin"/>
       <xacro:box_geometry width="${width}" height="${height}" depth="${depth}"/>
     </collision>

File: leobot_description/urdf/sensors/hokuyo.urdf.xacro (robot description, xacro)
@@ -1,18 +1,18 @@
 <?xml version="1.0"?>
 <robot xmlns:xacro="http://ros.org/wiki/xacro">
-    <xacro:property name="hokuyo_width" value="0.001"/>
+    <xacro:property name="hokuyo_radius" value="0.05"/>
     <xacro:property name="hokuyo_height" value="0.05"/>
-    <xacro:property name="hokuyo_depth" value="0.06"/>
-    <xacro:macro name="lidar_hokuyo" params="parent_link_name">
+    <xacro:property name="hokuyo_mass" value="0.2"/>
+    <xacro:macro name="lidar_hokuyo" params="parent_link_name parent_height">
         <link name="laser_link">
             <visual>
-                <xacro:box_geometry width="${hokuyo_width}" height="${hokuyo_height}" depth="${hokuyo_depth}"/>
-                <xacro:green_material/>
+                <xacro:cylinder_geometry height="${hokuyo_height}" radius="${hokuyo_radius}"/>
+                <xacro:navajo_white_material/>
             </visual>
-            <xacro:box_collision width="${hokuyo_width}" height="${hokuyo_height}" depth="${hokuyo_depth}"/>
-            <xacro:box_inertia mass="0.001" width="${hokuyo_width}" height="${hokuyo_height}" depth="${hokuyo_depth}"/>
+            <xacro:cylinder_collision height="${hokuyo_height}" radius="${hokuyo_radius}"/>
+            <xacro:cylinder_inertia mass="${hokuyo_mass}" height="${hokuyo_height}" radius="${hokuyo_radius}"/>
         </link>
         <joint name="laser_base_joint" type="fixed">
-            <origin xyz="0 0 ${hokuyo_height}" rpy="0 0 0"/>
+            <origin xyz="0 0 ${hokuyo_height/2 + parent_height/2}" rpy="0 0 0"/>
             <parent link="${parent_link_name}" />
             <child link="laser_link" />

File: leobot_description/urdf/wheels.urdf.xacro (robot description, xacro)
@@ -1,35 +1,39 @@
 <?xml version="1.0"?>
 <robot xmlns:xacro="http://ros.org/wiki/xacro">
-    <xacro:macro name="standard_wheel"
-                 params="prefix direction bearing_radius radius width mass distance_between_wheels x z">
-        <link name="${prefix}_bearing_link">>
+    <xacro:property name="motor_holder_radius" value="0.02"/>
+    <xacro:property name="motor_holder_height" value="0.1"/>
+    <xacro:property name="motor_holder_mass" value="0.8"/>
+    <xacro:property name="mecanum_radius" value="0.1"/>
+    <xacro:property name="mecanum_height" value="0.05"/>
+    <xacro:property name="mecanum_mass" value="0.3"/>
+    <xacro:macro name="mecanum_wheel"
+                 params="prefix wheel_type side position parent_length parent_height parent_width">
+        <link name="${prefix}_motor_holder">>
             <visual>
-                <xacro:cylinder_geometry radius="${bearing_radius}" height="${2 * wheel_width}"/>
+                <xacro:cylinder_geometry radius="${motor_holder_radius}" height="${motor_holder_height}"/>
                 <xacro:blue_material/>
             </visual>
-            <xacro:cylinder_collision radius="${bearing_radius}" height="${2 * wheel_width}"/>
-            <xacro:cylinder_inertia mass="0.01" radius="${bearing_radius}" height="${2 * wheel_width}"/>
+            <xacro:cylinder_collision radius="${motor_holder_radius}" height="${motor_holder_height}"/>
+            <xacro:cylinder_inertia mass="${motor_holder_mass}" radius="${motor_holder_radius}" height="${motor_holder_height}"/>
         </link>
-        <joint name="${prefix}_bearing_base_joint" type="fixed">
-            <origin rpy="${-pi / 2} 0 0"
-                    xyz="${x} ${direction * (distance_between_wheels/2 + wheel_width)} ${z}"/>
-            <parent link="chassis"/>
-            <child link="${prefix}_bearing_link"/>
+        <joint name="${prefix}_motor_holder_base_joint" type="fixed">
+            <origin rpy="${pi/2} 0 0"
+                    xyz="${position * (parent_width/2 - motor_holder_height/2)} ${position * parent_length} ${side * (parent_height/2 - motor_holder_radius/2)}"/>
+            <parent link="base_link"/>
+            <child link="${prefix}_motor_holder"/>
         </joint>
         <link name="${prefix}_wheel_link">
             <visual>
-                <origin rpy="${pi / 2} 0  0 " xyz="0 0 0"/>
+                <origin rpy="${pi / 2} 0 0 " xyz="0 0 0"/>
                 <geometry>
-                    <mesh filename="package://leobot_description/meshes/wheel.stl" scale="0.001 0.001 0.001"/>
-                    <xacro:blue_material/>
+                    <mesh filename="package://leobot_description/meshes/Mecanum_Wheel_${wheel_type}.STL" scale="0.001 0.001 0.001"/>
                 </geometry>
-                <xacro:red_material/>
             </visual>
-            <xacro:cylinder_collision radius="${radius}" height="${width}"/>
-            <xacro:cylinder_inertia mass="${mass}" radius="${radius}" height="${width}"/>
+            <xacro:cylinder_collision radius="${mecanum_radius}" height="${mecanum_height}"/>
+            <xacro:cylinder_inertia mass="${mecanum_mass}" radius="${mecanum_radius}" height="${mecanum_height}"/>
         </link>
-        <joint name="${prefix}_wheel_bearing_joint" type="continuous">
-            <origin rpy="0 0 0" xyz="0 0 ${direction * wheel_width/2}"/>
-            <parent link="${prefix}_bearing_link"/>
+        <joint name="${prefix}_wheel_motor_joint" type="continuous">
+            <origin rpy="0 0 0" xyz="0 0 ${side * mecanum_height/2}"/>
+            <parent link="${prefix}_motor_holder"/>
             <child link="${prefix}_wheel_link"/>
             <axis xyz="0 0 1"/>
@@ -37,5 +41,5 @@
         <transmission name="${prefix}_wheel_transmission">
             <type>transmission_interface/SimpleTransmission</type>
-            <joint name="${prefix}_wheel_bearing_joint">
+            <joint name="${prefix}_wheel_motor_joint">
                 <hardwareInterface>hardware_interface/VelocityJointInterface</hardwareInterface>
             </joint>
@@ -47,21 +51,3 @@
         </transmission>
     </xacro:macro>
-    <xacro:macro name="caster_wheel" params="radius mass x z">
-        <link name="caster_wheel_link">
-            <visual>
-                <geometry>
-                    <mesh filename="package://leobot_description/meshes/wheel-2-with-ball.stl"
-                          scale="0.001 0.001 0.001"/>
-                    <xacro:red_material/>
-                </geometry>
-            </visual>
-            <xacro:sphere_collision radius="${radius}"/>
-            <xacro:sphere_inertia mass="${mass}" radius="${radius}"/>
-        </link>
-        <joint name="caster_wheel_base_joint" type="fixed">
-            <parent link="chassis"/>
-            <child link="caster_wheel_link"/>
-            <origin rpy="0 0 0" xyz="${x} 0.0 ${z}"/>
-        </joint>
-    </xacro:macro>
 </robot>
