Commit message: Install the camera on rotating link in simulation
For task: Create rotational stereo camera URDF #130

File: leobot_description/robot/robot.urdf.xacro (robot description, xacro)
@@ -1,60 +1,62 @@
 <robot name="leobot" xmlns:xacro="http://ros.org/wiki/xacro">
-  <xacro:include filename="$(find leobot_description)/urdf/materials.urdf.xacro"/>
-  <xacro:include filename="$(find leobot_description)/urdf/common.urdf.xacro"/>
-  <xacro:include filename="$(find leobot_description)/urdf/sensors/camera.urdf.xacro"/>
-  <xacro:include filename="$(find leobot_description)/urdf/sensors/hokuyo.urdf.xacro"/>
-  <xacro:include filename="$(find leobot_description)/urdf/wheels.urdf.xacro"/>
-  <xacro:property name="base_width" value="0.54"/>
-  <xacro:property name="base_length" value="0.3"/>
-  <xacro:property name="base_height" value="0.5"/>
-  <xacro:property name="base_mass" value="10"/>
-  <xacro:property name="neck_width" value="0.04"/>
-  <xacro:property name="neck_length" value="0.04"/>
-  <xacro:property name="neck_height" value="1.45"/>
-  <xacro:property name="neck_mass" value="1.0"/>
+    <xacro:include filename="$(find leobot_description)/urdf/materials.urdf.xacro"/>
+    <xacro:include filename="$(find leobot_description)/urdf/common.urdf.xacro"/>
+    <xacro:include filename="$(find leobot_description)/urdf/sensors/camera.urdf.xacro"/>
+    <xacro:include filename="$(find leobot_description)/urdf/sensors/hokuyo.urdf.xacro"/>
+    <xacro:include filename="$(find leobot_description)/urdf/wheels.urdf.xacro"/>
+    <xacro:property name="base_width" value="0.54"/>
+    <xacro:property name="base_length" value="0.3"/>
+    <xacro:property name="base_height" value="0.5"/>
+    <xacro:property name="base_mass" value="10"/>
+    <xacro:property name="neck_width" value="0.04"/>
+    <xacro:property name="neck_length" value="0.04"/>
+    <xacro:property name="neck_height" value="1.45"/>
+    <xacro:property name="neck_mass" value="1.0"/>
   <xacro:property name="head_width" value="0.04"/>
   <xacro:property name="head_length" value="0.04"/>
   <xacro:property name="head_height" value="0.29"/>
   <xacro:property name="head_mass" value="0.5"/>
-  <link name="base_link">
-    <visual>
-      <xacro:box_geometry width="${base_width}" height="${base_height}" depth="${base_length}"/>
-      <xacro:green_material/>
-    </visual>
-    <xacro:box_collision width="${base_width}" height="${base_height}" depth="${base_length}"/>
-    <xacro:box_inertia width="${base_width}" height="${base_height}" depth="${base_length}" mass="${base_mass}"/>
-  </link>
-  <link name="neck_link">
-    <visual>
-      <xacro:box_geometry width="${neck_width}" height="${neck_height}" depth="${neck_length}"/>
-      <xacro:red_material/>
-    </visual>
-    <xacro:box_collision width="${neck_width}" height="${neck_height}" depth="${neck_length}"/>
-    <xacro:box_inertia width="${neck_width}" height="${neck_height}" depth="${neck_length}" mass="${head_mass}"/>
-  </link>
-  <joint name="base_neck_joint" type="fixed">
-    <origin rpy="${pi/2} 0  0" xyz="${-base_height/2 - neck_width} 0 ${-base_length/2 + neck_height / 2 }"/>
-    <parent link="base_link"/>
-    <child link="neck_link"/>
-  </joint>
-  <link name="head_link">
-    <visual>
-      <xacro:box_geometry width="${head_width}" height="${head_height}" depth="${head_length}"/>
-      <xacro:blue_material/>
-    </visual>
-    <xacro:box_collision width="${head_width}" height="${head_height}" depth="${head_length}"/>
-    <xacro:box_inertia width="${head_width}" height="${head_height}" depth="${head_length}" mass="${head_mass}"/>
-  </link>
-  <joint name="neck_head_joint" type="fixed">
-    <origin rpy="${pi/2} ${pi/2} ${pi}" xyz="${-neck_length/2 + head_height/2} ${neck_height/2 + head_width/2} 0"/>
-    <parent link="neck_link"/>
-    <child link="head_link"/>
-  </joint>
-  <xacro:fish_camera prefix = "left" parent_link_name="head_link" parent_height="${head_height}" parent_width = "${head_width}" side="1"/>
-  <xacro:fish_camera prefix = "right" parent_link_name="head_link" parent_height="${head_height}"  parent_width = "${head_width}" side="-1"/>
-  <xacro:lidar_hokuyo parent_link_name="base_link" parent_height="${base_length}"/>
-  <xacro:mecanum_wheel prefix="FL" wheel_type="2" side="1" position="1" parent_length="${base_width}" parent_height="${base_length}" parent_width="${base_height}"/>
-  <xacro:mecanum_wheel prefix="FR" wheel_type="1" side="-1" position="1" parent_length="${base_width}" parent_height="${base_length}" parent_width="${base_height}"/>
-  <xacro:mecanum_wheel prefix="RL" wheel_type="1" side="1" position="-1" parent_length="${base_width}" parent_height="${base_length}" parent_width="${base_height}"/>
-  <xacro:mecanum_wheel prefix="RR" wheel_type="2" side="-1" position="-1" parent_length="${base_width}" parent_height="${base_length}" parent_width="${base_height}"/>
+    <link name="base_link">
+        <visual>
+            <xacro:box_geometry width="${base_width}" height="${base_height}" depth="${base_length}"/>
+            <xacro:green_material/>
+        </visual>
+        <xacro:box_collision width="${base_width}" height="${base_height}" depth="${base_length}"/>
+        <xacro:box_inertia width="${base_width}" height="${base_height}" depth="${base_length}" mass="${base_mass}"/>
+    </link>
+    <link name="neck_link">
+        <visual>
+            <xacro:box_geometry width="${neck_width}" height="${neck_height}" depth="${neck_length}"/>
+            <xacro:red_material/>
+        </visual>
+        <xacro:box_collision width="${neck_width}" height="${neck_height}" depth="${neck_length}"/>
+        <xacro:box_inertia width="${neck_width}" height="${neck_height}" depth="${neck_length}" mass="${head_mass}"/>
+    </link>
+    <joint name="base_neck_joint" type="fixed">
+        <origin rpy="${pi/2} 0  0" xyz="${-base_height/2 - neck_width} 0 ${-base_length/2 + neck_height / 2 }"/>
+        <parent link="base_link"/>
+        <child link="neck_link"/>
+    </joint>
+    <link name="head_link">
+        <visual>
+            <xacro:box_geometry width="${head_width}" height="${head_height}" depth="${head_length}"/>
+            <origin xyz="0 ${neck_width/2 - head_height/2} 0"/>
+            <xacro:blue_material/>
+        </visual>
+        <xacro:box_collision width="${head_width}" height="${head_height}" depth="${head_length}"/>
+        <xacro:box_inertia width="${head_width}" height="${head_height}" depth="${head_length}" mass="${head_mass}"/>
+    </link>
+    <joint name="neck_head_joint" type="continuous">
+        <origin rpy="${pi/2} ${pi/2} ${pi}" xyz="0 ${neck_height/2 + head_width/2} 0"/>
+        <axis xyz="0 0 1"/>
+        <parent link="neck_link"/>
+        <child link="head_link"/>
+    </joint>
+    <xacro:fish_camera prefix = "left" parent_link_name="head_link" parent_height="${head_height}" parent_width = "${head_width}" side="1"/>
+    <xacro:fish_camera prefix = "right" parent_link_name="head_link" parent_height="${head_height}"  parent_width = "${head_width}" side="-1"/>
+    <xacro:lidar_hokuyo parent_link_name="base_link" parent_height="${base_length}"/>
+    <xacro:mecanum_wheel prefix="FL" wheel_type="2" side="1" position="1" parent_length="${base_width}" parent_height="${base_length}" parent_width="${base_height}"/>
+    <xacro:mecanum_wheel prefix="FR" wheel_type="1" side="-1" position="1" parent_length="${base_width}" parent_height="${base_length}" parent_width="${base_height}"/>
+    <xacro:mecanum_wheel prefix="RL" wheel_type="1" side="1" position="-1" parent_length="${base_width}" parent_height="${base_length}" parent_width="${base_height}"/>
+    <xacro:mecanum_wheel prefix="RR" wheel_type="2" side="-1" position="-1" parent_length="${base_width}" parent_height="${base_length}" parent_width="${base_height}"/>
 </robot>

File: leobot_description/urdf/sensors/camera.urdf.xacro (robot description, xacro)
@@ -13,5 +13,5 @@
         </link>
         <joint name="head_${prefix}_camera_joint" type="fixed">
-            <origin xyz="${side*(camera_radius + parent_width/2) - side*0.005} ${-parent_height/2 + camera_radius} 0" rpy="${pi/2 + side * pi/2 } ${pi/2 + side * pi/2 } 0"/>
+            <origin xyz="${side*(camera_radius + parent_width/2) - side*0.005} ${-parent_height + camera_radius} 0" rpy="${pi/2 + side * pi/2 } ${pi/2 + side * pi/2 } 0"/>
             <parent link="${parent_link_name}" />
             <child link="${prefix}_camera_link" />

Commit message: Revert "Install the camera on rotating link in simulation"
This reverts commit 8316707305632c3cccc847144fdf64394e86608e.

File: leobot_description/robot/robot.urdf.xacro (robot description, xacro)
@@ -1,62 +1,60 @@
 <robot name="leobot" xmlns:xacro="http://ros.org/wiki/xacro">
-    <xacro:include filename="$(find leobot_description)/urdf/materials.urdf.xacro"/>
-    <xacro:include filename="$(find leobot_description)/urdf/common.urdf.xacro"/>
-    <xacro:include filename="$(find leobot_description)/urdf/sensors/camera.urdf.xacro"/>
-    <xacro:include filename="$(find leobot_description)/urdf/sensors/hokuyo.urdf.xacro"/>
-    <xacro:include filename="$(find leobot_description)/urdf/wheels.urdf.xacro"/>
-    <xacro:property name="base_width" value="0.54"/>
-    <xacro:property name="base_length" value="0.3"/>
-    <xacro:property name="base_height" value="0.5"/>
-    <xacro:property name="base_mass" value="10"/>
-    <xacro:property name="neck_width" value="0.04"/>
-    <xacro:property name="neck_length" value="0.04"/>
-    <xacro:property name="neck_height" value="1.45"/>
-    <xacro:property name="neck_mass" value="1.0"/>
+  <xacro:include filename="$(find leobot_description)/urdf/materials.urdf.xacro"/>
+  <xacro:include filename="$(find leobot_description)/urdf/common.urdf.xacro"/>
+  <xacro:include filename="$(find leobot_description)/urdf/sensors/camera.urdf.xacro"/>
+  <xacro:include filename="$(find leobot_description)/urdf/sensors/hokuyo.urdf.xacro"/>
+  <xacro:include filename="$(find leobot_description)/urdf/wheels.urdf.xacro"/>
+  <xacro:property name="base_width" value="0.54"/>
+  <xacro:property name="base_length" value="0.3"/>
+  <xacro:property name="base_height" value="0.5"/>
+  <xacro:property name="base_mass" value="10"/>
+  <xacro:property name="neck_width" value="0.04"/>
+  <xacro:property name="neck_length" value="0.04"/>
+  <xacro:property name="neck_height" value="1.45"/>
+  <xacro:property name="neck_mass" value="1.0"/>
   <xacro:property name="head_width" value="0.04"/>
   <xacro:property name="head_length" value="0.04"/>
   <xacro:property name="head_height" value="0.29"/>
   <xacro:property name="head_mass" value="0.5"/>
-    <link name="base_link">
-        <visual>
-            <xacro:box_geometry width="${base_width}" height="${base_height}" depth="${base_length}"/>
-            <xacro:green_material/>
-        </visual>
-        <xacro:box_collision width="${base_width}" height="${base_height}" depth="${base_length}"/>
-        <xacro:box_inertia width="${base_width}" height="${base_height}" depth="${base_length}" mass="${base_mass}"/>
-    </link>
-    <link name="neck_link">
-        <visual>
-            <xacro:box_geometry width="${neck_width}" height="${neck_height}" depth="${neck_length}"/>
-            <xacro:red_material/>
-        </visual>
-        <xacro:box_collision width="${neck_width}" height="${neck_height}" depth="${neck_length}"/>
-        <xacro:box_inertia width="${neck_width}" height="${neck_height}" depth="${neck_length}" mass="${head_mass}"/>
-    </link>
-    <joint name="base_neck_joint" type="fixed">
-        <origin rpy="${pi/2} 0  0" xyz="${-base_height/2 - neck_width} 0 ${-base_length/2 + neck_height / 2 }"/>
-        <parent link="base_link"/>
-        <child link="neck_link"/>
-    </joint>
-    <link name="head_link">
-        <visual>
-            <xacro:box_geometry width="${head_width}" height="${head_height}" depth="${head_length}"/>
-            <origin xyz="0 ${neck_width/2 - head_height/2} 0"/>
-            <xacro:blue_material/>
-        </visual>
-        <xacro:box_collision width="${head_width}" height="${head_height}" depth="${head_length}"/>
-        <xacro:box_inertia width="${head_width}" height="${head_height}" depth="${head_length}" mass="${head_mass}"/>
-    </link>
-    <joint name="neck_head_joint" type="continuous">
-        <origin rpy="${pi/2} ${pi/2} ${pi}" xyz="0 ${neck_height/2 + head_width/2} 0"/>
-        <axis xyz="0 0 1"/>
-        <parent link="neck_link"/>
-        <child link="head_link"/>
-    </joint>
-    <xacro:fish_camera prefix = "left" parent_link_name="head_link" parent_height="${head_height}" parent_width = "${head_width}" side="1"/>
-    <xacro:fish_camera prefix = "right" parent_link_name="head_link" parent_height="${head_height}"  parent_width = "${head_width}" side="-1"/>
-    <xacro:lidar_hokuyo parent_link_name="base_link" parent_height="${base_length}"/>
-    <xacro:mecanum_wheel prefix="FL" wheel_type="2" side="1" position="1" parent_length="${base_width}" parent_height="${base_length}" parent_width="${base_height}"/>
-    <xacro:mecanum_wheel prefix="FR" wheel_type="1" side="-1" position="1" parent_length="${base_width}" parent_height="${base_length}" parent_width="${base_height}"/>
-    <xacro:mecanum_wheel prefix="RL" wheel_type="1" side="1" position="-1" parent_length="${base_width}" parent_height="${base_length}" parent_width="${base_height}"/>
-    <xacro:mecanum_wheel prefix="RR" wheel_type="2" side="-1" position="-1" parent_length="${base_width}" parent_height="${base_length}" parent_width="${base_height}"/>
+  <link name="base_link">
+    <visual>
+      <xacro:box_geometry width="${base_width}" height="${base_height}" depth="${base_length}"/>
+      <xacro:green_material/>
+    </visual>
+    <xacro:box_collision width="${base_width}" height="${base_height}" depth="${base_length}"/>
+    <xacro:box_inertia width="${base_width}" height="${base_height}" depth="${base_length}" mass="${base_mass}"/>
+  </link>
+  <link name="neck_link">
+    <visual>
+      <xacro:box_geometry width="${neck_width}" height="${neck_height}" depth="${neck_length}"/>
+      <xacro:red_material/>
+    </visual>
+    <xacro:box_collision width="${neck_width}" height="${neck_height}" depth="${neck_length}"/>
+    <xacro:box_inertia width="${neck_width}" height="${neck_height}" depth="${neck_length}" mass="${head_mass}"/>
+  </link>
+  <joint name="base_neck_joint" type="fixed">
+    <origin rpy="${pi/2} 0  0" xyz="${-base_height/2 - neck_width} 0 ${-base_length/2 + neck_height / 2 }"/>
+    <parent link="base_link"/>
+    <child link="neck_link"/>
+  </joint>
+  <link name="head_link">
+    <visual>
+      <xacro:box_geometry width="${head_width}" height="${head_height}" depth="${head_length}"/>
+      <xacro:blue_material/>
+    </visual>
+    <xacro:box_collision width="${head_width}" height="${head_height}" depth="${head_length}"/>
+    <xacro:box_inertia width="${head_width}" height="${head_height}" depth="${head_length}" mass="${head_mass}"/>
+  </link>
+  <joint name="neck_head_joint" type="fixed">
+    <origin rpy="${pi/2} ${pi/2} ${pi}" xyz="${-neck_length/2 + head_height/2} ${neck_height/2 + head_width/2} 0"/>
+    <parent link="neck_link"/>
+    <child link="head_link"/>
+  </joint>
+  <xacro:fish_camera prefix = "left" parent_link_name="head_link" parent_height="${head_height}" parent_width = "${head_width}" side="1"/>
+  <xacro:fish_camera prefix = "right" parent_link_name="head_link" parent_height="${head_height}"  parent_width = "${head_width}" side="-1"/>
+  <xacro:lidar_hokuyo parent_link_name="base_link" parent_height="${base_length}"/>
+  <xacro:mecanum_wheel prefix="FL" wheel_type="2" side="1" position="1" parent_length="${base_width}" parent_height="${base_length}" parent_width="${base_height}"/>
+  <xacro:mecanum_wheel prefix="FR" wheel_type="1" side="-1" position="1" parent_length="${base_width}" parent_height="${base_length}" parent_width="${base_height}"/>
+  <xacro:mecanum_wheel prefix="RL" wheel_type="1" side="1" position="-1" parent_length="${base_width}" parent_height="${base_length}" parent_width="${base_height}"/>
+  <xacro:mecanum_wheel prefix="RR" wheel_type="2" side="-1" position="-1" parent_length="${base_width}" parent_height="${base_length}" parent_width="${base_height}"/>
 </robot>

File: leobot_description/urdf/sensors/camera.urdf.xacro (robot description, xacro)
@@ -13,5 +13,5 @@
         </link>
         <joint name="head_${prefix}_camera_joint" type="fixed">
-            <origin xyz="${side*(camera_radius + parent_width/2) - side*0.005} ${-parent_height + camera_radius} 0" rpy="${pi/2 + side * pi/2 } ${pi/2 + side * pi/2 } 0"/>
+            <origin xyz="${side*(camera_radius + parent_width/2) - side*0.005} ${-parent_height/2 + camera_radius} 0" rpy="${pi/2 + side * pi/2 } ${pi/2 + side * pi/2 } 0"/>
             <parent link="${parent_link_name}" />
             <child link="${prefix}_camera_link" />
