Commit message: Attach the cameras to rotating camera stick in simulation
For task: Create rotational stereo camera URDF #130

File: leobot_description/robot/robot.urdf.xacro (robot description, xacro)
@@ -5,16 +5,20 @@
     <xacro:include filename="$(find leobot_description)/urdf/sensors/hokuyo.urdf.xacro"/>
     <xacro:include filename="$(find leobot_description)/urdf/wheels.urdf.xacro"/>
-    <xacro:property name="base_width" value="0.54"/>
+    <xacro:property name="base_width"  value="0.54"/>
     <xacro:property name="base_length" value="0.3"/>
     <xacro:property name="base_height" value="0.5"/>
-    <xacro:property name="base_mass" value="10"/>
-    <xacro:property name="neck_width" value="0.04"/>
+    <xacro:property name="base_mass"   value="10"/>
+    <xacro:property name="neck_width"  value="0.04"/>
     <xacro:property name="neck_length" value="0.04"/>
     <xacro:property name="neck_height" value="1.45"/>
-    <xacro:property name="neck_mass" value="1.0"/>
-    <xacro:property name="head_width" value="0.04"/>
+    <xacro:property name="neck_mass"   value="1.0"/>
+    <xacro:property name="head_width"  value="0.04"/>
     <xacro:property name="head_length" value="0.04"/>
     <xacro:property name="head_height" value="0.29"/>
-    <xacro:property name="head_mass" value="0.5"/>
+    <xacro:property name="head_mass"   value="0.5"/>
+    <xacro:property name="camera_stick_width"  value="0.02"/>
+    <xacro:property name="camera_stick_length" value="0.04"/>
+    <xacro:property name="camera_stick_height" value="0.1"/>
+    <xacro:property name="camera_stick_mass"   value="0.2"/>
     <link name="base_link">
         <visual>
@@ -23,5 +27,5 @@
         </visual>
         <xacro:box_collision width="${base_width}" height="${base_height}" depth="${base_length}"/>
-        <xacro:box_inertia width="${base_width}" height="${base_height}" depth="${base_length}" mass="${base_mass}"/>
+        <xacro:box_inertia   width="${base_width}" height="${base_height}" depth="${base_length}" mass="${base_mass}"/>
     </link>
     <link name="neck_link">
@@ -31,5 +35,5 @@
         </visual>
         <xacro:box_collision width="${neck_width}" height="${neck_height}" depth="${neck_length}"/>
-        <xacro:box_inertia width="${neck_width}" height="${neck_height}" depth="${neck_length}" mass="${head_mass}"/>
+        <xacro:box_inertia   width="${neck_width}" height="${neck_height}" depth="${neck_length}" mass="${head_mass}"/>
     </link>
     <joint name="base_neck_joint" type="fixed">
@@ -44,5 +48,5 @@
         </visual>
         <xacro:box_collision width="${head_width}" height="${head_height}" depth="${head_length}"/>
-        <xacro:box_inertia width="${head_width}" height="${head_height}" depth="${head_length}" mass="${head_mass}"/>
+        <xacro:box_inertia   width="${head_width}" height="${head_height}" depth="${head_length}" mass="${head_mass}"/>
     </link>
     <joint name="neck_head_joint" type="fixed">
@@ -51,10 +55,24 @@
         <child link="head_link"/>
     </joint>
-    <xacro:fish_camera prefix = "left" parent_link_name="head_link" parent_height="${head_height}" parent_width = "${head_width}" side="1"/>
-    <xacro:fish_camera prefix = "right" parent_link_name="head_link" parent_height="${head_height}"  parent_width = "${head_width}" side="-1"/>
+    <link name="camera_stick_link">
+        <visual>
+            <xacro:box_geometry width="${camera_stick_width}" height="${camera_stick_height}" depth="${camera_stick_length}"/>
+            <xacro:yellow_material/>
+        </visual>
+        <xacro:box_collision width="${camera_stick_width}" height="${camera_stick_height}" depth="${camera_stick_length}"/>
+        <xacro:box_inertia   width="${camera_stick_width}" height="${camera_stick_height}" depth="${camera_stick_length}" mass="${camera_stick_mass}"/>
+    </link>
+    <joint name="head_camera_stick_joint" type="continuous">
+        <origin rpy="${pi/2} ${pi/2} ${pi}"
+                xyz="0 ${camera_stick_length/2 - head_height/2} ${head_width/2 + camera_stick_width/2}"/>
+        <parent link="head_link"/>
+        <child link="camera_stick_link"/>
+    </joint>
+    <xacro:fish_camera prefix="left"  parent_link_name="camera_stick_link" parent_height="${camera_stick_height}" parent_width="${camera_stick_width}" side="1"/>
+    <xacro:fish_camera prefix="right" parent_link_name="camera_stick_link" parent_height="${camera_stick_height}" parent_width="${camera_stick_width}" side="-1"/>
     <xacro:lidar_hokuyo parent_link_name="base_link" parent_height="${base_length}"/>
-    <xacro:mecanum_wheel prefix="FL" wheel_type="2" side="1" position="1" parent_length="${base_width}" parent_height="${base_length}" parent_width="${base_height}"/>
-    <xacro:mecanum_wheel prefix="FR" wheel_type="1" side="-1" position="1" parent_length="${base_width}" parent_height="${base_length}" parent_width="${base_height}"/>
-    <xacro:mecanum_wheel prefix="RL" wheel_type="1" side="1" position="-1" parent_length="${base_width}" parent_height="${base_length}" parent_width="${base_height}"/>
+    <xacro:mecanum_wheel prefix="FL" wheel_type="2" side="1"  position="1"  parent_length="${base_width}" parent_height="${base_length}" parent_width="${base_height}"/>
+    <xacro:mecanum_wheel prefix="FR" wheel_type="1" side="-1" position="1"  parent_length="${base_width}" parent_height="${base_length}" parent_width="${base_height}"/>
+    <xacro:mecanum_wheel prefix="RL" wheel_type="1" side="1"  position="-1" parent_length="${base_width}" parent_height="${base_length}" parent_width="${base_height}"/>
     <xacro:mecanum_wheel prefix="RR" wheel_type="2" side="-1" position="-1" parent_length="${base_width}" parent_height="${base_length}" parent_width="${base_height}"/>
 </robot>

File: leobot_description/urdf/materials.urdf.xacro (robot description, xacro)
@@ -30,3 +30,8 @@
         </material>
     </xacro:macro>
+    <xacro:macro name="yellow_material">
+        <material name="yellow">
+            <color rgba="1.0 1.0 0.0 1.0"/>
+        </material>
+    </xacro:macro>
 </robot>

File: leobot_description/urdf/sensors/camera.urdf.xacro (robot description, xacro)
@@ -1,5 +1,5 @@
 <robot xmlns:xacro="http://ros.org/wiki/xacro">
     <xacro:property name="camera_radius" value="0.025"/>
-    <xacro:property name="camera_mass" value="0.1"/>
+    <xacro:property name="camera_mass"   value="0.1"/>
     <xacro:macro name="fish_camera" params="prefix parent_link_name parent_height side parent_width">
         <link name="${prefix}_camera_link">
@@ -11,8 +11,9 @@
             <xacro:sphere_inertia mass="${camera_mass}" radius="${camera_radius}"/>
         </link>
-        <joint name="head_${prefix}_camera_joint" type="fixed">
-            <origin xyz="${side*(camera_radius + parent_width/2) - side*0.005} ${-parent_height/2 + camera_radius} 0" rpy="${pi/2 + side * pi/2 } ${pi/2 + side * pi/2 } 0"/>
-            <parent link="${parent_link_name}" />
-            <child link="${prefix}_camera_link" />
+        <joint name="${prefix}_camera_joint" type="fixed">
+            <origin xyz="${-camera_radius - parent_width/2} ${side*(-camera_radius/2 + parent_height/2)} 0"
+                    rpy="${pi/2 + side * pi/2} ${pi/2 + side * pi/2} 0"/>
+            <parent link="${parent_link_name}"/>
+            <child link="${prefix}_camera_link"/>
         </joint>
     </xacro:macro>

Commit message: Revert "Attach the cameras to rotating camera stick in simulation"
This reverts commit fd95d78359684576527301b66394138c925b441a.

File: leobot_description/robot/robot.urdf.xacro (robot description, xacro)
@@ -5,20 +5,16 @@
     <xacro:include filename="$(find leobot_description)/urdf/sensors/hokuyo.urdf.xacro"/>
     <xacro:include filename="$(find leobot_description)/urdf/wheels.urdf.xacro"/>
-    <xacro:property name="base_width"  value="0.54"/>
+    <xacro:property name="base_width" value="0.54"/>
     <xacro:property name="base_length" value="0.3"/>
     <xacro:property name="base_height" value="0.5"/>
-    <xacro:property name="base_mass"   value="10"/>
-    <xacro:property name="neck_width"  value="0.04"/>
+    <xacro:property name="base_mass" value="10"/>
+    <xacro:property name="neck_width" value="0.04"/>
     <xacro:property name="neck_length" value="0.04"/>
     <xacro:property name="neck_height" value="1.45"/>
-    <xacro:property name="neck_mass"   value="1.0"/>
-    <xacro:property name="head_width"  value="0.04"/>
+    <xacro:property name="neck_mass" value="1.0"/>
+    <xacro:property name="head_width" value="0.04"/>
     <xacro:property name="head_length" value="0.04"/>
     <xacro:property name="head_height" value="0.29"/>
-    <xacro:property name="head_mass"   value="0.5"/>
-    <xacro:property name="camera_stick_width"  value="0.02"/>
-    <xacro:property name="camera_stick_length" value="0.04"/>
-    <xacro:property name="camera_stick_height" value="0.1"/>
-    <xacro:property name="camera_stick_mass"   value="0.2"/>
+    <xacro:property name="head_mass" value="0.5"/>
     <link name="base_link">
         <visual>
@@ -27,5 +23,5 @@
         </visual>
         <xacro:box_collision width="${base_width}" height="${base_height}" depth="${base_length}"/>
-        <xacro:box_inertia   width="${base_width}" height="${base_height}" depth="${base_length}" mass="${base_mass}"/>
+        <xacro:box_inertia width="${base_width}" height="${base_height}" depth="${base_length}" mass="${base_mass}"/>
     </link>
     <link name="neck_link">
@@ -35,5 +31,5 @@
         </visual>
         <xacro:box_collision width="${neck_width}" height="${neck_height}" depth="${neck_length}"/>
-        <xacro:box_inertia   width="${neck_width}" height="${neck_height}" depth="${neck_length}" mass="${head_mass}"/>
+        <xacro:box_inertia width="${neck_width}" height="${neck_height}" depth="${neck_length}" mass="${head_mass}"/>
     </link>
     <joint name="base_neck_joint" type="fixed">
@@ -48,5 +44,5 @@
         </visual>
         <xacro:box_collision width="${head_width}" height="${head_height}" depth="${head_length}"/>
-        <xacro:box_inertia   width="${head_width}" height="${head_height}" depth="${head_length}" mass="${head_mass}"/>
+        <xacro:box_inertia width="${head_width}" height="${head_height}" depth="${head_length}" mass="${head_mass}"/>
     </link>
     <joint name="neck_head_joint" type="fixed">
@@ -55,24 +51,10 @@
         <child link="head_link"/>
     </joint>
-    <link name="camera_stick_link">
-        <visual>
-            <xacro:box_geometry width="${camera_stick_width}" height="${camera_stick_height}" depth="${camera_stick_length}"/>
-            <xacro:yellow_material/>
-        </visual>
-        <xacro:box_collision width="${camera_stick_width}" height="${camera_stick_height}" depth="${camera_stick_length}"/>
-        <xacro:box_inertia   width="${camera_stick_width}" height="${camera_stick_height}" depth="${camera_stick_length}" mass="${camera_stick_mass}"/>
-    </link>
-    <joint name="head_camera_stick_joint" type="continuous">
-        <origin rpy="${pi/2} ${pi/2} ${pi}"
-                xyz="0 ${camera_stick_length/2 - head_height/2} ${head_width/2 + camera_stick_width/2}"/>
-        <parent link="head_link"/>
-        <child link="camera_stick_link"/>
-    </joint>
-    <xacro:fish_camera prefix="left"  parent_link_name="camera_stick_link" parent_height="${camera_stick_height}" parent_width="${camera_stick_width}" side="1"/>
-    <xacro:fish_camera prefix="right" parent_link_name="camera_stick_link" parent_height="${camera_stick_height}" parent_width="${camera_stick_width}" side="-1"/>
+    <xacro:fish_camera prefix = "left" parent_link_name="head_link" parent_height="${head_height}" parent_width = "${head_width}" side="1"/>
+    <xacro:fish_camera prefix = "right" parent_link_name="head_link" parent_height="${head_height}"  parent_width = "${head_width}" side="-1"/>
     <xacro:lidar_hokuyo parent_link_name="base_link" parent_height="${base_length}"/>
-    <xacro:mecanum_wheel prefix="FL" wheel_type="2" side="1"  position="1"  parent_length="${base_width}" parent_height="${base_length}" parent_width="${base_height}"/>
-    <xacro:mecanum_wheel prefix="FR" wheel_type="1" side="-1" position="1"  parent_length="${base_width}" parent_height="${base_length}" parent_width="${base_height}"/>
-    <xacro:mecanum_wheel prefix="RL" wheel_type="1" side="1"  position="-1" parent_length="${base_width}" parent_height="${base_length}" parent_width="${base_height}"/>
+    <xacro:mecanum_wheel prefix="FL" wheel_type="2" side="1" position="1" parent_length="${base_width}" parent_height="${base_length}" parent_width="${base_height}"/>
+    <xacro:mecanum_wheel prefix="FR" wheel_type="1" side="-1" position="1" parent_length="${base_width}" parent_height="${base_length}" parent_width="${base_height}"/>
+    <xacro:mecanum_wheel prefix="RL" wheel_type="1" side="1" position="-1" parent_length="${base_width}" parent_height="${base_length}" parent_width="${base_height}"/>
     <xacro:mecanum_wheel prefix="RR" wheel_type="2" side="-1" position="-1" parent_length="${base_width}" parent_height="${base_length}" parent_width="${base_height}"/>
 </robot>

File: leobot_description/urdf/materials.urdf.xacro (robot description, xacro)
@@ -30,8 +30,3 @@
         </material>
     </xacro:macro>
-    <xacro:macro name="yellow_material">
-        <material name="yellow">
-            <color rgba="1.0 1.0 0.0 1.0"/>
-        </material>
-    </xacro:macro>
 </robot>

File: leobot_description/urdf/sensors/camera.urdf.xacro (robot description, xacro)
@@ -1,5 +1,5 @@
 <robot xmlns:xacro="http://ros.org/wiki/xacro">
     <xacro:property name="camera_radius" value="0.025"/>
-    <xacro:property name="camera_mass"   value="0.1"/>
+    <xacro:property name="camera_mass" value="0.1"/>
     <xacro:macro name="fish_camera" params="prefix parent_link_name parent_height side parent_width">
         <link name="${prefix}_camera_link">
@@ -11,9 +11,8 @@
             <xacro:sphere_inertia mass="${camera_mass}" radius="${camera_radius}"/>
         </link>
-        <joint name="${prefix}_camera_joint" type="fixed">
-            <origin xyz="${-camera_radius - parent_width/2} ${side*(-camera_radius/2 + parent_height/2)} 0"
-                    rpy="${pi/2 + side * pi/2} ${pi/2 + side * pi/2} 0"/>
-            <parent link="${parent_link_name}"/>
-            <child link="${prefix}_camera_link"/>
+        <joint name="head_${prefix}_camera_joint" type="fixed">
+            <origin xyz="${side*(camera_radius + parent_width/2) - side*0.005} ${-parent_height/2 + camera_radius} 0" rpy="${pi/2 + side * pi/2 } ${pi/2 + side * pi/2 } 0"/>
+            <parent link="${parent_link_name}" />
+            <child link="${prefix}_camera_link" />
         </joint>
     </xacro:macro>

Commit message: Attach the cameras to rotating camera stick in simulation
For task: Create rotational stereo camera URDF #130

File: leobot_description/robot/robot.urdf.xacro (robot description, xacro)
@@ -17,4 +17,8 @@
   <xacro:property name="head_height" value="0.29"/>
   <xacro:property name="head_mass" value="0.5"/>
+  <xacro:property name="camera_stick_width"  value="0.02"/>
+  <xacro:property name="camera_stick_length" value="0.04"/>
+  <xacro:property name="camera_stick_height" value="0.1"/>
+  <xacro:property name="camera_stick_mass"   value="0.2"/>
   <link name="base_link">
     <visual>
@@ -51,6 +55,20 @@
     <child link="head_link"/>
   </joint>
-  <xacro:fish_camera prefix = "left" parent_link_name="head_link" parent_height="${head_height}" parent_width = "${head_width}" side="1"/>
-  <xacro:fish_camera prefix = "right" parent_link_name="head_link" parent_height="${head_height}"  parent_width = "${head_width}" side="-1"/>
+  <link name="camera_stick_link">
+    <visual>
+      <xacro:box_geometry width="${camera_stick_width}" height="${camera_stick_height}" depth="${camera_stick_length}"/>
+      <xacro:yellow_material/>
+    </visual>
+    <xacro:box_collision width="${camera_stick_width}" height="${camera_stick_height}" depth="${camera_stick_length}"/>
+    <xacro:box_inertia   width="${camera_stick_width}" height="${camera_stick_height}" depth="${camera_stick_length}" mass="${camera_stick_mass}"/>
+  </link>
+  <joint name="head_camera_stick_joint" type="continuous">
+    <origin rpy="${pi/2} ${pi/2} ${pi}"
+            xyz="0 ${camera_stick_length/2 - head_height/2} ${head_width/2 + camera_stick_width/2}"/>
+    <parent link="head_link"/>
+    <child link="camera_stick_link"/>
+  </joint>
+  <xacro:fish_camera prefix="left"  parent_link_name="camera_stick_link" parent_height="${camera_stick_height}" parent_width="${camera_stick_width}" side="1"/>
+  <xacro:fish_camera prefix="right" parent_link_name="camera_stick_link" parent_height="${camera_stick_height}" parent_width="${camera_stick_width}" side="-1"/>
   <xacro:lidar_hokuyo parent_link_name="base_link" parent_height="${base_length}"/>
   <xacro:mecanum_wheel prefix="FL" wheel_type="2" side="1" position="1" parent_length="${base_width}" parent_height="${base_length}" parent_width="${base_height}"/>

File: leobot_description/urdf/sensors/camera.urdf.xacro (robot description, xacro)
@@ -13,5 +13,5 @@
         </link>
         <joint name="${prefix}_camera_joint" type="fixed">
-            <origin xyz="${-camera_radius - parent_width/2} ${side*(-camera_radius/2 + parent_height/2)} 0"
+            <origin xyz="${-camera_radius - parent_width/2} ${side*(parent_height/2 - camera_radius/2)} 0"
                     rpy="${pi/2 + side * pi/2} ${pi/2 + side * pi/2} 0"/>
             <parent link="${parent_link_name}"/>
