Commit message: Indent xacro files with 4 spaces per level and delete the optional xml declaration

File: leobot_description/robot/robot.urdf.xacro (robot description, xacro)
@@ -1,78 +1,78 @@
 <robot name="leobot" xmlns:xacro="http://ros.org/wiki/xacro">
-  <xacro:include filename="$(find leobot_description)/urdf/materials.urdf.xacro"/>
-  <xacro:include filename="$(find leobot_description)/urdf/common.urdf.xacro"/>
-  <xacro:include filename="$(find leobot_description)/urdf/sensors/camera.urdf.xacro"/>
-  <xacro:include filename="$(find leobot_description)/urdf/sensors/hokuyo.urdf.xacro"/>
-  <xacro:include filename="$(find leobot_description)/urdf/wheels.urdf.xacro"/>
-  <xacro:property name="base_width" value="0.54"/>
-  <xacro:property name="base_length" value="0.3"/>
-  <xacro:property name="base_height" value="0.5"/>
-  <xacro:property name="base_mass" value="10"/>
-  <xacro:property name="neck_width" value="0.04"/>
-  <xacro:property name="neck_length" value="0.04"/>
-  <xacro:property name="neck_height" value="1.45"/>
-  <xacro:property name="neck_mass" value="1.0"/>
-  <xacro:property name="head_width" value="0.04"/>
-  <xacro:property name="head_length" value="0.04"/>
-  <xacro:property name="head_height" value="0.29"/>
-  <xacro:property name="head_mass" value="0.5"/>
-  <xacro:property name="camera_stick_width"  value="0.02"/>
-  <xacro:property name="camera_stick_length" value="0.04"/>
-  <xacro:property name="camera_stick_height" value="0.1"/>
-  <xacro:property name="camera_stick_mass"   value="0.2"/>
-  <link name="base_link">
-    <visual>
-      <xacro:box_geometry width="${base_width}" height="${base_height}" depth="${base_length}"/>
-      <xacro:green_material/>
-    </visual>
-    <xacro:box_collision width="${base_width}" height="${base_height}" depth="${base_length}"/>
-    <xacro:box_inertia width="${base_width}" height="${base_height}" depth="${base_length}" mass="${base_mass}"/>
-  </link>
-  <link name="neck_link">
-    <visual>
-      <xacro:box_geometry width="${neck_width}" height="${neck_height}" depth="${neck_length}"/>
-      <xacro:red_material/>
-    </visual>
-    <xacro:box_collision width="${neck_width}" height="${neck_height}" depth="${neck_length}"/>
-    <xacro:box_inertia width="${neck_width}" height="${neck_height}" depth="${neck_length}" mass="${head_mass}"/>
-  </link>
-  <joint name="base_neck_joint" type="fixed">
-    <origin rpy="${pi/2} 0  0" xyz="${-base_height/2 - neck_width} 0 ${-base_length/2 + neck_height / 2 }"/>
-    <parent link="base_link"/>
-    <child link="neck_link"/>
-  </joint>
-  <link name="head_link">
-    <visual>
-      <xacro:box_geometry width="${head_width}" height="${head_height}" depth="${head_length}"/>
-      <xacro:blue_material/>
-    </visual>
-    <xacro:box_collision width="${head_width}" height="${head_height}" depth="${head_length}"/>
-    <xacro:box_inertia width="${head_width}" height="${head_height}" depth="${head_length}" mass="${head_mass}"/>
-  </link>
-  <joint name="neck_head_joint" type="fixed">
-    <origin rpy="${pi/2} ${pi/2} ${pi}" xyz="${-neck_length/2 + head_height/2} ${neck_height/2 + head_width/2} 0"/>
-    <parent link="neck_link"/>
-    <child link="head_link"/>
-  </joint>
-  <link name="camera_stick_link">
-    <visual>
-      <xacro:box_geometry width="${camera_stick_width}" height="${camera_stick_height}" depth="${camera_stick_length}"/>
-      <xacro:yellow_material/>
-    </visual>
-    <xacro:box_collision width="${camera_stick_width}" height="${camera_stick_height}" depth="${camera_stick_length}"/>
-    <xacro:box_inertia   width="${camera_stick_width}" height="${camera_stick_height}" depth="${camera_stick_length}" mass="${camera_stick_mass}"/>
-  </link>
-  <joint name="head_camera_stick_joint" type="continuous">
-    <origin rpy="${pi/2} ${pi/2} ${pi}"
-            xyz="0 ${camera_stick_length/2 - head_height/2} ${head_width/2 + camera_stick_width/2}"/>
-    <parent link="head_link"/>
-    <child link="camera_stick_link"/>
-  </joint>
-  <xacro:fish_camera prefix="left"  parent_link_name="camera_stick_link" parent_height="${camera_stick_height}" parent_width="${camera_stick_width}" side="1"/>
-  <xacro:fish_camera prefix="right" parent_link_name="camera_stick_link" parent_height="${camera_stick_height}" parent_width="${camera_stick_width}" side="-1"/>
-  <xacro:lidar_hokuyo parent_link_name="base_link" parent_height="${base_length}"/>
-  <xacro:mecanum_wheel prefix="FL" wheel_type="2" side="1" position="1" parent_length="${base_width}" parent_height="${base_length}" parent_width="${base_height}"/>
-  <xacro:mecanum_wheel prefix="FR" wheel_type="1" side="-1" position="1" parent_length="${base_width}" parent_height="${base_length}" parent_width="${base_height}"/>
-  <xacro:mecanum_wheel prefix="RL" wheel_type="1" side="1" position="-1" parent_length="${base_width}" parent_height="${base_length}" parent_width="${base_height}"/>
-  <xacro:mecanum_wheel prefix="RR" wheel_type="2" side="-1" position="-1" parent_length="${base_width}" parent_height="${base_length}" parent_width="${base_height}"/>
+    <xacro:include filename="$(find leobot_description)/urdf/materials.urdf.xacro"/>
+    <xacro:include filename="$(find leobot_description)/urdf/common.urdf.xacro"/>
+    <xacro:include filename="$(find leobot_description)/urdf/sensors/camera.urdf.xacro"/>
+    <xacro:include filename="$(find leobot_description)/urdf/sensors/hokuyo.urdf.xacro"/>
+    <xacro:include filename="$(find leobot_description)/urdf/wheels.urdf.xacro"/>
+    <xacro:property name="base_width"  value="0.54"/>
+    <xacro:property name="base_length" value="0.3"/>
+    <xacro:property name="base_height" value="0.5"/>
+    <xacro:property name="base_mass"   value="10"/>
+    <xacro:property name="neck_width"  value="0.04"/>
+    <xacro:property name="neck_length" value="0.04"/>
+    <xacro:property name="neck_height" value="1.45"/>
+    <xacro:property name="neck_mass"   value="1.0"/>
+    <xacro:property name="head_width"  value="0.04"/>
+    <xacro:property name="head_length" value="0.04"/>
+    <xacro:property name="head_height" value="0.29"/>
+    <xacro:property name="head_mass"   value="0.5"/>
+    <xacro:property name="camera_stick_width"  value="0.02"/>
+    <xacro:property name="camera_stick_length" value="0.04"/>
+    <xacro:property name="camera_stick_height" value="0.1"/>
+    <xacro:property name="camera_stick_mass"   value="0.2"/>
+    <link name="base_link">
+        <visual>
+            <xacro:box_geometry width="${base_width}" height="${base_height}" depth="${base_length}"/>
+            <xacro:green_material/>
+        </visual>
+        <xacro:box_collision width="${base_width}" height="${base_height}" depth="${base_length}"/>
+        <xacro:box_inertia   width="${base_width}" height="${base_height}" depth="${base_length}" mass="${base_mass}"/>
+    </link>
+    <link name="neck_link">
+        <visual>
+            <xacro:box_geometry width="${neck_width}" height="${neck_height}" depth="${neck_length}"/>
+            <xacro:red_material/>
+        </visual>
+        <xacro:box_collision width="${neck_width}" height="${neck_height}" depth="${neck_length}"/>
+        <xacro:box_inertia   width="${neck_width}" height="${neck_height}" depth="${neck_length}" mass="${head_mass}"/>
+    </link>
+    <joint name="base_neck_joint" type="fixed">
+        <origin rpy="${pi/2} 0 0" xyz="${-base_height/2 - neck_width} 0 ${-base_length/2 + neck_height / 2 }"/>
+        <parent link="base_link"/>
+        <child link="neck_link"/>
+    </joint>
+    <link name="head_link">
+        <visual>
+            <xacro:box_geometry width="${head_width}" height="${head_height}" depth="${head_length}"/>
+            <xacro:blue_material/>
+        </visual>
+        <xacro:box_collision width="${head_width}" height="${head_height}" depth="${head_length}"/>
+        <xacro:box_inertia   width="${head_width}" height="${head_height}" depth="${head_length}" mass="${head_mass}"/>
+    </link>
+    <joint name="neck_head_joint" type="fixed">
+        <origin rpy="${pi/2} ${pi/2} ${pi}" xyz="${-neck_length/2 + head_height/2} ${neck_height/2 + head_width/2} 0"/>
+        <parent link="neck_link"/>
+        <child link="head_link"/>
+    </joint>
+    <link name="camera_stick_link">
+        <visual>
+            <xacro:box_geometry width="${camera_stick_width}" height="${camera_stick_height}" depth="${camera_stick_length}"/>
+            <xacro:yellow_material/>
+        </visual>
+        <xacro:box_collision width="${camera_stick_width}" height="${camera_stick_height}" depth="${camera_stick_length}"/>
+        <xacro:box_inertia   width="${camera_stick_width}" height="${camera_stick_height}" depth="${camera_stick_length}" mass="${camera_stick_mass}"/>
+    </link>
+    <joint name="head_camera_stick_joint" type="continuous">
+        <origin rpy="${pi/2} ${pi/2} ${pi}"
+                xyz="0 ${camera_stick_length/2 - head_height/2} ${head_width/2 + camera_stick_width/2}"/>
+        <parent link="head_link"/>
+        <child link="camera_stick_link"/>
+    </joint>
+    <xacro:fish_camera prefix="left"  parent_link_name="camera_stick_link" parent_height="${camera_stick_height}" parent_width="${camera_stick_width}" side="1"/>
+    <xacro:fish_camera prefix="right" parent_link_name="camera_stick_link" parent_height="${camera_stick_height}" parent_width="${camera_stick_width}" side="-1"/>
+    <xacro:lidar_hokuyo parent_link_name="base_link" parent_height="${base_length}"/>
+    <xacro:mecanum_wheel prefix="FL" wheel_type="2" side="1"  position="1"  parent_length="${base_width}" parent_height="${base_length}" parent_width="${base_height}"/>
+    <xacro:mecanum_wheel prefix="FR" wheel_type="1" side="-1" position="1"  parent_length="${base_width}" parent_height="${base_length}" parent_width="${base_height}"/>
+    <xacro:mecanum_wheel prefix="RL" wheel_type="1" side="1"  position="-1" parent_length="${base_width}" parent_height="${base_length}" parent_width="${base_height}"/>
+    <xacro:mecanum_wheel prefix="RR" wheel_type="2" side="-1" position="-1" parent_length="${base_width}" parent_height="${base_length}" parent_width="${base_height}"/>
 </robot>

File: leobot_description/urdf/common.urdf.xacro (robot description, xacro)
@@ -1,80 +1,79 @@
-<?xml version="1.0"?>
 <robot xmlns:xacro="http://ros.org/wiki/xacro">
-  <xacro:macro name="sphere_inertia" params="mass radius">
-    <inertial>
-      <mass value="${mass}"/>
-      <origin xyz="0 0 0"/>
-      <inertia ixx="${2*mass*radius*radius/5}" ixy="0.0" ixz="0.0"
-               iyy="${2*mass*radius*radius/5}" iyz="0.0"
-               izz="${2*mass*radius*radius/5}"/>
-    </inertial>
-  </xacro:macro>
-  <xacro:macro name="sphere_inertia_gazebo" params="mass radius">
-    <inertial>
-      <mass>${mass}</mass>
-      <inertia>
-        <ixx>${2*mass*radius*radius/5}</ixx>
-        <ixy>0</ixy>
-        <iyy>${2*mass*radius*radius/5}</iyy>
-        <ixz>0</ixz>
-        <iyz>0</iyz>
-        <izz>${2*mass*radius*radius/5}</izz>
-      </inertia>
-    </inertial>
-  </xacro:macro>
-  <xacro:macro name="sphere_geometry" params="radius">
-    <geometry>
-      <sphere radius="${radius}"/>
-    </geometry>
-  </xacro:macro>
-  <xacro:macro name="sphere_geometry_gazebo" params="radius">
-    <geometry>
-      <sphere>
-        <radius>${radius}</radius>
-      </sphere>
-    </geometry>
-  </xacro:macro>
-  <xacro:macro name="sphere_collision" params="radius">
-    <collision>
-      <xacro:sphere_geometry radius="${radius}"/>
-    </collision>
-  </xacro:macro>
-  <xacro:macro name="cylinder_inertia" params="mass radius height">
-    <inertial>
-      <mass value="${mass}"/>
-      <origin xyz="0 0 0"/>
-      <inertia ixx="${(3*radius*radius + height*height)*mass/12}" ixy="0.0" ixz="0.0"
-               iyy="${(3*radius*radius + height*height)*mass/12}" iyz="0.0"
-               izz="${radius*radius*mass/2}"/>
-    </inertial>
-  </xacro:macro>
-  <xacro:macro name="cylinder_geometry" params="radius height">
-    <geometry>
-      <cylinder length="${height}" radius="${radius}"/>
-    </geometry>
-  </xacro:macro>
-  <xacro:macro name="cylinder_collision" params="radius height">
-    <collision>
-      <xacro:cylinder_geometry radius="${radius}" height="${height}"/>
-    </collision>
-  </xacro:macro>
-  <xacro:macro name="box_inertia" params="mass width height depth x:=0 y:=0 z:=0 roll:=0 pitch:=0 yaw:=0">
-    <inertial>
-      <origin xyz="${x} ${y} ${z}" rpy="${roll} ${pitch} ${yaw}"/>
-      <mass value="${mass}"/>
-      <inertia ixx="${(depth*depth + height*height)*mass/12}" ixy="0.0" ixz="0.0"
-               iyy="${(depth*depth + width*width)*mass/12}" iyz="0.0"
-               izz="${(width*width + height*height)*mass/12}"/>
-    </inertial>
-  </xacro:macro>
-  <xacro:macro name="box_geometry" params="width height depth">
-    <geometry>
-      <box size="${width} ${height} ${depth}"/>
-    </geometry>
-  </xacro:macro>
-  <xacro:macro name="box_collision" params="width height depth">
-    <collision>
-      <xacro:box_geometry width="${width}" height="${height}" depth="${depth}"/>
-    </collision>
-  </xacro:macro>
+    <xacro:macro name="sphere_inertia" params="mass radius">
+        <inertial>
+            <mass value="${mass}"/>
+            <origin xyz="0 0 0"/>
+            <inertia ixx="${2*mass*radius*radius/5}" ixy="0.0" ixz="0.0"
+                     iyy="${2*mass*radius*radius/5}" iyz="0.0"
+                     izz="${2*mass*radius*radius/5}"/>
+        </inertial>
+    </xacro:macro>
+    <xacro:macro name="sphere_inertia_gazebo" params="mass radius">
+        <inertial>
+            <mass>${mass}</mass>
+            <inertia>
+                <ixx>${2*mass*radius*radius/5}</ixx>
+                <ixy>0</ixy>
+                <iyy>${2*mass*radius*radius/5}</iyy>
+                <ixz>0</ixz>
+                <iyz>0</iyz>
+                <izz>${2*mass*radius*radius/5}</izz>
+            </inertia>
+        </inertial>
+    </xacro:macro>
+    <xacro:macro name="sphere_geometry" params="radius">
+        <geometry>
+            <sphere radius="${radius}"/>
+        </geometry>
+    </xacro:macro>
+    <xacro:macro name="sphere_geometry_gazebo" params="radius">
+        <geometry>
+            <sphere>
+                <radius>${radius}</radius>
+            </sphere>
+        </geometry>
+    </xacro:macro>
+    <xacro:macro name="sphere_collision" params="radius">
+        <collision>
+            <xacro:sphere_geometry radius="${radius}"/>
+        </collision>
+    </xacro:macro>
+    <xacro:macro name="cylinder_inertia" params="mass radius height">
+        <inertial>
+            <mass value="${mass}"/>
+            <origin xyz="0 0 0"/>
+            <inertia ixx="${(3*radius*radius + height*height)*mass/12}" ixy="0.0" ixz="0.0"
+                     iyy="${(3*radius*radius + height*height)*mass/12}" iyz="0.0"
+                     izz="${radius*radius*mass/2}"/>
+        </inertial>
+    </xacro:macro>
+    <xacro:macro name="cylinder_geometry" params="radius height">
+        <geometry>
+            <cylinder length="${height}" radius="${radius}"/>
+        </geometry>
+    </xacro:macro>
+    <xacro:macro name="cylinder_collision" params="radius height">
+        <collision>
+            <xacro:cylinder_geometry radius="${radius}" height="${height}"/>
+        </collision>
+    </xacro:macro>
+    <xacro:macro name="box_inertia" params="mass width height depth x:=0 y:=0 z:=0 roll:=0 pitch:=0 yaw:=0">
+        <inertial>
+            <origin xyz="${x} ${y} ${z}" rpy="${roll} ${pitch} ${yaw}"/>
+            <mass value="${mass}"/>
+            <inertia ixx="${(depth*depth + height*height)*mass/12}" ixy="0.0" ixz="0.0"
+                     iyy="${(depth*depth + width*width  )*mass/12}" iyz="0.0"
+                     izz="${(width*width + height*height)*mass/12}"/>
+        </inertial>
+    </xacro:macro>
+    <xacro:macro name="box_geometry" params="width height depth">
+        <geometry>
+            <box size="${width} ${height} ${depth}"/>
+        </geometry>
+    </xacro:macro>
+    <xacro:macro name="box_collision" params="width height depth">
+        <collision>
+            <xacro:box_geometry width="${width}" height="${height}" depth="${depth}"/>
+        </collision>
+    </xacro:macro>
 </robot>

File: leobot_description/urdf/materials.urdf.xacro (robot description, xacro)
@@ -1,34 +1,33 @@
-<?xml version="1.0"?>
 <robot xmlns:xacro="http://ros.org/wiki/xacro">
-  <xacro:macro name="white_material">
-    <material name="white">
-      <color rgba="1.0 1.0 1.0 1.0"/>
-    </material>
-  </xacro:macro>
-  <xacro:macro name="black_material">
-    <material name="black">
-      <color rgba="0.0 0.0 0.0 1.0"/>
-    </material>
-  </xacro:macro>
-  <xacro:macro name="navajo_white_material">
-    <material name="navajo_white">
-      <color rgba="1.0 0.87 0.68 1.0"/>
-    </material>
-  </xacro:macro>
-  <xacro:macro name="red_material">
-    <material name="red">
-      <color rgba="1.0 0.0 0.0 1.0"/>
-    </material>
-  </xacro:macro>
-  <xacro:macro name="green_material">
-    <material name="green">
-      <color rgba="0.0 1.0 0.0 1.0"/>
-    </material>
-  </xacro:macro>
-  <xacro:macro name="blue_material">
-    <material name="blue">
-      <color rgba="0.0 0.0 1.0 1.0"/>
-    </material>
-  </xacro:macro>
+    <xacro:macro name="white_material">
+        <material name="white">
+            <color rgba="1.0 1.0 1.0 1.0"/>
+        </material>
+    </xacro:macro>
+    <xacro:macro name="black_material">
+        <material name="black">
+            <color rgba="0.0 0.0 0.0 1.0"/>
+        </material>
+    </xacro:macro>
+    <xacro:macro name="navajo_white_material">
+        <material name="navajo_white">
+            <color rgba="1.0 0.87 0.68 1.0"/>
+        </material>
+    </xacro:macro>
+    <xacro:macro name="red_material">
+        <material name="red">
+            <color rgba="1.0 0.0 0.0 1.0"/>
+        </material>
+    </xacro:macro>
+    <xacro:macro name="green_material">
+        <material name="green">
+            <color rgba="0.0 1.0 0.0 1.0"/>
+        </material>
+    </xacro:macro>
+    <xacro:macro name="blue_material">
+        <material name="blue">
+            <color rgba="0.0 0.0 1.0 1.0"/>
+        </material>
+    </xacro:macro>
     <xacro:macro name="yellow_material">
         <material name="yellow">

File: leobot_description/urdf/sensors/camera.urdf.xacro (robot description, xacro)
@@ -1,3 +1,2 @@
-<?xml version="1.0"?>
 <robot xmlns:xacro="http://ros.org/wiki/xacro">
     <xacro:property name="camera_radius" value="0.025"/>

File: leobot_description/urdf/sensors/hokuyo.urdf.xacro (robot description, xacro)
@@ -1,7 +1,6 @@
-<?xml version="1.0"?>
 <robot xmlns:xacro="http://ros.org/wiki/xacro">
     <xacro:property name="hokuyo_radius" value="0.05"/>
     <xacro:property name="hokuyo_height" value="0.05"/>
-    <xacro:property name="hokuyo_mass" value="0.2"/>
+    <xacro:property name="hokuyo_mass"   value="0.2"/>
     <xacro:macro name="lidar_hokuyo" params="parent_link_name parent_height">
         <link name="laser_link">

File: leobot_description/urdf/wheels.urdf.xacro (robot description, xacro)
@@ -1,10 +1,9 @@
-<?xml version="1.0"?>
 <robot xmlns:xacro="http://ros.org/wiki/xacro">
     <xacro:property name="motor_holder_radius" value="0.02"/>
     <xacro:property name="motor_holder_height" value="0.1"/>
-    <xacro:property name="motor_holder_mass" value="0.8"/>
+    <xacro:property name="motor_holder_mass"   value="0.8"/>
     <xacro:property name="mecanum_radius" value="0.1"/>
     <xacro:property name="mecanum_height" value="0.1"/>
-    <xacro:property name="mecanum_mass" value="0.3"/>
+    <xacro:property name="mecanum_mass"   value="0.3"/>
     <xacro:macro name="mecanum_wheel"
                  params="prefix wheel_type side position parent_length parent_height parent_width">
@@ -15,5 +14,5 @@
             </visual>
             <xacro:cylinder_collision radius="${motor_holder_radius}" height="${motor_holder_height}"/>
-            <xacro:cylinder_inertia mass="${motor_holder_mass}" radius="${motor_holder_radius}" height="${motor_holder_height}"/>
+            <xacro:cylinder_inertia   radius="${motor_holder_radius}" height="${motor_holder_height}" mass="${motor_holder_mass}"/>
         </link>
         <joint name="${prefix}_motor_holder_base_joint" type="fixed">
@@ -25,5 +24,5 @@
         <link name="${prefix}_wheel_link">
             <visual>
-                <origin rpy="0 0 0 " xyz="${-mecanum_radius*1.05} ${-mecanum_radius} ${-mecanum_height*0.75}"/>
+                <origin rpy="0 0 0" xyz="${-mecanum_radius*1.05} ${-mecanum_radius} ${-mecanum_height*0.75}"/>
                 <geometry>
                     <mesh filename="package://leobot_description/meshes/Mecanum_Wheel_${wheel_type}.STL" scale="0.0015 0.0015 0.0015"/>
@@ -31,8 +30,8 @@
             </visual>
             <xacro:cylinder_collision radius="${mecanum_radius}" height="${mecanum_height}"/>
-            <xacro:cylinder_inertia mass="${mecanum_mass}" radius="${mecanum_radius}" height="${mecanum_height}"/>
+            <xacro:cylinder_inertia   radius="${mecanum_radius}" height="${mecanum_height}" mass="${mecanum_mass}"/>
         </link>
         <joint name="${prefix}_wheel_motor_joint" type="continuous">
-            <origin rpy="0 0 0" xyz="0 0 ${ -1 * side * motor_holder_height/2}"/>
+            <origin rpy="0 0 0" xyz="0 0 ${-1 * side * motor_holder_height/2}"/>
             <parent link="${prefix}_motor_holder"/>
             <child link="${prefix}_wheel_link"/>

Commit message: Attempt to add a camera_position_controller
For task #136: Add position controller for head link

File: leobot_description/robot/robot.urdf.xacro (robot description, xacro)
@@ -69,4 +69,14 @@
     <child link="camera_stick_link"/>
   </joint>
+  <transmission name="camera_transmission">
+    <type>transmission_interface/SimpleTransmission</type>
+    <joint name="head_camera_stick_joint">
+      <hardwareInterface>hardware_interface/EffortJointInterface</hardwareInterface>
+    </joint>
+    <actuator name="camera_motor">
+      <hardwareInterface>EffortJointInterface</hardwareInterface>
+      <mechanicalReduction>1</mechanicalReduction>
+    </actuator>
+  </transmission>
   <xacro:fish_camera prefix="left"  parent_link_name="camera_stick_link" parent_height="${camera_stick_height}" parent_width="${camera_stick_width}" side="1"/>
   <xacro:fish_camera prefix="right" parent_link_name="camera_stick_link" parent_height="${camera_stick_height}" parent_width="${camera_stick_width}" side="-1"/>
