Commit message: Add the head transmission to fix the issue with head controller initialization
For task: F#136 head controller #139

File: leobot_description/robot/robot.urdf.xacro (robot description, xacro)
@@ -69,4 +69,11 @@
         <child link="camera_stick_link"/>
     </joint>
+    <transmission name="head_transmission">
+        <type>transmission_interface/SimpleTransmission</type>
+        <joint name="head_camera_stick_joint">
+            <hardwareInterface>EffortJointInterface</hardwareInterface>
+        </joint>
+        <actuator name="head_motor"/>
+    </transmission>
     <xacro:fish_camera prefix="left"  parent_link_name="camera_stick_link" parent_height="${camera_stick_height}" parent_width="${camera_stick_width}" side="1"/>
     <xacro:fish_camera prefix="right" parent_link_name="camera_stick_link" parent_height="${camera_stick_height}" parent_width="${camera_stick_width}" side="-1"/>

Commit message: Fixed naming convention for boxes widht, length and height.

File: leobot_description/robot/robot.urdf.xacro (robot description, xacro)
@@ -6,6 +6,6 @@
     <xacro:include filename="$(find leobot_description)/urdf/wheels.urdf.xacro"/>
     <xacro:property name="base_width"  value="0.54"/>
-    <xacro:property name="base_length" value="0.3"/>
-    <xacro:property name="base_height" value="0.5"/>
+    <xacro:property name="base_length" value="0.5"/>
+    <xacro:property name="base_height" value="0.3"/>
     <xacro:property name="base_mass"   value="10"/>
     <xacro:property name="neck_width"  value="0.04"/>
@@ -13,30 +13,30 @@
     <xacro:property name="neck_height" value="1.45"/>
     <xacro:property name="neck_mass"   value="1.0"/>
-    <xacro:property name="head_width"  value="0.04"/>
+    <xacro:property name="head_width"  value="0.29"/>
     <xacro:property name="head_length" value="0.04"/>
-    <xacro:property name="head_height" value="0.29"/>
+    <xacro:property name="head_height" value="0.04"/>
     <xacro:property name="head_mass"   value="0.5"/>
-    <xacro:property name="camera_stick_width"  value="0.02"/>
-    <xacro:property name="camera_stick_length" value="0.04"/>
-    <xacro:property name="camera_stick_height" value="0.1"/>
+    <xacro:property name="camera_stick_width"  value="0.04"/>
+    <xacro:property name="camera_stick_length" value="0.1"/>
+    <xacro:property name="camera_stick_height" value="0.02"/>
     <xacro:property name="camera_stick_mass"   value="0.2"/>
     <link name="base_link">
         <visual>
-            <xacro:box_geometry width="${base_width}" height="${base_height}" depth="${base_length}"/>
+            <xacro:box_geometry width="${base_width}" length="${base_length}" height="${base_height}"/>
             <xacro:green_material/>
         </visual>
-        <xacro:box_collision width="${base_width}" height="${base_height}" depth="${base_length}"/>
-        <xacro:box_inertia   width="${base_width}" height="${base_height}" depth="${base_length}" mass="${base_mass}"/>
+        <xacro:box_collision width="${base_width}" length="${base_length}" height="${base_height}"/>
+        <xacro:box_inertia   width="${base_width}" length="${base_length}" height="${base_height}" mass="${base_mass}"/>
     </link>
     <link name="neck_link">
         <visual>
-            <xacro:box_geometry width="${neck_width}" height="${neck_height}" depth="${neck_length}"/>
+            <xacro:box_geometry width="${neck_width}" length="${neck_length}" height="${neck_height}"/>
             <xacro:red_material/>
         </visual>
-        <xacro:box_collision width="${neck_width}" height="${neck_height}" depth="${neck_length}"/>
-        <xacro:box_inertia   width="${neck_width}" height="${neck_height}" depth="${neck_length}" mass="${head_mass}"/>
+        <xacro:box_collision width="${neck_width}" length="${neck_length}" height="${neck_height}"/>
+        <xacro:box_inertia   width="${neck_width}" length="${neck_length}" height="${neck_height}" mass="${head_mass}"/>
     </link>
     <joint name="base_neck_joint" type="fixed">
-        <origin rpy="${pi/2} 0 0" xyz="${-base_height/2 - neck_width} 0 ${-base_length/2 + neck_height / 2 }"/>
+        <origin rpy="0 0 0" xyz="${-(base_width + neck_width) / 2} 0 ${(neck_height - base_height) / 2 }"/>
         <parent link="base_link"/>
         <child link="neck_link"/>
@@ -44,12 +44,12 @@
     <link name="head_link">
         <visual>
-            <xacro:box_geometry width="${head_width}" height="${head_height}" depth="${head_length}"/>
+            <xacro:box_geometry width="${head_width}" length="${head_length}" height="${head_height}"/>
             <xacro:blue_material/>
         </visual>
-        <xacro:box_collision width="${head_width}" height="${head_height}" depth="${head_length}"/>
-        <xacro:box_inertia   width="${head_width}" height="${head_height}" depth="${head_length}" mass="${head_mass}"/>
+        <xacro:box_collision width="${head_width}" length="${head_length}" height="${head_height}"/>
+        <xacro:box_inertia   width="${head_width}" length="${head_length}" height="${head_height}" mass="${head_mass}"/>
     </link>
     <joint name="neck_head_joint" type="fixed">
-        <origin rpy="${pi/2} ${pi/2} ${pi}" xyz="${-neck_length/2 + head_height/2} ${neck_height/2 + head_width/2} 0"/>
+        <origin rpy="0 0 0" xyz="${(head_width - neck_width) / 2} 0 ${(neck_height + head_height) / 2}"/>
         <parent link="neck_link"/>
         <child link="head_link"/>
@@ -57,16 +57,17 @@
     <link name="camera_stick_link">
         <visual>
-            <xacro:box_geometry width="${camera_stick_width}" height="${camera_stick_height}"
-                                depth="${camera_stick_length}"/>
+            <xacro:box_geometry width="${camera_stick_width}" length="${camera_stick_length}"
+                                height="${camera_stick_height}"/>
             <xacro:yellow_material/>
         </visual>
-        <xacro:box_collision width="${camera_stick_width}" height="${camera_stick_height}"
-                             depth="${camera_stick_length}"/>
-        <xacro:box_inertia   width="${camera_stick_width}" height="${camera_stick_height}"
-                             depth="${camera_stick_length}" mass="${camera_stick_mass}"/>
+        <xacro:box_collision width="${camera_stick_width}" length="${camera_stick_length}"
+                             height="${camera_stick_height}"/>
+        <xacro:box_inertia width="${camera_stick_width}" length="${camera_stick_length}"
+                           height="${camera_stick_height}" mass="${camera_stick_mass}"/>
     </link>
     <joint name="head_camera_stick_joint" type="revolute">
-        <origin rpy="${pi/2} ${pi/2} ${pi}"
-                xyz="0 ${camera_stick_length/2 - head_height/2} ${head_width/2 + camera_stick_width/2}"/>
+        <origin rpy="0 0 0"
+                xyz="${(head_width - camera_stick_width) / 2} 0 ${(head_height + camera_stick_height) / 2}"/>
+        <axis xyz="0 0 1"/>
         <parent link="head_link"/>
         <child link="camera_stick_link"/>
@@ -84,15 +85,15 @@
     </transmission>
     <xacro:simple_camera prefix="left"  parent_link_name="camera_stick_link" parent_height="${camera_stick_height}"
-                  parent_width="${camera_stick_width}" side="1"/>
+                  parent_length="${camera_stick_length}" side="1"/>
     <xacro:simple_camera prefix="right" parent_link_name="camera_stick_link" parent_height="${camera_stick_height}"
-                  parent_width="${camera_stick_width}" side="-1"/>
-    <xacro:lidar_hokuyo parent_link_name="base_link" parent_height="${base_length}"/>
-    <xacro:mecanum_wheel prefix="FL" wheel_type="2" side="1"  position="1"  parent_length="${base_width}"
-                         parent_height="${base_length}" parent_width="${base_height}"/>
-    <xacro:mecanum_wheel prefix="FR" wheel_type="1" side="-1" position="1"  parent_length="${base_width}"
-                         parent_height="${base_length}" parent_width="${base_height}"/>
-    <xacro:mecanum_wheel prefix="RL" wheel_type="1" side="1"  position="-1" parent_length="${base_width}"
-                         parent_height="${base_length}" parent_width="${base_height}"/>
-    <xacro:mecanum_wheel prefix="RR" wheel_type="2" side="-1" position="-1" parent_length="${base_width}"
-                         parent_height="${base_length}" parent_width="${base_height}"/>
+                  parent_length="${camera_stick_length}" side="-1"/>
+    <xacro:lidar_hokuyo parent_link_name="base_link" parent_height="${base_height}"/>
+    <xacro:mecanum_wheel prefix="FL" wheel_type="2" side="1" position="1" parent_length="${base_length}"
+                         parent_height="${base_height}" parent_width="${base_width}"/>
+    <xacro:mecanum_wheel prefix="FR" wheel_type="1" side="-1" position="1" parent_length="${base_length}"
+                         parent_height="${base_height}" parent_width="${base_width}"/>
+    <xacro:mecanum_wheel prefix="RL" wheel_type="1" side="1" position="-1" parent_length="${base_length}"
+                         parent_height="${base_height}" parent_width="${base_width}"/>
+    <xacro:mecanum_wheel prefix="RR" wheel_type="2" side="-1" position="-1" parent_length="${base_length}"
+                         parent_height="${base_height}" parent_width="${base_width}"/>
 </robot>

File: leobot_description/urdf/common.urdf.xacro (robot description, xacro)
@@ -58,21 +58,28 @@
         </collision>
     </xacro:macro>
-    <xacro:macro name="box_inertia" params="mass width height depth x:=0 y:=0 z:=0 roll:=0 pitch:=0 yaw:=0">
+    <xacro:macro name="box_inertia" params="mass width length height x:=0 y:=0 z:=0 roll:=0 pitch:=0 yaw:=0">
         <inertial>
             <origin xyz="${x} ${y} ${z}" rpy="${roll} ${pitch} ${yaw}"/>
             <mass value="${mass}"/>
-            <inertia ixx="${(depth*depth + height*height)*mass/12}" ixy="0.0" ixz="0.0"
-                     iyy="${(depth*depth + width*width  )*mass/12}" iyz="0.0"
-                     izz="${(width*width + height*height)*mass/12}"/>
+            <inertia ixx="${(height*height + length*length)*mass/12}" ixy="0.0" ixz="0.0"
+                     iyy="${(height*height + width*width  )*mass/12}" iyz="0.0"
+                     izz="${(width*width + length*length)*mass/12}"/>
         </inertial>
     </xacro:macro>
-    <xacro:macro name="box_geometry" params="width height depth">
+    <!-- Box dimensions approach:
+         X axis is facing towards observer
+         Y axis is in the horizontal plane with X axis
+         Z axis is vertical
+         Length is dimension along Y axis
+         Width is along X axis
+         Height is along Z axis -->
+    <xacro:macro name="box_geometry" params="width length height">
         <geometry>
-            <box size="${width} ${height} ${depth}"/>
+            <box size="${width} ${length} ${height}"/>
         </geometry>
     </xacro:macro>
-    <xacro:macro name="box_collision" params="width height depth">
+    <xacro:macro name="box_collision" params="width length height">
         <collision>
-            <xacro:box_geometry width="${width}" height="${height}" depth="${depth}"/>
+            <xacro:box_geometry width="${width}" length="${length}" height="${height}"/>
         </collision>
     </xacro:macro>

File: leobot_description/urdf/sensors/camera.urdf.xacro (robot description, xacro)
@@ -3,5 +3,5 @@
     <xacro:property name="camera_size" value="0.03"/>
     <xacro:property name="camera_mass"   value="0.1"/>
-    <xacro:macro name="fish_camera" params="prefix parent_link_name parent_height side parent_width">
+    <xacro:macro name="fish_camera" params="prefix parent_link_name parent_length parent_height side">
         <link name="${prefix}_camera_link">
             <visual>
@@ -13,23 +13,23 @@
         </link>
         <joint name="${prefix}_camera_joint" type="fixed">
-            <origin xyz="${-camera_radius - parent_width/2} ${side*(parent_height/2 - camera_radius/2)} 0"
-                    rpy="${pi/2 + side * pi/2} ${pi/2 + side * pi/2} 0"/>
+            <origin xyz="0 ${side * parent_length / 2} ${(parent_height + camera_radius) / 2}"
+                    rpy="0 0 0"/>
             <parent link="${parent_link_name}"/>
             <child link="${prefix}_camera_link"/>
         </joint>
     </xacro:macro>
-    <xacro:macro name="simple_camera" params="prefix parent_link_name parent_height side parent_width">
+    <xacro:macro name="simple_camera" params="prefix parent_link_name parent_length parent_height side">
         <link name="${prefix}_camera_link">
             <visual>
-              <xacro:box_geometry width="${camera_size}" height="${camera_size}" depth="${camera_size}"/>
+              <xacro:box_geometry width="${camera_size}" length="${camera_size}" height="${camera_size}"/>
               <xacro:green_material/>
             </visual>
-            <xacro:box_collision width="${camera_size}" height="${camera_size}" depth="${camera_size}"/>
-            <xacro:box_inertia mass="${camera_mass}" width="${camera_size}" height="${camera_size}"
-                               depth="${camera_size}"/>
+            <xacro:box_collision width="${camera_size}" length="${camera_size}" height="${camera_size}"/>
+            <xacro:box_inertia mass="${camera_mass}" width="${camera_size}" length="${camera_size}"
+                               height="${camera_size}"/>
         </link>
         <joint name="${prefix}_camera_joint" type="fixed">
-            <origin xyz="${(-camera_size - parent_width) / 2} ${side * (parent_height - camera_size / 2) / 2} 0"
-                    rpy="${-pi / 2} ${pi / 2} ${pi / 2}"/>
+            <origin xyz="0 ${side * parent_length / 2} ${(parent_height + camera_size) / 2}"
+                    rpy="0 0 0"/>
             <parent link="${parent_link_name}"/>
             <child link="${prefix}_camera_link"/>

File: leobot_description/urdf/wheels.urdf.xacro (robot description, xacro)
@@ -7,5 +7,5 @@
     <xacro:property name="mecanum_mass"   value="0.3"/>
     <xacro:macro name="mecanum_wheel"
-                 params="prefix wheel_type side position parent_length parent_height parent_width">
+                 params="prefix wheel_type side position parent_width parent_length parent_height">
         <link name="${prefix}_motor_holder">
             <visual>
@@ -18,5 +18,5 @@
         <joint name="${prefix}_motor_holder_base_joint" type="fixed">
             <origin rpy="${pi/2} 0 0"
-                    xyz="${position * (parent_length/2 - motor_holder_radius*2)} ${side * (parent_width/2 + motor_holder_height/2)} ${(-parent_height/2 + motor_holder_radius*2)}"/>
+                    xyz="${position * (parent_width/2 - motor_holder_radius*2)} ${side * (parent_length/2 + motor_holder_height/2)} ${(-parent_height/2 + motor_holder_radius*2)}"/>
             <parent link="base_link"/>
             <child link="${prefix}_motor_holder"/>
