Commit message: Added simple stereo camera to simulation

File: leobot_description/robot/leobot.gazebo.xacro (robot description, xacro)
@@ -15,3 +15,94 @@
     <material>Gazebo/White</material>
   </gazebo>
+  <gazebo reference="camera_left_link">
+    <sensor type="camera" name="camera_left">
+      <update_rate>30.0</update_rate>
+      <camera name="left">
+        <horizontal_fov>1.3962634</horizontal_fov>
+        <image>
+          <width>800</width>
+          <height>800</height>
+          <format>R8G8B8</format>
+        </image>
+        <clip>
+          <near>0.02</near>
+          <far>300</far>
+        </clip>
+        <noise>
+          <type>gaussian</type>
+          <mean>0.0</mean>
+          <stddev>0.007</stddev>
+        </noise>
+      </camera>
+      <plugin name="camera_controller" filename="libgazebo_ros_camera.so">
+        <alwaysOn>true</alwaysOn>
+        <updateRate>0.0</updateRate>
+        <cameraName>leobot/camera1</cameraName>
+        <imageTopicName>image_raw</imageTopicName>
+        <cameraInfoTopicName>camera_info</cameraInfoTopicName>
+        <frameName>camera_left_link</frameName>
+        <hackBaseline>0.07</hackBaseline>
+        <distortionK1>0.0</distortionK1>
+        <distortionK2>0.0</distortionK2>
+        <distortionK3>0.0</distortionK3>
+        <distortionT1>0.0</distortionT1>
+        <distortionT2>0.0</distortionT2>
+      </plugin>
+    </sensor>
+  </gazebo>
+  <!--<gazebo reference="camera_left_link">-->
+    <!--<sensor type="multicamera" name="stereo_camera">-->
+      <!--<update_rate>30.0</update_rate>-->
+      <!--<camera name="left">-->
+        <!--<horizontal_fov>1.3962634</horizontal_fov>-->
+        <!--<image>-->
+          <!--<width>800</width>-->
+          <!--<height>800</height>-->
+          <!--<format>R8G8B8</format>-->
+        <!--</image>-->
+        <!--<clip>-->
+          <!--<near>0.02</near>-->
+          <!--<far>300</far>-->
+        <!--</clip>-->
+        <!--<noise>-->
+          <!--<type>gaussian</type>-->
+          <!--<mean>0.0</mean>-->
+          <!--<stddev>0.007</stddev>-->
+        <!--</noise>-->
+      <!--</camera>-->
+      <!--<camera name="right">-->
+        <!--<pose>0 -0.07 0 0 0 0</pose>-->
+        <!--<horizontal_fov>1.3962634</horizontal_fov>-->
+        <!--<image>-->
+          <!--<width>800</width>-->
+          <!--<height>800</height>-->
+          <!--<format>R8G8B8</format>-->
+        <!--</image>-->
+        <!--<clip>-->
+          <!--<near>0.02</near>-->
+          <!--<far>300</far>-->
+        <!--</clip>-->
+        <!--<noise>-->
+          <!--<type>gaussian</type>-->
+          <!--<mean>0.0</mean>-->
+          <!--<stddev>0.007</stddev>-->
+        <!--</noise>-->
+      <!--</camera>-->
+      <!--<plugin name="stereo_camera_controller" filename="libgazebo_ros_multicamera.so">-->
+        <!--<alwaysOn>true</alwaysOn>-->
+        <!--<updateRate>0.0</updateRate>-->
+        <!--<cameraName>leobot/stereocamera</cameraName>-->
+        <!--<imageTopicName>image_raw</imageTopicName>-->
+        <!--<cameraInfoTopicName>camera_info</cameraInfoTopicName>-->
+        <!--<frameName>camera_left_link</frameName>-->
+        <!--<rightFrameName>camera_right_link</rightFrameName>-->
+        <!--<hackBaseline>0.07</hackBaseline>-->
+        <!--<distortionK1>0.0</distortionK1>-->
+        <!--<distortionK2>0.0</distortionK2>-->
+        <!--<distortionK3>0.0</distortionK3>-->
+        <!--<distortionT1>0.0</distortionT1>-->
+        <!--<distortionT2>0.0</distortionT2>-->
+      <!--</plugin>-->
+    <!--</sensor>-->
+  <!--</gazebo>-->
 </robot>

File: leobot_description/robot/robot.urdf.xacro (robot description, xacro)
@@ -13,3 +13,29 @@
     <xacro:cylinder_inertia mass="10" radius="0.25" height="1.0"/>
   </link>
+  <link name="camera_left_link">
+    <visual>
+      <xacro:box_geometry width="0.05" height="0.05" depth="0.05"/>
+      <xacro:green_material/>
+    </visual>
+    <xacro:box_collision width="0.05" height="0.05" depth="0.05"/>
+    <xacro:box_inertia mass="0.1" width="0.05" height="0.05" depth="0.05"/>
+  </link>
+  <joint name="camera_left_link_joint" type="fixed">
+    <origin rpy="0 0 0" xyz="0 0.075 0.525"/>
+    <parent link="base_link"/>
+    <child link="camera_left_link"/>
+  </joint>
+  <link name="camera_right_link">
+    <visual>
+      <xacro:box_geometry width="0.05" height="0.05" depth="0.05"/>
+      <xacro:green_material/>
+    </visual>
+    <xacro:box_collision width="0.05" height="0.05" depth="0.05"/>
+    <xacro:box_inertia mass="0.1" width="0.05" height="0.05" depth="0.05"/>
+  </link>
+  <joint name="camera_right_link_joint" type="fixed">
+    <origin rpy="0 0 0" xyz="0 -0.075 0.525"/>
+    <parent link="base_link"/>
+    <child link="camera_right_link"/>
+  </joint>
 </robot>

Commit message: Added stereo camera to simulation

File: leobot_description/robot/leobot.gazebo.xacro (robot description, xacro)
@@ -16,5 +16,6 @@
   </gazebo>
   <gazebo reference="camera_left_link">
-    <sensor type="camera" name="camera_left">
+    <material>Gazebo/Green</material>
+    <sensor type="multicamera" name="stereo_camera">
       <update_rate>30.0</update_rate>
       <camera name="left">
@@ -35,11 +36,30 @@
         </noise>
       </camera>
-      <plugin name="camera_controller" filename="libgazebo_ros_camera.so">
+      <camera name="right">
+        <pose>0 -0.07 0 0 0 0</pose>
+        <horizontal_fov>1.3962634</horizontal_fov>
+        <image>
+          <width>800</width>
+          <height>800</height>
+          <format>R8G8B8</format>
+        </image>
+        <clip>
+          <near>0.02</near>
+          <far>300</far>
+        </clip>
+        <noise>
+          <type>gaussian</type>
+          <mean>0.0</mean>
+          <stddev>0.007</stddev>
+        </noise>
+      </camera>
+      <plugin name="stereo_camera_controller" filename="libgazebo_ros_multicamera.so">
         <alwaysOn>true</alwaysOn>
         <updateRate>0.0</updateRate>
-        <cameraName>leobot/camera1</cameraName>
+        <cameraName>leobot/stereocamera</cameraName>
         <imageTopicName>image_raw</imageTopicName>
         <cameraInfoTopicName>camera_info</cameraInfoTopicName>
         <frameName>camera_left_link</frameName>
+        <rightFrameName>camera_right_link</rightFrameName>
         <hackBaseline>0.07</hackBaseline>
         <distortionK1>0.0</distortionK1>
@@ -51,58 +71,6 @@
     </sensor>
   </gazebo>
-  <!--<gazebo reference="camera_left_link">-->
-    <!--<sensor type="multicamera" name="stereo_camera">-->
-      <!--<update_rate>30.0</update_rate>-->
-      <!--<camera name="left">-->
-        <!--<horizontal_fov>1.3962634</horizontal_fov>-->
-        <!--<image>-->
-          <!--<width>800</width>-->
-          <!--<height>800</height>-->
-          <!--<format>R8G8B8</format>-->
-        <!--</image>-->
-        <!--<clip>-->
-          <!--<near>0.02</near>-->
-          <!--<far>300</far>-->
-        <!--</clip>-->
-        <!--<noise>-->
-          <!--<type>gaussian</type>-->
-          <!--<mean>0.0</mean>-->
-          <!--<stddev>0.007</stddev>-->
-        <!--</noise>-->
-      <!--</camera>-->
-      <!--<camera name="right">-->
-        <!--<pose>0 -0.07 0 0 0 0</pose>-->
-        <!--<horizontal_fov>1.3962634</horizontal_fov>-->
-        <!--<image>-->
-          <!--<width>800</width>-->
-          <!--<height>800</height>-->
-          <!--<format>R8G8B8</format>-->
-        <!--</image>-->
-        <!--<clip>-->
-          <!--<near>0.02</near>-->
-          <!--<far>300</far>-->
-        <!--</clip>-->
-        <!--<noise>-->
-          <!--<type>gaussian</type>-->
-          <!--<mean>0.0</mean>-->
-          <!--<stddev>0.007</stddev>-->
-        <!--</noise>-->
-      <!--</camera>-->
-      <!--<plugin name="stereo_camera_controller" filename="libgazebo_ros_multicamera.so">-->
-        <!--<alwaysOn>true</alwaysOn>-->
-        <!--<updateRate>0.0</updateRate>-->
-        <!--<cameraName>leobot/stereocamera</cameraName>-->
-        <!--<imageTopicName>image_raw</imageTopicName>-->
-        <!--<cameraInfoTopicName>camera_info</cameraInfoTopicName>-->
-        <!--<frameName>camera_left_link</frameName>-->
-        <!--<rightFrameName>camera_right_link</rightFrameName>-->
-        <!--<hackBaseline>0.07</hackBaseline>-->
-        <!--<distortionK1>0.0</distortionK1>-->
-        <!--<distortionK2>0.0</distortionK2>-->
-        <!--<distortionK3>0.0</distortionK3>-->
-        <!--<distortionT1>0.0</distortionT1>-->
-        <!--<distortionT2>0.0</distortionT2>-->
-      <!--</plugin>-->
-    <!--</sensor>-->
-  <!--</gazebo>-->
+  <gazebo reference="camera_right_link">
+    <material>Gazebo/Green</material>
+  </gazebo>
 </robot>

Commit message: LeoBotUrdf

File: leobot_description/robot/leobot.gazebo.xacro (robot description, xacro)
@@ -8,5 +8,5 @@
     </plugin>
   </gazebo>
-  <gazebo reference="base_link">
+  <gazebo reference="body_link">
     <mu1 value="1.0"/>
     <mu2 value="1.0"/>
@@ -15,5 +15,39 @@
     <material>Gazebo/White</material>
   </gazebo>
-<!--
+  <gazebo reference="head_link">
+    <mu1 value="1.0"/>
+    <mu2 value="1.0"/>
+    <kp value="10000000.0"/>
+    <kd value="1.0"/>
+    <material>Gazebo/Black</material>
+  </gazebo>
+   <gazebo reference="tail_link">
+    <mu1 value="1.0"/>
+    <mu2 value="1.0"/>
+    <kp value="10000000.0"/>
+    <kd value="1.0"/>
+    <material>Gazebo/Black</material>
+  </gazebo>
+   <gazebo reference="left_wheel_link">
+    <mu1 value="1.0"/>
+    <mu2 value="1.0"/>
+    <kp value="10000000.0"/>
+    <kd value="1.0"/>
+    <material>Gazebo/White</material>
+  </gazebo>
+   <gazebo reference="right_wheel_link">
+    <mu1 value="1.0"/>
+    <mu2 value="1.0"/>
+    <kp value="10000000.0"/>
+    <kd value="1.0"/>
+    <material>Gazebo/White</material>
+  </gazebo>
+     <gazebo reference="caster_wheel_link">
+    <mu1 value="0.0"/>
+    <mu2 value="0.0"/>
+    <kp value="10000000.0"/>
+    <kd value="1.0"/>
+    <material>Gazebo/Red</material>
+  </gazebo>
   <gazebo reference="camera_left_link">
     <material>Gazebo/Green</material>
@@ -75,4 +109,3 @@
     <material>Gazebo/Green</material>
   </gazebo>
--->
 </robot>

File: leobot_description/robot/robot.urdf.xacro (robot description, xacro)
@@ -4,14 +4,88 @@
   <xacro:include filename="$(find leobot_description)/urdf/materials.urdf.xacro"/>
   <xacro:include filename="$(find leobot_description)/urdf/common.urdf.xacro"/>
-  <!-- Robot links -->
-  <link name="base_link">
+  <!-- Loebody -->
+  <link name="body_link">
     <visual>
-      <xacro:cylinder_geometry radius="0.25" height="1.0"/>
+      <xacro:cylinder_geometry radius="0.3" height="0.1"/>
       <xacro:navajo_white_material/>
     </visual>
-    <xacro:cylinder_collision radius="0.25" height="1.0"/>
-    <xacro:cylinder_inertia mass="10" radius="0.25" height="1.0"/>
+    <xacro:cylinder_collision radius="0.3" height="0.1"/>
+    <xacro:cylinder_inertia mass="20" radius="0.3" height="0.1"/>
   </link>
-<!--
+  <!-- Leoehead -->
+  <link name="head_link">
+    <visual>
+      <xacro:sphere_geometry radius="0.1"/>
+      <xacro:black_material/>
+    </visual>
+    <xacro:sphere_collision radius="0.25"/>
+    <xacro:sphere_inertia mass="5" radius="0.25"/>
+  </link>
+  <!-- head-body -->
+  <joint name="head_body_joint" type="fixed">
+    <origin rpy="0 0 0" xyz="0.22 0.0 0.12"/>
+    <parent link="body_link"/>
+    <child link="head_link"/>
+  </joint>
+  <!-- Leotail -->
+    <link name="tail_link">
+    <visual>
+      <xacro:cylinder_geometry radius="0.03" height="0.3"/>
+      <xacro:black_material/>
+    </visual>
+    <xacro:cylinder_collision radius="0.03" height="0.3"/>
+    <xacro:cylinder_inertia mass="1" radius="0.03" height="0.3"/>
+  </link>
+  <!-- tail-body -->
+  <joint name="tail_body_joint" type="fixed">
+    <origin rpy="0 -0.55 0" xyz="-0.32 0.0 0.15"/>
+    <parent link="body_link"/>
+    <child link="tail_link"/>
+  </joint>
+   <!-- Leo_left_wheel -->
+    <link name="left_wheel_link">
+    <visual>
+      <xacro:cylinder_geometry radius="0.1" height="0.05"/>
+      <xacro:red_material/>
+    </visual>
+    <xacro:cylinder_collision radius="0.1" height="0.05"/>
+    <xacro:cylinder_inertia mass="10" radius="0.1" height="0.05"/>
+  </link>
+    <!-- left_wheel-body -->
+  <joint name="left_wheel_body_joint" type="continuous">
+    <origin rpy="1.570795 0 0" xyz="0.0 0.32 -0.05"/>
+    <parent link="body_link"/>
+    <child link="left_wheel_link"/>
+  </joint>
+       <!-- Leo_right_wheel -->
+    <link name="right_wheel_link">
+    <visual>
+      <xacro:cylinder_geometry radius="0.1" height="0.05"/>
+      <xacro:red_material/>
+    </visual>
+    <xacro:cylinder_collision radius="0.1" height="0.05"/>
+    <xacro:cylinder_inertia mass="10" radius="0.1" height="0.05"/>
+  </link>
+      <!-- right_wheel-body -->
+  <joint name="right_wheel_body_joint" type="continuous">
+    <origin rpy="1.570795 0 0" xyz="0.0 -0.32 -0.05"/>
+    <parent link="body_link"/>
+    <child link="right_wheel_link"/>
+  </joint>
+       <!-- Leo_caster_wheel -->
+    <link name="caster_wheel_link">
+    <visual>
+      <xacro:sphere_geometry radius="0.08"/>
+      <xacro:red_material/>
+    </visual>
+    <xacro:sphere_collision radius="0.08"/>
+    <xacro:sphere_inertia mass="1" radius="0.08"/>
+  </link>
+      <!-- left_wheel-body -->
+  <joint name="caster_wheel_body_joint" type="fixed">
+    <origin rpy="0 0 0" xyz="0.2 0.0 -0.08"/>
+    <parent link="body_link"/>
+    <child link="caster_wheel_link"/>
+  </joint>
   <link name="camera_left_link">
     <visual>
@@ -23,6 +97,6 @@
   </link>
   <joint name="camera_left_link_joint" type="fixed">
-    <origin rpy="0 0 0" xyz="0 0.075 0.525"/>
-    <parent link="base_link"/>
+    <origin rpy="0 0 0" xyz="0.075 0.075 0.025"/>
+    <parent link="head_link"/>
     <child link="camera_left_link"/>
   </joint>
@@ -36,8 +110,7 @@
   </link>
   <joint name="camera_right_link_joint" type="fixed">
-    <origin rpy="0 0 0" xyz="0 -0.075 0.525"/>
-    <parent link="base_link"/>
+    <origin rpy="0 0 0" xyz="0.075 -0.075 0.025"/>
+    <parent link="head_link"/>
     <child link="camera_right_link"/>
   </joint>
--->
 </robot>

Commit message: LeoBotUrdf

File: leobot_description/robot/leobot.gazebo.xacro (robot description, xacro)
@@ -14,4 +14,25 @@
     <kd value="1.0"/>
     <material>Gazebo/White</material>
+  </gazebo>
+  <gazebo reference="left_wheel_link">
+    <mu1 value="1.0"/>
+    <mu2 value="1.0"/>
+    <kp value="10000000.0"/>
+    <kd value="1.0"/>
+    <material>Gazebo/White</material>
+  </gazebo>
+   <gazebo reference="right_wheel_link">
+    <mu1 value="1.0"/>
+    <mu2 value="1.0"/>
+    <kp value="10000000.0"/>
+    <kd value="1.0"/>
+    <material>Gazebo/White</material>
+  </gazebo>
+     <gazebo reference="caster_wheel_link">
+    <mu1 value="0.0"/>
+    <mu2 value="0.0"/>
+    <kp value="10000000.0"/>
+    <kd value="1.0"/>
+    <material>Gazebo/Red</material>
   </gazebo>
   <gazebo reference="camera_left_link">

File: leobot_description/robot/robot.urdf.xacro (robot description, xacro)
@@ -13,4 +13,51 @@
     <xacro:cylinder_inertia mass="10" radius="0.25" height="1.0"/>
   </link>
+       <!-- Leo_left_wheel -->
+    <link name="left_wheel_link">
+    <visual>
+      <xacro:cylinder_geometry radius="0.1" height="0.05"/>
+      <xacro:red_material/>
+    </visual>
+    <xacro:cylinder_collision radius="0.1" height="0.05"/>
+    <xacro:cylinder_inertia mass="10" radius="0.1" height="0.05"/>
+  </link>
+    <!-- left_wheel-body -->
+  <joint name="left_wheel_body_joint" type="continuous">
+    <origin rpy="1.570795 0 0" xyz="0.0 0.275 -0.55"/>
+    <parent link="base_link"/>
+    <child link="left_wheel_link"/>
+    <axis xyz="0 0 1" />
+  </joint>
+       <!-- Leo_right_wheel -->
+    <link name="right_wheel_link">
+    <visual>
+      <xacro:cylinder_geometry radius="0.1" height="0.05"/>
+      <xacro:red_material/>
+    </visual>
+    <xacro:cylinder_collision radius="0.1" height="0.05"/>
+    <xacro:cylinder_inertia mass="10" radius="0.1" height="0.05"/>
+  </link>
+      <!-- right_wheel-body -->
+  <joint name="right_wheel_body_joint" type="continuous">
+    <origin rpy="1.570795 0 0" xyz="0.0 -0.275 -0.55"/>
+    <parent link="base_link"/>
+    <child link="right_wheel_link"/>
+    <axis xyz="0 0 1" />
+  </joint>
+       <!-- Leo_caster_wheel -->
+    <link name="caster_wheel_link">
+    <visual>
+      <xacro:sphere_geometry radius="0.08"/>
+      <xacro:red_material/>
+    </visual>
+    <xacro:sphere_collision radius="0.08"/>
+    <xacro:sphere_inertia mass="1" radius="0.08"/>
+  </link>
+      <!-- left_wheel-body -->
+  <joint name="caster_wheel_body_joint" type="fixed">
+    <origin rpy="0 0 0" xyz="0.2 0.0 -0.57"/>
+    <parent link="base_link"/>
+    <child link="caster_wheel_link"/>
+  </joint>
   <link name="camera_left_link">
     <visual>

Commit message: LeoBotUrdf

File: leobot_description/robot/leobot.gazebo.xacro (robot description, xacro)
@@ -20,14 +20,14 @@
     <kp value="10000000.0"/>
     <kd value="1.0"/>
-    <material>Gazebo/White</material>
+    <material>Gazebo/Red</material>
   </gazebo>
-   <gazebo reference="right_wheel_link">
+  <gazebo reference="right_wheel_link">
     <mu1 value="1.0"/>
     <mu2 value="1.0"/>
     <kp value="10000000.0"/>
     <kd value="1.0"/>
-    <material>Gazebo/White</material>
+    <material>Gazebo/Red</material>
   </gazebo>
-     <gazebo reference="caster_wheel_link">
+  <gazebo reference="caster_wheel_link">
     <mu1 value="0.0"/>
     <mu2 value="0.0"/>

File: leobot_description/robot/robot.urdf.xacro (robot description, xacro)
@@ -13,6 +13,5 @@
     <xacro:cylinder_inertia mass="10" radius="0.25" height="1.0"/>
   </link>
-       <!-- Leo_left_wheel -->
-    <link name="left_wheel_link">
+  <link name="left_wheel_link">
     <visual>
       <xacro:cylinder_geometry radius="0.1" height="0.05"/>
@@ -22,13 +21,11 @@
     <xacro:cylinder_inertia mass="10" radius="0.1" height="0.05"/>
   </link>
-    <!-- left_wheel-body -->
   <joint name="left_wheel_body_joint" type="continuous">
-    <origin rpy="1.570795 0 0" xyz="0.0 0.275 -0.55"/>
+    <origin rpy="${pi / 2} 0 0" xyz="0.0 0.275 -0.55"/>
     <parent link="base_link"/>
     <child link="left_wheel_link"/>
     <axis xyz="0 0 1" />
   </joint>
-       <!-- Leo_right_wheel -->
-    <link name="right_wheel_link">
+  <link name="right_wheel_link">
     <visual>
       <xacro:cylinder_geometry radius="0.1" height="0.05"/>
@@ -38,13 +35,11 @@
     <xacro:cylinder_inertia mass="10" radius="0.1" height="0.05"/>
   </link>
-      <!-- right_wheel-body -->
   <joint name="right_wheel_body_joint" type="continuous">
-    <origin rpy="1.570795 0 0" xyz="0.0 -0.275 -0.55"/>
+    <origin rpy="${pi / 2} 0 0" xyz="0.0 -0.275 -0.55"/>
     <parent link="base_link"/>
     <child link="right_wheel_link"/>
     <axis xyz="0 0 1" />
   </joint>
-       <!-- Leo_caster_wheel -->
-    <link name="caster_wheel_link">
+  <link name="caster_wheel_link">
     <visual>
       <xacro:sphere_geometry radius="0.08"/>
@@ -54,5 +49,4 @@
     <xacro:sphere_inertia mass="1" radius="0.08"/>
   </link>
-      <!-- left_wheel-body -->
   <joint name="caster_wheel_body_joint" type="fixed">
     <origin rpy="0 0 0" xyz="0.2 0.0 -0.57"/>

Commit message: Add head_link to gazebo config and change position camera on axis z

File: leobot_description/robot/leobot.gazebo.xacro (robot description, xacro)
@@ -9,4 +9,11 @@
   </gazebo>
   <gazebo reference="base_link">
+    <mu1 value="1.0"/>
+    <mu2 value="1.0"/>
+    <kp value="10000000.0"/>
+    <kd value="1.0"/>
+    <material>Gazebo/White</material>
+  </gazebo>
+  <gazebo reference="head_link">
     <mu1 value="1.0"/>
     <mu2 value="1.0"/>

File: leobot_description/robot/robot.urdf.xacro (robot description, xacro)
@@ -38,5 +38,5 @@
   </link>
   <joint name="camera_left_link_joint" type="fixed">
-    <origin rpy="0 0 0" xyz="0 0.075 0.1"/>
+    <origin rpy="0 0 0" xyz="0 0.075 0.075"/>
     <parent link="head_link"/>
     <child link="camera_left_link"/>
@@ -51,5 +51,5 @@
   </link>
   <joint name="camera_right_link_joint" type="fixed">
-    <origin rpy="0 0 0" xyz="0 -0.075 0.1"/>
+    <origin rpy="0 0 0" xyz="0 -0.075 0.075"/>
     <parent link="head_link"/>
     <child link="camera_right_link"/>

Commit message: Resolved Conflicts
Closing #29

File: leobot_description/robot/leobot.gazebo.xacro (robot description, xacro)
@@ -36,4 +36,36 @@
     <material>Gazebo/Red</material>
   </gazebo>
+  <gazebo reference="head_link">
+    <mu1 value="1.0"/>
+    <mu2 value="1.0"/>
+    <kp value="10000000.0"/>
+    <kd value="1.0"/>
+    <material>Gazebo/Red</material>
+  </gazebo>
+  <link name="head_link">
+    <visual>
+      <xacro:cylinder_geometry radius="0.15" height="0.1"/>
+      <xacro:navajo_white_material/>
+    </visual>
+    <xacro:cylinder_collision radius="0.15" height="0.1"/>
+    <xacro:cylinder_inertia mass="1" radius="0.15" height="0.1"/>
+  </link>
+  <joint name="head_link_joint" type="revolute">
+    <origin rpy="0 0 0" xyz="0 0 0.525"/>
+    <axis xyz="0 0 1" />
+    <parent link="base_link"/>
+    <child link="head_link"/>
+    <limit effort="10" velocity="10" lower="${-pi/2}" upper="${pi/2}" />
+  </joint>
+  <transmission name="head_transmission">
+     <type>transmission_interface/SimpleTransmission</type>
+     <joint name="head_link_joint">
+       <hardwareInterface>hardware_interface/EffortJointInterface</hardwareInterface>
+     </joint>
+     <actuator name="head_motor">
+       <hardwareInterface>EffortJointInterface</hardwareInterface>
+       <mechanicalReduction>1</mechanicalReduction>
+     </actuator>
+  </transmission>
   <gazebo reference="camera_left_link">
     <material>Gazebo/Green</material>

File: leobot_description/robot/robot.urdf.xacro (robot description, xacro)
@@ -47,5 +47,5 @@
     </visual>
     <xacro:sphere_collision radius="0.08"/>
-    <xacro:sphere_inertia mass="1" radius="0.08"/>
+    <xacro:sphere_inertia mass="10" radius="0.08"/>
   </link>
   <joint name="caster_wheel_body_joint" type="fixed">
