Commit message: Resolved Conflicts Added transmission Added wheel xacro macros Added wheel-base bearing
Closing #29

File: leobot_description/robot/leobot.gazebo.xacro (robot description, xacro)
@@ -29,4 +29,18 @@
     <material>Gazebo/Red</material>
   </gazebo>
+  <gazebo reference="right_bearing_link">
+    <mu1 value="0.0"/>
+    <mu2 value="0.0"/>
+    <kp value="10000000.0"/>
+    <kd value="1.0"/>
+    <material>Gazebo/Blue</material>
+  </gazebo>
+  <gazebo reference="right_bearing_link">
+    <mu1 value="0.0"/>
+    <mu2 value="0.0"/>
+    <kp value="10000000.0"/>
+    <kd value="1.0"/>
+    <material>Gazebo/Blue</material>
+  </gazebo>
   <gazebo reference="caster_wheel_link">
     <mu1 value="0.0"/>
@@ -43,29 +57,4 @@
     <material>Gazebo/Red</material>
   </gazebo>
-  <link name="head_link">
-    <visual>
-      <xacro:cylinder_geometry radius="0.15" height="0.1"/>
-      <xacro:navajo_white_material/>
-    </visual>
-    <xacro:cylinder_collision radius="0.15" height="0.1"/>
-    <xacro:cylinder_inertia mass="1" radius="0.15" height="0.1"/>
-  </link>
-  <joint name="head_link_joint" type="revolute">
-    <origin rpy="0 0 0" xyz="0 0 0.525"/>
-    <axis xyz="0 0 1" />
-    <parent link="base_link"/>
-    <child link="head_link"/>
-    <limit effort="10" velocity="10" lower="${-pi/2}" upper="${pi/2}" />
-  </joint>
-  <transmission name="head_transmission">
-     <type>transmission_interface/SimpleTransmission</type>
-     <joint name="head_link_joint">
-       <hardwareInterface>hardware_interface/EffortJointInterface</hardwareInterface>
-     </joint>
-     <actuator name="head_motor">
-       <hardwareInterface>EffortJointInterface</hardwareInterface>
-       <mechanicalReduction>1</mechanicalReduction>
-     </actuator>
-  </transmission>
   <gazebo reference="camera_left_link">
     <material>Gazebo/Green</material>

File: leobot_description/robot/robot.urdf.xacro (robot description, xacro)
@@ -4,55 +4,52 @@
   <xacro:include filename="$(find leobot_description)/urdf/materials.urdf.xacro"/>
   <xacro:include filename="$(find leobot_description)/urdf/common.urdf.xacro"/>
+  <xacro:include filename="$(find leobot_description)/urdf/wheels.urdf.xacro"/>
+    <!-- Robot properties -->
+  <xacro:property name="base_radius" value="0.25"/>
+  <xacro:property name="base_height" value="1.0"/>
+  <xacro:property name="caster_radius" value="0.08"/>
+  <xacro:property name="caster_mass" value="10"/>
+  <xacro:property name="wheel_width" value="0.005"/>
+  <xacro:property name="wheel_radius" value="0.1"/>
+  <xacro:property name="wheel_mass" value="10"/>
+  <xacro:property name="bearing_radius" value="0.01"/>
   <!-- Robot links -->
   <link name="base_link">
     <visual>
-      <xacro:cylinder_geometry radius="0.25" height="1.0"/>
+      <xacro:cylinder_geometry radius="${base_radius}" height="${base_height}"/>
       <xacro:navajo_white_material/>
     </visual>
-    <xacro:cylinder_collision radius="0.25" height="1.0"/>
-    <xacro:cylinder_inertia mass="10" radius="0.25" height="1.0"/>
+    <xacro:cylinder_collision radius="${base_radius}" height="${base_height}"/>
+    <xacro:cylinder_inertia mass="10" radius="${base_radius}" height="${base_height}"/>
   </link>
-  <link name="left_wheel_link">
+  <xacro:caster_wheel radius="${caster_radius}" mass="${caster_mass}" x="0.2" y="0.0" z="-0.57"/>
+  <xacro:standard_wheel prefix="left" direction="1.0" bearing_radius="${bearing_radius}" radius="${wheel_radius}" width="${wheel_width}" mass="${wheel_mass}" base_radius="${base_radius}"/>
+  <xacro:standard_wheel prefix="right" direction="-1.0" bearing_radius="${bearing_radius}" radius="${wheel_radius}" width="${wheel_width}" mass="${wheel_mass}" base_radius="${base_radius}"/>
+  <link name="head_link">
     <visual>
-      <xacro:cylinder_geometry radius="0.1" height="0.05"/>
-      <xacro:red_material/>
+      <xacro:cylinder_geometry radius="0.15" height="0.1"/>
+      <xacro:navajo_white_material/>
     </visual>
-    <xacro:cylinder_collision radius="0.1" height="0.05"/>
-    <xacro:cylinder_inertia mass="10" radius="0.1" height="0.05"/>
+    <xacro:cylinder_collision radius="0.15" height="0.1"/>
+    <xacro:cylinder_inertia mass="1" radius="0.15" height="0.1"/>
   </link>
-  <joint name="left_wheel_body_joint" type="continuous">
-    <origin rpy="${pi / 2} 0 0" xyz="0.0 0.275 -0.55"/>
+  <joint name="head_link_joint" type="revolute">
+    <origin rpy="0 0 0" xyz="0 0 0.525"/>
+    <axis xyz="0 0 1" />
     <parent link="base_link"/>
-    <child link="left_wheel_link"/>
-    <axis xyz="0 0 1" />
+    <child link="head_link"/>
+    <limit effort="10" velocity="10" lower="${-pi/2}" upper="${pi/2}" />
   </joint>
-  <link name="right_wheel_link">
-    <visual>
-      <xacro:cylinder_geometry radius="0.1" height="0.05"/>
-      <xacro:red_material/>
-    </visual>
-    <xacro:cylinder_collision radius="0.1" height="0.05"/>
-    <xacro:cylinder_inertia mass="10" radius="0.1" height="0.05"/>
-  </link>
-  <joint name="right_wheel_body_joint" type="continuous">
-    <origin rpy="${pi / 2} 0 0" xyz="0.0 -0.275 -0.55"/>
-    <parent link="base_link"/>
-    <child link="right_wheel_link"/>
-    <axis xyz="0 0 1" />
-  </joint>
-  <link name="caster_wheel_link">
-    <visual>
-      <xacro:sphere_geometry radius="0.08"/>
-      <xacro:red_material/>
-    </visual>
-    <xacro:sphere_collision radius="0.08"/>
-    <xacro:sphere_inertia mass="10" radius="0.08"/>
-  </link>
-  <joint name="caster_wheel_body_joint" type="fixed">
-    <origin rpy="0 0 0" xyz="0.2 0.0 -0.57"/>
-    <parent link="base_link"/>
-    <child link="caster_wheel_link"/>
-  </joint>
-  <link name="camera_left_link">
+  <transmission name="head_transmission">
+     <type>transmission_interface/SimpleTransmission</type>
+     <joint name="head_link_joint">
+       <hardwareInterface>hardware_interface/EffortJointInterface</hardwareInterface>
+     </joint>
+     <actuator name="head_motor">
+       <hardwareInterface>EffortJointInterface</hardwareInterface>
+       <mechanicalReduction>1</mechanicalReduction>
+     </actuator>
+  </transmission>
+   <link name="camera_left_link">
     <visual>
       <xacro:box_geometry width="0.05" height="0.05" depth="0.05"/>
@@ -63,6 +60,6 @@
   </link>
   <joint name="camera_left_link_joint" type="fixed">
-    <origin rpy="0 0 0" xyz="0 0.075 0.525"/>
-    <parent link="base_link"/>
+    <origin rpy="0 0 0" xyz="0 0.075 0.075"/>
+    <parent link="head_link"/>
     <child link="camera_left_link"/>
   </joint>
@@ -76,6 +73,6 @@
   </link>
   <joint name="camera_right_link_joint" type="fixed">
-    <origin rpy="0 0 0" xyz="0 -0.075 0.525"/>
-    <parent link="base_link"/>
+    <origin rpy="0 0 0" xyz="0 -0.075 0.075"/>
+    <parent link="head_link"/>
     <child link="camera_right_link"/>
   </joint>

File: leobot_description/urdf/materials.urdf.xacro (robot description, xacro)
@@ -26,3 +26,8 @@
     </material>
   </xacro:macro>
+  <xacro:macro name="blue_material">
+    <material name="blue">
+      <color rgba="0.0 0.0 1.0 1.0"/>
+    </material>
+  </xacro:macro>
 </robot>

Commit message: Resolved Conflicts Added transmission Added wheel xacro macros Added wheel-base bearing
Closing #29

File: leobot_description/robot/leobot.gazebo.xacro (robot description, xacro)
@@ -29,5 +29,5 @@
     <material>Gazebo/Red</material>
   </gazebo>
-  <gazebo reference="right_bearing_link">
+  <gazebo reference="left_bearing_link">
     <mu1 value="0.0"/>
     <mu2 value="0.0"/>

File: leobot_description/robot/robot.urdf.xacro (robot description, xacro)
@@ -8,5 +8,5 @@
   <xacro:property name="base_radius" value="0.25"/>
   <xacro:property name="base_height" value="1.0"/>
-  <xacro:property name="caster_radius" value="0.08"/>
+  <xacro:property name="caster_radius" value="0.05"/>
   <xacro:property name="caster_mass" value="10"/>
   <xacro:property name="wheel_width" value="0.005"/>
@@ -23,5 +23,5 @@
     <xacro:cylinder_inertia mass="10" radius="${base_radius}" height="${base_height}"/>
   </link>
-  <xacro:caster_wheel radius="${caster_radius}" mass="${caster_mass}" x="0.2" y="0.0" z="-0.57"/>
+  <xacro:caster_wheel radius="${caster_radius}" mass="${caster_mass}" base_radius="${base_radius}" base_height="${base_height}"/>
   <xacro:standard_wheel prefix="left" direction="1.0" bearing_radius="${bearing_radius}" radius="${wheel_radius}" width="${wheel_width}" mass="${wheel_mass}" base_radius="${base_radius}"/>
   <xacro:standard_wheel prefix="right" direction="-1.0" bearing_radius="${bearing_radius}" radius="${wheel_radius}" width="${wheel_width}" mass="${wheel_mass}" base_radius="${base_radius}"/>

File: leobot_description/urdf/wheels.urdf.xacro (robot description, xacro)
@@ -31,5 +31,5 @@
         <transmission name="${prefix}_wheel_transmission">
             <type>transmission_interface/SimpleTransmission</type>
-            <joint name="${prefix}_wheel_joint">
+            <joint name="${prefix}_wheel_bearing_joint">
                 <hardwareInterface>hardware_interface/VelocityJointInterface</hardwareInterface>
             </joint>
@@ -40,35 +40,5 @@
         </transmission>
     </xacro:macro>
-<!--
-  <link name="left_wheel_link">
-    <visual>
-      <xacro:cylinder_geometry radius="0.1" height="0.05"/>
-      <xacro:red_material/>
-    </visual>
-    <xacro:cylinder_collision radius="0.1" height="0.05"/>
-    <xacro:cylinder_inertia mass="10" radius="0.1" height="0.05"/>
-  </link>
-  <joint name="left_wheel_body_joint" type="continuous">
-    <origin rpy="${pi / 2} 0 0" xyz="0.0 0.275 -0.55"/>
-    <parent link="base_link"/>
-    <child link="left_wheel_link"/>
-    <axis xyz="0 0 1" />
-  </joint>
-  <link name="right_wheel_link">
-    <visual>
-      <xacro:cylinder_geometry radius="0.1" height="0.05"/>
-      <xacro:red_material/>
-    </visual>
-    <xacro:cylinder_collision radius="0.1" height="0.05"/>
-    <xacro:cylinder_inertia mass="10" radius="0.1" height="0.05"/>
-  </link>
-  <joint name="right_wheel_body_joint" type="continuous">
-    <origin rpy="${pi / 2} 0 0" xyz="0.0 -0.275 -0.55"/>
-    <parent link="base_link"/>
-    <child link="right_wheel_link"/>
-    <axis xyz="0 0 1" />
-  </joint>
--->
-    <xacro:macro name="caster_wheel" params="radius mass x y z">
+    <xacro:macro name="caster_wheel" params="radius mass base_radius base_height">
         <link name="caster_wheel_link">
             <visual>
@@ -82,5 +52,5 @@
             <parent link="base_link"/>
             <child link="caster_wheel_link"/>
-            <origin rpy="0 0 0" xyz="${x} ${y} ${z}"/>
+            <origin rpy="0 0 0" xyz="${base_radius - radius - 0.01} 0.0 ${-(base_height/2 + radius - 0.01)}"/>
         </joint>
     </xacro:macro>

Commit message: Added Lirad Sensor
Closin #54

File: leobot_description/robot/leobot.gazebo.xacro (robot description, xacro)
@@ -118,4 +118,5 @@
   <!-- Hokuyo LIDAR for simulation -->
    <gazebo reference="laser_link">
+      <material>Gazebo/Green</material>
       <sensor type="ray" name="laser">
         <pose>0 0 0 0 0 0</pose>
@@ -142,7 +143,6 @@
           </noise>
         </ray>
-        <!--<plugin name="hokuyo_node" filename="libgazebo_ros_laser.so">-->
         <plugin name="gazebo_ros_hokuyo_controller" filename="libgazebo_ros_laser.so">
-          <topicName>/lidar_scan</topicName>
+          <topicName>/leobot/lidar/scan</topicName>
           <frameName>laser_link</frameName>
         </plugin>

File: leobot_description/urdf/sensors/hokuyo.urdf.xacro (robot description, xacro)
@@ -1,5 +1,5 @@
 <?xml version="1.0"?>
 <robot xmlns:xacro="http://ros.org/wiki/xacro">
-     <xacro:property name="hokuyo_width" value="0.001"/>
+     <xacro:property name="hokuyo_width" value="0.1"/>
      <xacro:property name="hokuyo_height" value="0.05"/>
      <xacro:property name="hokuyo_depth" value="0.06"/>
@@ -12,8 +12,8 @@
       </visual>
       <xacro:box_collision width="${hokuyo_width}" height="${hokuyo_height}" depth="${hokuyo_depth}"/>
-      <xacro:box_inertia mass="0.0001" width="${hokuyo_width}" height="${hokuyo_height}" depth="${hokuyo_depth}"/>
+      <xacro:box_inertia mass="0.01" width="${hokuyo_width}" height="${hokuyo_height}" depth="${hokuyo_depth}"/>
     </link>
     <joint name="laser_base_joint" type="fixed">
-      <origin xyz="${-(base_radius - 0.0001)} 0.0 ${-base_height/2 + 0.01}" rpy="${pi} 0.0 0.0" />
+      <origin xyz="${-(base_radius - 0.0001)} 0.0 ${-base_height/2 + 0.01}" rpy="0.0 ${pi} 0.0" />
       <parent link="base_link" />
       <child link="laser_link" />

Commit message: Fixed Gazebo Core Dump issue

File: leobot_description/robot/leobot.gazebo.xacro (robot description, xacro)
@@ -121,5 +121,5 @@
       <sensor type="ray" name="laser">
         <pose>0 0 0 0 0 0</pose>
-        <visualize>false</visualize>
+        <visualize>true</visualize>
         <update_rate>40</update_rate>
         <ray>
@@ -138,5 +138,5 @@
           </range>
           <noise>
-            <type>Gaussian</type>
+            <type>gaussian</type>
             <mean>0.0</mean>
             <stddev>0.01</stddev>

File: leobot_description/robot/robot.urdf.xacro (robot description, xacro)
@@ -27,5 +27,5 @@
   <xacro:standard_wheel prefix="left" direction="1.0" bearing_radius="${bearing_radius}" radius="${wheel_radius}" width="${wheel_width}" mass="${wheel_mass}" base_radius="${base_radius}"/>
   <xacro:standard_wheel prefix="right" direction="-1.0" bearing_radius="${bearing_radius}" radius="${wheel_radius}" width="${wheel_width}" mass="${wheel_mass}" base_radius="${base_radius}"/>
-  <xacro:LIDAR_hokuyo base_radius="${base_radius}" base_height="${base_height}"/>
+  <xacro:lidar_hokuyo base_radius="${base_radius}" base_height="${base_height}"/>
   <link name="head_link">
     <visual>

File: leobot_description/urdf/sensors/hokuyo.urdf.xacro (robot description, xacro)
@@ -1,22 +1,21 @@
 <?xml version="1.0"?>
-<robot xmlns:xacro="http://ros.org/wiki/xacro">
-     <xacro:property name="hokuyo_width" value="0.001"/>
-     <xacro:property name="hokuyo_height" value="0.05"/>
-     <xacro:property name="hokuyo_depth" value="0.06"/>
-  <!-- Hokuyo 2D LIDAR -->
-  <xacro:macro name="LIDAR_hokuyo" params="base_radius base_height">
-    <link name="laser_link">
-      <visual>
-          <xacro:box_geometry width="${hokuyo_width}" height="${hokuyo_height}" depth="${hokuyo_depth}"/>
-          <xacro:green_material/>
-      </visual>
-      <xacro:box_collision width="${hokuyo_width}" height="${hokuyo_height}" depth="${hokuyo_depth}"/>
-      <xacro:box_inertia mass="0.001" width="${hokuyo_width}" height="${hokuyo_height}" depth="${hokuyo_depth}"/>
-    </link>
-    <joint name="laser_base_joint" type="fixed">
-      <origin xyz="${-(base_radius - 0.0001)} 0.0 ${-base_height/2 + 0.01}" rpy="0.0 ${pi} 0.0" />
-      <parent link="base_link" />
-      <child link="laser_link" />
-    </joint>
-  </xacro:macro>
-</robot>
+    <robot xmlns:xacro="http://ros.org/wiki/xacro">
+        <xacro:property name="hokuyo_width" value="0.001"/>
+        <xacro:property name="hokuyo_height" value="0.05"/>
+        <xacro:property name="hokuyo_depth" value="0.06"/>
+        <xacro:macro name="lidar_hokuyo" params="base_radius base_height">
+            <link name="laser_link">
+              <visual>
+                  <xacro:box_geometry width="${hokuyo_width}" height="${hokuyo_height}" depth="${hokuyo_depth}"/>
+                  <xacro:green_material/>
+              </visual>
+              <xacro:box_collision width="${hokuyo_width}" height="${hokuyo_height}" depth="${hokuyo_depth}"/>
+              <xacro:box_inertia mass="0.001" width="${hokuyo_width}" height="${hokuyo_height}" depth="${hokuyo_depth}"/>
+            </link>
+            <joint name="laser_base_joint" type="fixed">
+              <origin xyz="${-(base_radius - 0.0001)} 0.0 ${-base_height/2 + 0.01}" rpy="0.0 ${pi} 0.0" />
+              <parent link="base_link" />
+              <child link="laser_link" />
+            </joint>
+        </xacro:macro>
+    </robot>

Commit message: urdf modification

File: leobot_description/robot/leobot.gazebo.xacro (robot description, xacro)
@@ -51,4 +51,11 @@
   </gazebo>
   <gazebo reference="head_link">
+    <mu1 value="1.0"/>
+    <mu2 value="1.0"/>
+    <kp value="10000000.0"/>
+    <kd value="1.0"/>
+    <material>Gazebo/White</material>
+  </gazebo>
+  <gazebo reference="tower_link">
     <mu1 value="1.0"/>
     <mu2 value="1.0"/>

File: leobot_description/robot/robot.urdf.xacro (robot description, xacro)
@@ -6,9 +6,9 @@
   <xacro:include filename="$(find leobot_description)/urdf/wheels.urdf.xacro"/>
   <!-- Robot properties -->
-  <xacro:property name="base_width" value="0.7"/>
-  <xacro:property name="base_length" value="1.132"/>
-  <xacro:property name="base_height" value="0.4"/>
-  <xacro:property name="base_radius" value="0.25"/>
-  <xacro:property name="tower_height" value="1.225"/>
+  <xacro:property name="base_width" value="${(1.132/1.7)}"/>
+  <xacro:property name="base_length" value="${(0.7 / 2)}"/>
+  <xacro:property name="base_height" value="${(0.4 / 2.5)}"/>
+  <xacro:property name="base_radius" value="0.5"/>
+  <xacro:property name="tower_height" value="${(1.225 * 2.7)}"/>
   <xacro:property name="caster_radius" value="0.05"/>
   <xacro:property name="caster_mass" value="10"/>
@@ -20,5 +20,5 @@
   <link name="base_link">
     <visual>
-      <origin xyz="0 -0.25 0" rpy="0 0 ${pi}"/>
+      <origin xyz="0 -0.25 -0.08" rpy="0 0 ${pi}"/>
       <geometry>
           <mesh filename="package://leobot_description/meshes/base.stl" scale="0.001 0.001 0.001"/>
@@ -28,5 +28,5 @@
   </link>
    <link name="base_link_inertia">
-    <xacro:box_collision width="${base_width + 0.05}" depth="${base_length+0.05}" height="${base_height + 0.05}"/>
+    <xacro:box_collision width="${base_width + 0.05}" depth="${base_length + 0.05}" height="${base_height + 0.05}"/>
     <xacro:box_inertia mass="3.0" width="${base_length}" depth="${base_height}" height="${base_width}"/>
   </link>
@@ -37,6 +37,6 @@
   </joint>
   <xacro:caster_wheel radius="${caster_radius}" mass="${caster_mass}" base_radius="${base_radius}" base_height="${base_height}"/>
-  <xacro:standard_wheel prefix="left" direction="1.0" bearing_radius="${bearing_radius}" radius="${wheel_radius}" width="${wheel_width}" mass="${wheel_mass}" base_radius="${base_radius}"/>
-  <xacro:standard_wheel prefix="right" direction="-1.0" bearing_radius="${bearing_radius}" radius="${wheel_radius}" width="${wheel_width}" mass="${wheel_mass}" base_radius="${base_radius}"/>
+  <xacro:standard_wheel prefix="left" direction="1.0" bearing_radius="${bearing_radius}" radius="${wheel_radius}" width="${wheel_width}" mass="${wheel_mass}" base_radius="${base_radius/1.8}"/>
+  <xacro:standard_wheel prefix="right" direction="-1.0" bearing_radius="${bearing_radius}" radius="${wheel_radius}" width="${wheel_width}" mass="${wheel_mass}" base_radius="${base_radius/1.8}"/>
     <link name="tower_link">
         <visual>
@@ -48,7 +48,7 @@
         </visual>
       </link>
-       <joint name="tower_link_joint" type="fixed">
+     <joint name="tower_link_joint" type="fixed">
         <origin xyz="0 0 0" rpy="0 0 0"/>
-        <parent link="base_link_inertia"/>
+        <parent link="base_link"/>
         <child link="tower_link"/>
       </joint>
@@ -62,5 +62,5 @@
   </link>
   <joint name="head_link_joint" type="revolute">
-    <origin rpy="0 0 0" xyz="0 0 0"/>
+    <origin rpy="0 0 0" xyz="0.3 0.0 ${(tower_height / 2)}"/>
     <axis xyz="0 0 1" />
     <parent link="tower_link"/>

Commit message: Lidar moved to the front Lidar range updated

File: leobot_description/robot/leobot.gazebo.xacro (robot description, xacro)
@@ -128,10 +128,10 @@
               <samples>1081</samples>
               <resolution>1</resolution>
-              <min_angle>-2.3561944902</min_angle>
-              <max_angle>2.3561944902</max_angle>
+              <min_angle>-1.570796</min_angle>
+              <max_angle>1.570796</max_angle>
             </horizontal>
           </scan>
           <range>
-            <min>0.10</min>
+            <min>0.60</min>
             <max>10.0</max>
             <resolution>0.01</resolution>

File: leobot_description/urdf/sensors/hokuyo.urdf.xacro (robot description, xacro)
@@ -14,5 +14,5 @@
             </link>
             <joint name="laser_base_joint" type="fixed">
-              <origin xyz="${-(base_radius - 0.0001)} 0.0 ${-base_height/2 + 0.01}" rpy="0.0 ${pi} 0.0" />
+              <origin xyz="${(base_radius - 0.0001)} 0.0 ${-base_height/2 + 0.01}" rpy="0.0 ${pi} 0.0" />
               <parent link="base_link" />
               <child link="laser_link" />

File: leobot_description/urdf/wheels.urdf.xacro (robot description, xacro)
@@ -24,5 +24,5 @@
         </link>
         <joint name="${prefix}_wheel_bearing_joint" type="continuous">
-            <origin rpy="${pi / 2} 0 0" xyz="0.0 ${direction * (bearing_radius + width/2 - 0.0001)} 0.0"/>
+            <origin rpy="${pi / 2} 0 ${pi}" xyz="0.0 ${direction * (bearing_radius + width/2 - 0.0001)} 0.0"/>
             <parent link="${prefix}_bearing_link"/>
             <child link="${prefix}_wheel_link"/>
