Commit message: Added motor joints Added mecanum wheels Tuned Gazebo.urdf Added two fisheye cameras

File: leobot_description/robot/leobot.gazebo.xacro (robot description, xacro)
@@ -15,39 +15,4 @@
     <material>Gazebo/White</material>
   </gazebo>
-  <gazebo reference="left_wheel_link">
-    <mu1 value="1.0"/>
-    <mu2 value="1.0"/>
-    <kp value="10000000.0"/>
-    <kd value="1.0"/>
-    <material>Gazebo/Red</material>
-  </gazebo>
-  <gazebo reference="right_wheel_link">
-    <mu1 value="1.0"/>
-    <mu2 value="1.0"/>
-    <kp value="10000000.0"/>
-    <kd value="1.0"/>
-    <material>Gazebo/Red</material>
-  </gazebo>
-  <gazebo reference="left_bearing_link">
-    <mu1 value="0.0"/>
-    <mu2 value="0.0"/>
-    <kp value="10000000.0"/>
-    <kd value="1.0"/>
-    <material>Gazebo/Blue</material>
-  </gazebo>
-  <gazebo reference="right_bearing_link">
-    <mu1 value="0.0"/>
-    <mu2 value="0.0"/>
-    <kp value="10000000.0"/>
-    <kd value="1.0"/>
-    <material>Gazebo/Blue</material>
-  </gazebo>
-  <gazebo reference="caster_wheel_link">
-    <mu1 value="0.0"/>
-    <mu2 value="0.0"/>
-    <kp value="10000000.0"/>
-    <kd value="1.0"/>
-    <material>Gazebo/Red</material>
-  </gazebo>
   <gazebo reference="head_link">
     <mu1 value="1.0"/>
@@ -57,47 +22,105 @@
     <material>Gazebo/White</material>
   </gazebo>
-  <gazebo reference="camera_left_link">
+  <gazebo reference="neck_link">
+    <mu1 value="1.0"/>
+    <mu2 value="1.0"/>
+    <kp value="10000000.0"/>
+    <kd value="1.0"/>
+    <material>Gazebo/White</material>
+  </gazebo>
+  <gazebo reference="FL_wheel_link">
+    <mu1 value="1.0"/>
+    <mu2 value="1.0"/>
+    <kp value="10000000.0"/>
+    <kd value="1.0"/>
+    <material>Gazebo/Blue</material>
+  </gazebo>
+  <gazebo reference="FR_wheel_link">
+    <mu1 value="1.0"/>
+    <mu2 value="1.0"/>
+    <kp value="10000000.0"/>
+    <kd value="1.0"/>
+    <material>Gazebo/Blue</material>
+  </gazebo>
+  <gazebo reference="RL_wheel_link">
+    <mu1 value="1.0"/>
+    <mu2 value="1.0"/>
+    <kp value="10000000.0"/>
+    <kd value="1.0"/>
+    <material>Gazebo/Blue</material>
+  </gazebo>
+  <gazebo reference="RR_wheel_link">
+    <mu1 value="1.0"/>
+    <mu2 value="1.0"/>
+    <kp value="10000000.0"/>
+    <kd value="1.0"/>
+    <material>Gazebo/Blue</material>
+  </gazebo>
+  <gazebo reference="FR_motor_holder">
+    <mu1 value="1.0"/>
+    <mu2 value="1.0"/>
+    <kp value="10000000.0"/>
+    <kd value="1.0"/>
+    <material>Gazebo/Red</material>
+  </gazebo>
+  <gazebo reference="FL_motor_holder">
+    <mu1 value="1.0"/>
+    <mu2 value="1.0"/>
+    <kp value="10000000.0"/>
+    <kd value="1.0"/>
+    <material>Gazebo/Red</material>
+  </gazebo>
+  <gazebo reference="RL_motor_holder">
+    <mu1 value="1.0"/>
+    <mu2 value="1.0"/>
+    <kp value="10000000.0"/>
+    <kd value="1.0"/>
+    <material>Gazebo/Red</material>
+  </gazebo>
+  <gazebo reference="RR_motor_holder">
+    <mu1 value="1.0"/>
+    <mu2 value="1.0"/>
+    <kp value="10000000.0"/>
+    <kd value="1.0"/>
+    <material>Gazebo/Red</material>
+  </gazebo>
+  <gazebo reference="left_camera_link">
     <material>Gazebo/Green</material>
-    <sensor type="multicamera" name="stereo_camera">
-      <update_rate>30.0</update_rate>
-      <camera name="left">
-        <horizontal_fov>1.3962634</horizontal_fov>
-        <image>
-          <width>800</width>
-          <height>800</height>
-          <format>R8G8B8</format>
-        </image>
-        <clip>
-          <near>0.02</near>
-          <far>300</far>
-        </clip>
-        <noise>
-          <type>gaussian</type>
-          <mean>0.0</mean>
-          <stddev>0.007</stddev>
-        </noise>
-      </camera>
-      <camera name="right">
-        <pose>0 -0.07 0 0 0 0</pose>
-        <horizontal_fov>1.3962634</horizontal_fov>
-        <image>
-          <width>800</width>
-          <height>800</height>
-          <format>R8G8B8</format>
-        </image>
-        <clip>
-          <near>0.02</near>
-          <far>300</far>
-        </clip>
-        <noise>
-          <type>gaussian</type>
-          <mean>0.0</mean>
-          <stddev>0.007</stddev>
-        </noise>
-      </camera>
-      <plugin name="stereo_camera_controller" filename="libgazebo_ros_multicamera.so">
+    <sensor name="left_camera" type="wideanglecamera">
+  <camera>
+    <horizontal_fov>6.283</horizontal_fov>
+    <image>
+      <width>320</width>
+      <height>240</height>
+    </image>
+    <clip>
+      <near>0.1</near>
+      <far>100</far>
+    </clip>
+     <!-- A new section named `lens`. -->
+    <lens>
+      <!-- type element is mandatory -->
+      <type>custom</type>
+      <!-- manually defined mapping function r = c1*f*fun(theta/c2 + c3) -->
+      <!-- More information here: https://en.wikipedia.org/wiki/Fisheye_lens#Mapping_function -->
+      <custom_function>
+        <c1>1.05</c1>   <!-- linear scaling -->
+        <c2>4</c2>      <!-- angle scaling -->
+        <f>1.0</f>      <!-- one more scaling parameter -->
+        <fun>tan</fun>  <!-- one of sin,tan,id -->
+      </custom_function>
+      <!-- if it is set to `true` your horizontal FOV will ramain as defined -->
+      <!-- othervise it depends on lens type and custom function, if there is one -->
+      <scale_to_hfov>true</scale_to_hfov>
+      <!-- clip everything that is outside of this angle -->
+      <cutoff_angle>3.1415</cutoff_angle>
+      <!-- resolution of the cubemap texture, the highter it is - the sharper is your image -->
+      <env_texture_size>512</env_texture_size>
+    </lens>
+  </camera>
+      <plugin name="left_fisheye_camera_controller" filename="libgazebo_ros_camera.so">
         <alwaysOn>true</alwaysOn>
         <updateRate>0.0</updateRate>
-        <cameraName>stereocamera</cameraName>
+        <cameraName>fisheyecamera</cameraName>
         <imageTopicName>image_raw</imageTopicName>
         <cameraInfoTopicName>camera_info</cameraInfoTopicName>
@@ -111,8 +134,60 @@
         <distortionT2>0.0</distortionT2>
       </plugin>
-    </sensor>
-  </gazebo>
-  <gazebo reference="camera_right_link">
+  <always_on>1</always_on>
+  <update_rate>30</update_rate>
+</sensor>
+  </gazebo>
+  <gazebo reference="right_camera_link">
     <material>Gazebo/Green</material>
+      <sensor name="right_camera" type="wideanglecamera">
+  <camera>
+    <horizontal_fov>6.283</horizontal_fov>
+    <image>
+      <width>320</width>
+      <height>240</height>
+    </image>
+    <clip>
+      <near>0.1</near>
+      <far>100</far>
+    </clip>
+     <!-- A new section named `lens`. -->
+    <lens>
+      <!-- type element is mandatory -->
+      <type>custom</type>
+      <!-- manually defined mapping function r = c1*f*fun(theta/c2 + c3) -->
+      <!-- More information here: https://en.wikipedia.org/wiki/Fisheye_lens#Mapping_function -->
+      <custom_function>
+        <c1>1.05</c1>   <!-- linear scaling -->
+        <c2>4</c2>      <!-- angle scaling -->
+        <f>1.0</f>      <!-- one more scaling parameter -->
+        <fun>tan</fun>  <!-- one of sin,tan,id -->
+      </custom_function>
+      <!-- if it is set to `true` your horizontal FOV will ramain as defined -->
+      <!-- othervise it depends on lens type and custom function, if there is one -->
+      <scale_to_hfov>true</scale_to_hfov>
+      <!-- clip everything that is outside of this angle -->
+      <cutoff_angle>3.1415</cutoff_angle>
+      <!-- resolution of the cubemap texture, the highter it is - the sharper is your image -->
+      <env_texture_size>512</env_texture_size>
+    </lens>
+  </camera>
+      <plugin name="right_fisheye_camera_controller" filename="libgazebo_ros_camera.so">
+        <alwaysOn>true</alwaysOn>
+        <updateRate>0.0</updateRate>
+        <cameraName>fisheyecamera</cameraName>
+        <imageTopicName>image_raw</imageTopicName>
+        <cameraInfoTopicName>camera_info</cameraInfoTopicName>
+        <frameName>camera_left_link</frameName>
+        <rightFrameName>camera_right_link</rightFrameName>
+        <hackBaseline>0.07</hackBaseline>
+        <distortionK1>0.0</distortionK1>
+        <distortionK2>0.0</distortionK2>
+        <distortionK3>0.0</distortionK3>
+        <distortionT1>0.0</distortionT1>
+        <distortionT2>0.0</distortionT2>
+      </plugin>
+  <always_on>1</always_on>
+  <update_rate>30</update_rate>
+</sensor>
   </gazebo>
   <!-- Hokuyo LIDAR for simulation -->

File: leobot_description/robot/robot.urdf.xacro (robot description, xacro)
@@ -5,7 +5,7 @@
   <xacro:include filename="$(find leobot_description)/urdf/sensors/hokuyo.urdf.xacro"/>
   <xacro:include filename="$(find leobot_description)/urdf/wheels.urdf.xacro"/>
-  <xacro:property name="base_width" value="0.5"/>
+  <xacro:property name="base_width" value="0.54"/>
   <xacro:property name="base_length" value="0.3"/>
-  <xacro:property name="base_height" value="0.54"/>
+  <xacro:property name="base_height" value="0.5"/>
   <xacro:property name="base_mass" value="10"/>
   <xacro:property name="neck_width" value="0.04"/>
@@ -34,5 +34,5 @@
   </link>
   <joint name="base_neck_joint" type="fixed">
-    <origin rpy="${pi/2} 0  0" xyz="0 ${-base_width/2 - neck_width} ${-base_length/2 + neck_height / 2 }"/>
+    <origin rpy="${pi/2} 0  0" xyz="${-base_height/2 - neck_width} 0 ${-base_length/2 + neck_height / 2 }"/>
     <parent link="base_link"/>
     <child link="neck_link"/>
@@ -47,5 +47,5 @@
   </link>
   <joint name="neck_head_joint" type="fixed">
-    <origin rpy="${pi/2} 0  0" xyz="0 ${neck_height/2 + head_width/2} ${neck_length/2 - head_height/2}"/>
+    <origin rpy="${pi/2} ${pi/2} ${pi}" xyz="${-neck_length/2 + head_height/2} ${neck_height/2 + head_width/2} 0"/>
     <parent link="neck_link"/>
     <child link="head_link"/>
@@ -54,55 +54,7 @@
   <xacro:fish_camera prefix = "right" parent_link_name="head_link" parent_height="${head_height}"  parent_width = "${head_width}" side="-1"/>
   <xacro:lidar_hokuyo parent_link_name="base_link" parent_height="${base_length}"/>
-  <xacro:mecanum_wheel prefix="FR" wheel_type="1" side="1" position="1" parent_length="${base_width}" parent_height="${base_height}" parent_width="${base_length}"/>
-<!--  <xacro:macro name="mecanum_wheel" params="link_name mesh_file radius width *origin">
-    <link name="${link_name}">
-      <visual>
-        <xacro:insert_block name="origin"/>
-        <geometry>
-          <mesh filename="${mesh_file}" scale="1 1 1"/>
-        </geometry>
-        <xacro:navajo_white_material/>
-      </visual>
-      <collision>
-        <xacro:insert_block name="origin"/>
-        <geometry>
-          <cylinder length="${width}" radius="${radius}"/>
-        </geometry>
-      </collision>
-      <xacro:cylinder_inertia mass="10" radius="${radius}" height="${width}"/>
-    </link>
-  </xacro:macro>-->
-  <!--<xacro:macro name="leobot_mecanum_wheel" params="name variant origin_x origin_y">
-    <xacro:mecanum_wheel link_name="wheel_${name}"
-                         mesh_file="package://leobot_description/meshes/Mecanum_Wheel_0${variant}.STL"
-                         radius="${wheel_radius}" width="${wheel_width}">
-      <origin xyz="${origin_x * base_width/2} ${origin_y * base_length/2}"
-              rpy="${pi/2} 0 0"/>
-    </xacro:mecanum_wheel>
-  </xacro:macro>
-  <xacro:leobot_mecanum_wheel name="FR" variant="1" origin_x="1"  origin_y="1"/>
-  <xacro:leobot_mecanum_wheel name="FL" variant="1" origin_x="-1" origin_y="1"/>
-  <xacro:leobot_mecanum_wheel name="RL" variant="2" origin_x="-1" origin_y="-1"/>
-  <xacro:leobot_mecanum_wheel name="RR" variant="2" origin_x="1"  origin_y="-1"/>
-  <joint name="base_link_wheel_FR_joint" type="continuous">
-    <origin xyz="0 0 0.05" rpy="0 0 0" />
-    <parent link="base_link" />
-    <child link="wheel_FL" />
-  </joint>
-  <joint name="base_link_joint_wheel_FL_joint" type="continuous">
-    <origin xyz="0 0 0.05" rpy="0 0 0" />
-    <parent link="base_link" />
-    <child link="wheel_FR" />
-  </joint>
-  <joint name="base_link_joint_wheel_RL_joint" type="continuous">
-    <origin xyz="0 0 0" rpy="0 0 0" />
-    <parent link="base_link" />
-    <child link="wheel_RL" />
-  </joint>
-  <joint name="base_link_joint_wheel_RR_joint" type="continuous">
-    <origin xyz="0 0 0" rpy="0 0 0" />
-    <parent link="base_link" />
-    <child link="wheel_RR" />
-  </joint>
--->
+  <xacro:mecanum_wheel prefix="FL" wheel_type="2" side="1" position="1" parent_length="${base_width}" parent_height="${base_length}" parent_width="${base_height}"/>
+  <xacro:mecanum_wheel prefix="FR" wheel_type="1" side="-1" position="1" parent_length="${base_width}" parent_height="${base_length}" parent_width="${base_height}"/>
+  <xacro:mecanum_wheel prefix="RL" wheel_type="1" side="1" position="-1" parent_length="${base_width}" parent_height="${base_length}" parent_width="${base_height}"/>
+  <xacro:mecanum_wheel prefix="RR" wheel_type="2" side="-1" position="-1" parent_length="${base_width}" parent_height="${base_length}" parent_width="${base_height}"/>
 </robot>

File: leobot_description/urdf/sensors/camera.urdf.xacro (robot description, xacro)
@@ -13,5 +13,5 @@
         </link>
         <joint name="head_${prefix}_camera_joint" type="fixed">
-            <origin xyz="${side*(camera_radius + parent_width/2) - side*0.005} ${-parent_height/2 + camera_radius} 0" rpy="0 0 0"/>
+            <origin xyz="${side*(camera_radius + parent_width/2) - side*0.005} ${-parent_height/2 + camera_radius} 0" rpy="0 ${pi/2 + side * pi/2 } 0"/>
             <parent link="${parent_link_name}" />
             <child link="${prefix}_camera_link" />

File: leobot_description/urdf/wheels.urdf.xacro (robot description, xacro)
@@ -5,5 +5,5 @@
     <xacro:property name="motor_holder_mass" value="0.8"/>
     <xacro:property name="mecanum_radius" value="0.1"/>
-    <xacro:property name="mecanum_height" value="0.05"/>
+    <xacro:property name="mecanum_height" value="0.1"/>
     <xacro:property name="mecanum_mass" value="0.3"/>
     <xacro:macro name="mecanum_wheel"
@@ -19,5 +19,5 @@
         <joint name="${prefix}_motor_holder_base_joint" type="fixed">
             <origin rpy="${pi/2} 0 0"
-                    xyz="${position * (parent_width/2 - motor_holder_height/2)} ${position * parent_length} ${side * (parent_height/2 - motor_holder_radius/2)}"/>
+                    xyz="${position * (parent_length/2 - motor_holder_radius*2)} ${side * (parent_width/2 + motor_holder_height/2)} ${(-parent_height/2 + motor_holder_radius*2)}"/>
             <parent link="base_link"/>
             <child link="${prefix}_motor_holder"/>
@@ -25,7 +25,7 @@
         <link name="${prefix}_wheel_link">
             <visual>
-                <origin rpy="${pi / 2} 0 0 " xyz="0 0 0"/>
+                <origin rpy="0 0 0 " xyz="${-mecanum_radius*1.05} ${-mecanum_radius} ${-mecanum_height*0.75}"/>
                 <geometry>
-                    <mesh filename="package://leobot_description/meshes/Mecanum_Wheel_${wheel_type}.STL" scale="0.001 0.001 0.001"/>
+                    <mesh filename="package://leobot_description/meshes/Mecanum_Wheel_${wheel_type}.STL" scale="0.0015 0.0015 0.0015"/>
                 </geometry>
             </visual>
@@ -34,5 +34,5 @@
         </link>
         <joint name="${prefix}_wheel_motor_joint" type="continuous">
-            <origin rpy="0 0 0" xyz="0 0 ${side * mecanum_height/2}"/>
+            <origin rpy="0 0 0" xyz="0 0 ${ -1 * side * motor_holder_height/2}"/>
             <parent link="${prefix}_motor_holder"/>
             <child link="${prefix}_wheel_link"/>
@@ -46,6 +46,6 @@
             <actuator name="${prefix}_wheel_motor">
                 <hardwareInterface>hardware_interface/VelocityJointInterface</hardwareInterface>
-                <mechanicalReduction>1</mechanicalReduction>
-                <motorTorqueConstant>1</motorTorqueConstant>
+                <mechanicalReduction>131</mechanicalReduction>
+                <motorTorqueConstant>4.4</motorTorqueConstant>
             </actuator>
         </transmission>
