Commit message: Made the camera look up again Fixed small typos

File: leobot_description/robot/leobot.gazebo.xacro (robot description, xacro)
@@ -88,106 +88,106 @@
     <material>Gazebo/Green</material>
     <sensor name="left_camera" type="wideanglecamera">
-  <camera>
-    <horizontal_fov>6.283</horizontal_fov>
-    <image>
-      <width>320</width>
-      <height>240</height>
-    </image>
-    <clip>
-      <near>0.1</near>
-      <far>100</far>
-    </clip>
-     <!-- A new section named `lens`. -->
-    <lens>
-      <!-- type element is mandatory -->
-      <type>custom</type>
-      <!-- manually defined mapping function r = c1*f*fun(theta/c2 + c3) -->
-      <!-- More information here: https://en.wikipedia.org/wiki/Fisheye_lens#Mapping_function -->
-      <custom_function>
-        <c1>1.05</c1>   <!-- linear scaling -->
-        <c2>4</c2>      <!-- angle scaling -->
-        <f>1.0</f>      <!-- one more scaling parameter -->
-        <fun>tan</fun>  <!-- one of sin,tan,id -->
-      </custom_function>
-      <!-- if it is set to `true` your horizontal FOV will ramain as defined -->
-      <!-- othervise it depends on lens type and custom function, if there is one -->
-      <scale_to_hfov>true</scale_to_hfov>
-      <!-- clip everything that is outside of this angle -->
-      <cutoff_angle>3.1415</cutoff_angle>
-      <!-- resolution of the cubemap texture, the highter it is - the sharper is your image -->
-      <env_texture_size>512</env_texture_size>
-    </lens>
-  </camera>
-      <plugin name="left_fisheye_camera_controller" filename="libgazebo_ros_camera.so">
-        <alwaysOn>true</alwaysOn>
-        <updateRate>0.0</updateRate>
-        <cameraName>fisheyecamera</cameraName>
-        <imageTopicName>image_raw</imageTopicName>
-        <cameraInfoTopicName>camera_info</cameraInfoTopicName>
-        <frameName>camera_left_link</frameName>
-        <rightFrameName>camera_right_link</rightFrameName>
-        <hackBaseline>0.07</hackBaseline>
-        <distortionK1>0.0</distortionK1>
-        <distortionK2>0.0</distortionK2>
-        <distortionK3>0.0</distortionK3>
-        <distortionT1>0.0</distortionT1>
-        <distortionT2>0.0</distortionT2>
-      </plugin>
-  <always_on>1</always_on>
-  <update_rate>30</update_rate>
-</sensor>
+        <camera>
+          <horizontal_fov>6.283</horizontal_fov>
+          <image>
+            <width>320</width>
+            <height>240</height>
+          </image>
+          <clip>
+            <near>0.1</near>
+            <far>100</far>
+          </clip>
+           <!-- A new section named `lens`. -->
+          <lens>
+            <!-- type element is mandatory -->
+            <type>custom</type>
+            <!-- manually defined mapping function r = c1*f*fun(theta/c2 + c3) -->
+            <!-- More information here: https://en.wikipedia.org/wiki/Fisheye_lens#Mapping_function -->
+            <custom_function>
+              <c1>1.05</c1>   <!-- linear scaling -->
+              <c2>4</c2>      <!-- angle scaling -->
+              <f>1.0</f>      <!-- one more scaling parameter -->
+              <fun>tan</fun>  <!-- one of sin,tan,id -->
+            </custom_function>
+            <!-- if it is set to `true` your horizontal FOV will ramain as defined -->
+            <!-- othervise it depends on lens type and custom function, if there is one -->
+            <scale_to_hfov>true</scale_to_hfov>
+            <!-- clip everything that is outside of this angle -->
+            <cutoff_angle>3.1415</cutoff_angle>
+            <!-- resolution of the cubemap texture, the highter it is - the sharper is your image -->
+            <env_texture_size>512</env_texture_size>
+          </lens>
+        </camera>
+        <plugin name="left_fisheye_camera_controller" filename="libgazebo_ros_camera.so">
+          <alwaysOn>true</alwaysOn>
+          <updateRate>0.0</updateRate>
+          <cameraName>fisheyecamera</cameraName>
+          <imageTopicName>image_raw</imageTopicName>
+          <cameraInfoTopicName>camera_info</cameraInfoTopicName>
+          <frameName>camera_left_link</frameName>
+          <rightFrameName>camera_right_link</rightFrameName>
+          <hackBaseline>0.07</hackBaseline>
+          <distortionK1>0.0</distortionK1>
+          <distortionK2>0.0</distortionK2>
+          <distortionK3>0.0</distortionK3>
+          <distortionT1>0.0</distortionT1>
+          <distortionT2>0.0</distortionT2>
+        </plugin>
+        <always_on>1</always_on>
+        <update_rate>30</update_rate>
+    </sensor>
   </gazebo>
   <gazebo reference="right_camera_link">
     <material>Gazebo/Green</material>
       <sensor name="right_camera" type="wideanglecamera">
-  <camera>
-    <horizontal_fov>6.283</horizontal_fov>
-    <image>
-      <width>320</width>
-      <height>240</height>
-    </image>
-    <clip>
-      <near>0.1</near>
-      <far>100</far>
-    </clip>
-     <!-- A new section named `lens`. -->
-    <lens>
-      <!-- type element is mandatory -->
-      <type>custom</type>
-      <!-- manually defined mapping function r = c1*f*fun(theta/c2 + c3) -->
-      <!-- More information here: https://en.wikipedia.org/wiki/Fisheye_lens#Mapping_function -->
-      <custom_function>
-        <c1>1.05</c1>   <!-- linear scaling -->
-        <c2>4</c2>      <!-- angle scaling -->
-        <f>1.0</f>      <!-- one more scaling parameter -->
-        <fun>tan</fun>  <!-- one of sin,tan,id -->
-      </custom_function>
-      <!-- if it is set to `true` your horizontal FOV will ramain as defined -->
-      <!-- othervise it depends on lens type and custom function, if there is one -->
-      <scale_to_hfov>true</scale_to_hfov>
-      <!-- clip everything that is outside of this angle -->
-      <cutoff_angle>3.1415</cutoff_angle>
-      <!-- resolution of the cubemap texture, the highter it is - the sharper is your image -->
-      <env_texture_size>512</env_texture_size>
-    </lens>
-  </camera>
-      <plugin name="right_fisheye_camera_controller" filename="libgazebo_ros_camera.so">
-        <alwaysOn>true</alwaysOn>
-        <updateRate>0.0</updateRate>
-        <cameraName>fisheyecamera</cameraName>
-        <imageTopicName>image_raw</imageTopicName>
-        <cameraInfoTopicName>camera_info</cameraInfoTopicName>
-        <frameName>camera_left_link</frameName>
-        <rightFrameName>camera_right_link</rightFrameName>
-        <hackBaseline>0.07</hackBaseline>
-        <distortionK1>0.0</distortionK1>
-        <distortionK2>0.0</distortionK2>
-        <distortionK3>0.0</distortionK3>
-        <distortionT1>0.0</distortionT1>
-        <distortionT2>0.0</distortionT2>
-      </plugin>
-  <always_on>1</always_on>
-  <update_rate>30</update_rate>
-</sensor>
+          <camera>
+            <horizontal_fov>6.283</horizontal_fov>
+            <image>
+              <width>320</width>
+              <height>240</height>
+            </image>
+            <clip>
+              <near>0.1</near>
+              <far>100</far>
+            </clip>
+             <!-- A new section named `lens`. -->
+            <lens>
+              <!-- type element is mandatory -->
+              <type>custom</type>
+              <!-- manually defined mapping function r = c1*f*fun(theta/c2 + c3) -->
+              <!-- More information here: https://en.wikipedia.org/wiki/Fisheye_lens#Mapping_function -->
+              <custom_function>
+                <c1>1.05</c1>   <!-- linear scaling -->
+                <c2>4</c2>      <!-- angle scaling -->
+                <f>1.0</f>      <!-- one more scaling parameter -->
+                <fun>tan</fun>  <!-- one of sin,tan,id -->
+              </custom_function>
+              <!-- if it is set to `true` your horizontal FOV will ramain as defined -->
+              <!-- othervise it depends on lens type and custom function, if there is one -->
+              <scale_to_hfov>true</scale_to_hfov>
+              <!-- clip everything that is outside of this angle -->
+              <cutoff_angle>3.1415</cutoff_angle>
+              <!-- resolution of the cubemap texture, the highter it is - the sharper is your image -->
+              <env_texture_size>512</env_texture_size>
+            </lens>
+          </camera>
+          <plugin name="right_fisheye_camera_controller" filename="libgazebo_ros_camera.so">
+            <alwaysOn>true</alwaysOn>
+            <updateRate>0.0</updateRate>
+            <cameraName>fisheyecamera</cameraName>
+            <imageTopicName>image_raw</imageTopicName>
+            <cameraInfoTopicName>camera_info</cameraInfoTopicName>
+            <frameName>camera_left_link</frameName>
+            <rightFrameName>camera_right_link</rightFrameName>
+            <hackBaseline>0.07</hackBaseline>
+            <distortionK1>0.0</distortionK1>
+            <distortionK2>0.0</distortionK2>
+            <distortionK3>0.0</distortionK3>
+            <distortionT1>0.0</distortionT1>
+            <distortionT2>0.0</distortionT2>
+          </plugin>
+          <always_on>1</always_on>
+          <update_rate>30</update_rate>
+       </sensor>
   </gazebo>
   <!-- Hokuyo LIDAR for simulation -->

File: leobot_description/urdf/sensors/camera.urdf.xacro (robot description, xacro)
@@ -13,5 +13,5 @@
         </link>
         <joint name="head_${prefix}_camera_joint" type="fixed">
-            <origin xyz="${side*(camera_radius + parent_width/2) - side*0.005} ${-parent_height/2 + camera_radius} 0" rpy="0 ${pi/2 + side * pi/2 } 0"/>
+            <origin xyz="${side*(camera_radius + parent_width/2) - side*0.005} ${-parent_height/2 + camera_radius} 0" rpy="${pi/2 + side * pi/2 } ${pi/2 + side * pi/2 } 0"/>
             <parent link="${parent_link_name}" />
             <child link="${prefix}_camera_link" />
