Commit message: Revert "Indent xacro files with 4 spaces per level and delete the optional xml declaration"
This reverts commit 3711d6c2502273858bc2c684381f7cef3361f35a.

File: leobot_description/robot/leobot.gazebo.xacro (robot description, xacro)
@@ -1,223 +1,224 @@
+<?xml version="1.0"?>
 <robot xmlns:xacro="http://ros.org/wiki/xacro" name="leobot">
-    <xacro:include filename="$(find leobot_description)/robot/robot.urdf.xacro"/>
-    <gazebo>
-        <plugin name="gazebo_ros_control" filename="libgazebo_ros_control.so">
-            <robotNamespace>/</robotNamespace>
-            <robotSimType>gazebo_ros_control/DefaultRobotHWSim</robotSimType>
+  <xacro:include filename="$(find leobot_description)/robot/robot.urdf.xacro"/>
+  <gazebo>
+    <plugin name="gazebo_ros_control" filename="libgazebo_ros_control.so">
+      <robotNamespace>/</robotNamespace>
+      <robotSimType>gazebo_ros_control/DefaultRobotHWSim</robotSimType>
+    </plugin>
+  </gazebo>
+  <gazebo reference="base_link">
+    <mu1 value="1.0"/>
+    <mu2 value="1.0"/>
+    <kp value="10000000.0"/>
+    <kd value="1.0"/>
+    <material>Gazebo/White</material>
+  </gazebo>
+  <gazebo reference="head_link">
+    <mu1 value="1.0"/>
+    <mu2 value="1.0"/>
+    <kp value="10000000.0"/>
+    <kd value="1.0"/>
+    <material>Gazebo/White</material>
+  </gazebo>
+  <gazebo reference="neck_link">
+    <mu1 value="1.0"/>
+    <mu2 value="1.0"/>
+    <kp value="10000000.0"/>
+    <kd value="1.0"/>
+    <material>Gazebo/White</material>
+  </gazebo>
+  <gazebo reference="FL_wheel_link">
+    <mu1 value="1.0"/>
+    <mu2 value="1.0"/>
+    <kp value="10000000.0"/>
+    <kd value="1.0"/>
+    <material>Gazebo/Blue</material>
+  </gazebo>
+  <gazebo reference="FR_wheel_link">
+    <mu1 value="1.0"/>
+    <mu2 value="1.0"/>
+    <kp value="10000000.0"/>
+    <kd value="1.0"/>
+    <material>Gazebo/Blue</material>
+  </gazebo>
+  <gazebo reference="RL_wheel_link">
+    <mu1 value="1.0"/>
+    <mu2 value="1.0"/>
+    <kp value="10000000.0"/>
+    <kd value="1.0"/>
+    <material>Gazebo/Blue</material>
+  </gazebo>
+  <gazebo reference="RR_wheel_link">
+    <mu1 value="1.0"/>
+    <mu2 value="1.0"/>
+    <kp value="10000000.0"/>
+    <kd value="1.0"/>
+    <material>Gazebo/Blue</material>
+  </gazebo>
+  <gazebo reference="FR_motor_holder">
+    <mu1 value="1.0"/>
+    <mu2 value="1.0"/>
+    <kp value="10000000.0"/>
+    <kd value="1.0"/>
+    <material>Gazebo/Red</material>
+  </gazebo>
+  <gazebo reference="FL_motor_holder">
+    <mu1 value="1.0"/>
+    <mu2 value="1.0"/>
+    <kp value="10000000.0"/>
+    <kd value="1.0"/>
+    <material>Gazebo/Red</material>
+  </gazebo>
+  <gazebo reference="RL_motor_holder">
+    <mu1 value="1.0"/>
+    <mu2 value="1.0"/>
+    <kp value="10000000.0"/>
+    <kd value="1.0"/>
+    <material>Gazebo/Red</material>
+  </gazebo>
+  <gazebo reference="RR_motor_holder">
+    <mu1 value="1.0"/>
+    <mu2 value="1.0"/>
+    <kp value="10000000.0"/>
+    <kd value="1.0"/>
+    <material>Gazebo/Red</material>
+  </gazebo>
+  <gazebo reference="left_camera_link">
+    <material>Gazebo/Green</material>
+    <sensor name="left_camera" type="wideanglecamera">
+        <camera>
+          <horizontal_fov>6.283</horizontal_fov>
+          <image>
+            <width>320</width>
+            <height>240</height>
+          </image>
+          <clip>
+            <near>0.1</near>
+            <far>100</far>
+          </clip>
+           <!-- A new section named `lens`. -->
+          <lens>
+            <!-- type element is mandatory -->
+            <type>custom</type>
+            <!-- manually defined mapping function r = c1*f*fun(theta/c2 + c3) -->
+            <!-- More information here: https://en.wikipedia.org/wiki/Fisheye_lens#Mapping_function -->
+            <custom_function>
+              <c1>1.05</c1>   <!-- linear scaling -->
+              <c2>4</c2>      <!-- angle scaling -->
+              <f>1.0</f>      <!-- one more scaling parameter -->
+              <fun>tan</fun>  <!-- one of sin,tan,id -->
+            </custom_function>
+            <!-- if it is set to `true` your horizontal FOV will ramain as defined -->
+            <!-- othervise it depends on lens type and custom function, if there is one -->
+            <scale_to_hfov>true</scale_to_hfov>
+            <!-- clip everything that is outside of this angle -->
+            <cutoff_angle>3.1415</cutoff_angle>
+            <!-- resolution of the cubemap texture, the higher it is - the sharper is your image -->
+            <env_texture_size>512</env_texture_size>
+          </lens>
+        </camera>
+        <plugin name="left_fisheye_camera_controller" filename="libgazebo_ros_camera.so">
+          <alwaysOn>true</alwaysOn>
+          <updateRate>0.0</updateRate>
+          <cameraName>left_fisheye_camera</cameraName>
+          <imageTopicName>image_raw</imageTopicName>
+          <cameraInfoTopicName>camera_info</cameraInfoTopicName>
+          <frameName>camera_left_link</frameName>
+          <hackBaseline>0.07</hackBaseline>
+          <distortionK1>0.0</distortionK1>
+          <distortionK2>0.0</distortionK2>
+          <distortionK3>0.0</distortionK3>
+          <distortionT1>0.0</distortionT1>
+          <distortionT2>0.0</distortionT2>
         </plugin>
-    </gazebo>
-    <gazebo reference="base_link">
-        <mu1 value="1.0"/>
-        <mu2 value="1.0"/>
-        <kp value="10000000.0"/>
-        <kd value="1.0"/>
-        <material>Gazebo/White</material>
-    </gazebo>
-    <gazebo reference="head_link">
-        <mu1 value="1.0"/>
-        <mu2 value="1.0"/>
-        <kp value="10000000.0"/>
-        <kd value="1.0"/>
-        <material>Gazebo/White</material>
-    </gazebo>
-    <gazebo reference="neck_link">
-        <mu1 value="1.0"/>
-        <mu2 value="1.0"/>
-        <kp value="10000000.0"/>
-        <kd value="1.0"/>
-        <material>Gazebo/White</material>
-    </gazebo>
-    <gazebo reference="FL_wheel_link">
-        <mu1 value="1.0"/>
-        <mu2 value="1.0"/>
-        <kp value="10000000.0"/>
-        <kd value="1.0"/>
-        <material>Gazebo/Blue</material>
-    </gazebo>
-    <gazebo reference="FR_wheel_link">
-        <mu1 value="1.0"/>
-        <mu2 value="1.0"/>
-        <kp value="10000000.0"/>
-        <kd value="1.0"/>
-        <material>Gazebo/Blue</material>
-    </gazebo>
-    <gazebo reference="RL_wheel_link">
-        <mu1 value="1.0"/>
-        <mu2 value="1.0"/>
-        <kp value="10000000.0"/>
-        <kd value="1.0"/>
-        <material>Gazebo/Blue</material>
-    </gazebo>
-    <gazebo reference="RR_wheel_link">
-        <mu1 value="1.0"/>
-        <mu2 value="1.0"/>
-        <kp value="10000000.0"/>
-        <kd value="1.0"/>
-        <material>Gazebo/Blue</material>
-    </gazebo>
-    <gazebo reference="FR_motor_holder">
-        <mu1 value="1.0"/>
-        <mu2 value="1.0"/>
-        <kp value="10000000.0"/>
-        <kd value="1.0"/>
-        <material>Gazebo/Red</material>
-    </gazebo>
-    <gazebo reference="FL_motor_holder">
-        <mu1 value="1.0"/>
-        <mu2 value="1.0"/>
-        <kp value="10000000.0"/>
-        <kd value="1.0"/>
-        <material>Gazebo/Red</material>
-    </gazebo>
-    <gazebo reference="RL_motor_holder">
-        <mu1 value="1.0"/>
-        <mu2 value="1.0"/>
-        <kp value="10000000.0"/>
-        <kd value="1.0"/>
-        <material>Gazebo/Red</material>
-    </gazebo>
-    <gazebo reference="RR_motor_holder">
-        <mu1 value="1.0"/>
-        <mu2 value="1.0"/>
-        <kp value="10000000.0"/>
-        <kd value="1.0"/>
-        <material>Gazebo/Red</material>
-    </gazebo>
-    <gazebo reference="left_camera_link">
-        <material>Gazebo/Green</material>
-        <sensor name="left_camera" type="wideanglecamera">
-            <camera>
-                <horizontal_fov>6.283</horizontal_fov>
-                <image>
-                    <width>320</width>
-                    <height>240</height>
-                </image>
-                <clip>
-                    <near>0.1</near>
-                    <far>100</far>
-                </clip>
-                <!-- A new section named `lens`. -->
-                <lens>
-                    <!-- type element is mandatory -->
-                    <type>custom</type>
-                    <!-- manually defined mapping function r = c1*f*fun(theta/c2 + c3) -->
-                    <!-- More information here: https://en.wikipedia.org/wiki/Fisheye_lens#Mapping_function -->
-                    <custom_function>
-                        <c1>1.05</c1>   <!-- linear scaling -->
-                        <c2>4</c2>      <!-- angle scaling -->
-                        <f>1.0</f>      <!-- one more scaling parameter -->
-                        <fun>tan</fun>  <!-- one of sin,tan,id -->
-                    </custom_function>
-                    <!-- if it is set to `true` your horizontal FOV will ramain as defined -->
-                    <!-- othervise it depends on lens type and custom function, if there is one -->
-                    <scale_to_hfov>true</scale_to_hfov>
-                    <!-- clip everything that is outside of this angle -->
-                    <cutoff_angle>3.1415</cutoff_angle>
-                    <!-- resolution of the cubemap texture, the higher it is - the sharper is your image -->
-                    <env_texture_size>512</env_texture_size>
-                </lens>
-            </camera>
-            <plugin name="left_fisheye_camera_controller" filename="libgazebo_ros_camera.so">
-                <alwaysOn>true</alwaysOn>
-                <updateRate>0.0</updateRate>
-                <cameraName>left_fisheye_camera</cameraName>
-                <imageTopicName>image_raw</imageTopicName>
-                <cameraInfoTopicName>camera_info</cameraInfoTopicName>
-                <frameName>camera_left_link</frameName>
-                <hackBaseline>0.07</hackBaseline>
-                <distortionK1>0.0</distortionK1>
-                <distortionK2>0.0</distortionK2>
-                <distortionK3>0.0</distortionK3>
-                <distortionT1>0.0</distortionT1>
-                <distortionT2>0.0</distortionT2>
-            </plugin>
-            <always_on>1</always_on>
-            <update_rate>30</update_rate>
-        </sensor>
-    </gazebo>
-    <gazebo reference="right_camera_link">
-        <material>Gazebo/Green</material>
-        <sensor name="right_camera" type="wideanglecamera">
-            <camera>
-                <horizontal_fov>6.283</horizontal_fov>
-                <image>
-                    <width>320</width>
-                    <height>240</height>
-                </image>
-                <clip>
-                    <near>0.1</near>
-                    <far>100</far>
-                </clip>
-                <!-- A new section named `lens`. -->
-                <lens>
-                    <!-- type element is mandatory -->
-                    <type>custom</type>
-                    <!-- manually defined mapping function r = c1*f*fun(theta/c2 + c3) -->
-                    <!-- More information here: https://en.wikipedia.org/wiki/Fisheye_lens#Mapping_function -->
-                    <custom_function>
-                        <c1>1.05</c1>   <!-- linear scaling -->
-                        <c2>4</c2>      <!-- angle scaling -->
-                        <f>1.0</f>      <!-- one more scaling parameter -->
-                        <fun>tan</fun>  <!-- one of sin,tan,id -->
-                    </custom_function>
-                    <!-- if it is set to `true` your horizontal FOV will ramain as defined -->
-                    <!-- othervise it depends on lens type and custom function, if there is one -->
-                    <scale_to_hfov>true</scale_to_hfov>
-                    <!-- clip everything that is outside of this angle -->
-                    <cutoff_angle>3.1415</cutoff_angle>
-                    <!-- resolution of the cubemap texture, the higher it is - the sharper is your image -->
-                    <env_texture_size>512</env_texture_size>
-                </lens>
-            </camera>
-            <plugin name="right_fisheye_camera_controller" filename="libgazebo_ros_camera.so">
-                <alwaysOn>true</alwaysOn>
-                <updateRate>0.0</updateRate>
-                <cameraName>right_fisheye_camera</cameraName>
-                <imageTopicName>image_raw</imageTopicName>
-                <cameraInfoTopicName>camera_info</cameraInfoTopicName>
-                <frameName>camera_left_link</frameName>
-                <hackBaseline>0.07</hackBaseline>
-                <distortionK1>0.0</distortionK1>
-                <distortionK2>0.0</distortionK2>
-                <distortionK3>0.0</distortionK3>
-                <distortionT1>0.0</distortionT1>
-                <distortionT2>0.0</distortionT2>
-            </plugin>
-            <always_on>1</always_on>
-            <update_rate>30</update_rate>
-        </sensor>
-    </gazebo>
-    <!-- Hokuyo LIDAR for simulation -->
-    <gazebo reference="laser_link">
-        <material>Gazebo/Green</material>
-        <sensor type="ray" name="laser">
-            <pose>0 0 0 0 0 0</pose>
-            <visualize>false</visualize>
-            <update_rate>40</update_rate>
-            <ray>
-                <scan>
-                    <horizontal>
-                        <samples>1081</samples>
-                        <resolution>1</resolution>
-                        <min_angle>-1.570796</min_angle>
-                        <max_angle>1.570796</max_angle>
-                    </horizontal>
-                </scan>
-                <range>
-                    <min>0.60</min>
-                    <max>10.0</max>
-                    <resolution>0.01</resolution>
-                </range>
-                <noise>
-                    <type>gaussian</type>
-                    <mean>0.0</mean>
-                    <stddev>0.01</stddev>
-                </noise>
-            </ray>
-            <plugin name="gazebo_ros_hokuyo_controller" filename="libgazebo_ros_laser.so">
-                <topicName>laser/scan</topicName>
-                <frameName>laser_link</frameName>
-            </plugin>
-        </sensor>
+        <always_on>1</always_on>
+        <update_rate>30</update_rate>
+    </sensor>
+  </gazebo>
+  <gazebo reference="right_camera_link">
+    <material>Gazebo/Green</material>
+      <sensor name="right_camera" type="wideanglecamera">
+          <camera>
+            <horizontal_fov>6.283</horizontal_fov>
+            <image>
+              <width>320</width>
+              <height>240</height>
+            </image>
+            <clip>
+              <near>0.1</near>
+              <far>100</far>
+            </clip>
+             <!-- A new section named `lens`. -->
+            <lens>
+              <!-- type element is mandatory -->
+              <type>custom</type>
+              <!-- manually defined mapping function r = c1*f*fun(theta/c2 + c3) -->
+              <!-- More information here: https://en.wikipedia.org/wiki/Fisheye_lens#Mapping_function -->
+              <custom_function>
+                <c1>1.05</c1>   <!-- linear scaling -->
+                <c2>4</c2>      <!-- angle scaling -->
+                <f>1.0</f>      <!-- one more scaling parameter -->
+                <fun>tan</fun>  <!-- one of sin,tan,id -->
+              </custom_function>
+              <!-- if it is set to `true` your horizontal FOV will ramain as defined -->
+              <!-- othervise it depends on lens type and custom function, if there is one -->
+              <scale_to_hfov>true</scale_to_hfov>
+              <!-- clip everything that is outside of this angle -->
+              <cutoff_angle>3.1415</cutoff_angle>
+              <!-- resolution of the cubemap texture, the higher it is - the sharper is your image -->
+              <env_texture_size>512</env_texture_size>
+            </lens>
+          </camera>
+          <plugin name="right_fisheye_camera_controller" filename="libgazebo_ros_camera.so">
+            <alwaysOn>true</alwaysOn>
+            <updateRate>0.0</updateRate>
+            <cameraName>right_fisheye_camera</cameraName>
+            <imageTopicName>image_raw</imageTopicName>
+            <cameraInfoTopicName>camera_info</cameraInfoTopicName>
+            <frameName>camera_left_link</frameName>
+            <hackBaseline>0.07</hackBaseline>
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
File: leobot_description/robot/leobot.rviz.xacro (robot description, xacro)
@@ -1,3 +1,4 @@
+<?xml version="1.0"?>
 <robot xmlns:xacro="http://ros.org/wiki/xacro" name="leobot">
-    <xacro:include filename="$(find leobot_description)/robot/robot.urdf.xacro"/>
+  <xacro:include filename="$(find leobot_description)/robot/robot.urdf.xacro"/>
 </robot>
