Commit message: Reverted to simple cameras

File: leobot_description/robot/leobot.gazebo.xacro (robot description, xacro)
@@ -86,43 +86,49 @@
     <gazebo reference="left_camera_link">
         <material>Gazebo/Green</material>
-        <sensor name="left_camera" type="wideanglecamera">
-            <camera>
-                <horizontal_fov>6.283</horizontal_fov>
+        <sensor type="multicamera" name="stereo_camera">
+            <update_rate>30.0</update_rate>
+            <camera name="left">
+                <horizontal_fov>1.3962634</horizontal_fov>
                 <image>
-                    <width>320</width>
-                    <height>240</height>
+                    <width>800</width>
+                    <height>800</height>
+                    <format>R8G8B8</format>
                 </image>
                 <clip>
-                    <near>0.1</near>
-                    <far>100</far>
+                    <near>0.02</near>
+                    <far>300</far>
                 </clip>
-                <!-- A new section named `lens`. -->
-                <lens>
-                    <!-- type element is mandatory -->
-                    <type>custom</type>
-                    <!-- manually defined mapping function r = c1*f*fun(theta/c2 + c3) -->
-                    <!-- More information here: https://en.wikipedia.org/wiki/Fisheye_lens#Mapping_function -->
-                    <custom_function>
-                        <c1>1.05</c1>   <!-- linear scaling -->
-                        <c2>4</c2>      <!-- angle scaling -->
-                        <f>1.0</f>      <!-- one more scaling parameter -->
-                        <fun>tan</fun>  <!-- one of sin,tan,id -->
-                    </custom_function>
-                    <!-- if it is set to `true` your horizontal FOV will ramain as defined -->
-                    <!-- othervise it depends on lens type and custom function, if there is one -->
-                    <scale_to_hfov>true</scale_to_hfov>
-                    <!-- clip everything that is outside of this angle -->
-                    <cutoff_angle>3.1415</cutoff_angle>
-                    <!-- resolution of the cubemap texture, the higher it is - the sharper is your image -->
-                    <env_texture_size>512</env_texture_size>
-                </lens>
+                <noise>
+                    <type>gaussian</type>
+                    <mean>0.0</mean>
+                    <stddev>0.007</stddev>
+                </noise>
             </camera>
-            <plugin name="left_fisheye_camera_controller" filename="libgazebo_ros_camera.so">
+            <camera name="right">
+                <pose>0 -0.07 0 0 0 0</pose>
+                <horizontal_fov>1.3962634</horizontal_fov>
+                <image>
+                    <width>800</width>
+                    <height>800</height>
+                    <format>R8G8B8</format>
+                </image>
+                <clip>
+                    <near>0.02</near>
+                    <far>300</far>
+                </clip>
+                <noise>
+                    <type>gaussian</type>
+                    <mean>0.0</mean>
+                    <stddev>0.007</stddev>
+                </noise>
+            </camera>
+            <plugin name="stereo_camera_controller" filename="libgazebo_ros_multicamera.so">
                 <alwaysOn>true</alwaysOn>
                 <updateRate>0.0</updateRate>
-                <cameraName>left_fisheye_camera</cameraName>
+                <cameraName>stereocamera</cameraName>
                 <imageTopicName>image_raw</imageTopicName>
                 <cameraInfoTopicName>camera_info</cameraInfoTopicName>
-                <frameName>camera_left_link</frameName>
+                <frameName>left_camera_link</frameName>
+                <rightFrameName>right_camera_link</rightFrameName>
                 <hackBaseline>0.07</hackBaseline>
                 <distortionK1>0.0</distortionK1>
@@ -132,59 +138,8 @@
                 <distortionT2>0.0</distortionT2>
             </plugin>
-            <always_on>1</always_on>
-            <update_rate>30</update_rate>
         </sensor>
     </gazebo>
     <gazebo reference="right_camera_link">
         <material>Gazebo/Green</material>
-        <sensor name="right_camera" type="wideanglecamera">
-            <camera>
-                <horizontal_fov>6.283</horizontal_fov>
-                <image>
-                    <width>320</width>
-                    <height>240</height>
-                </image>
-                <clip>
-                    <near>0.1</near>
-                    <far>100</far>
-                </clip>
-                <!-- A new section named `lens`. -->
-                <lens>
-                    <!-- type element is mandatory -->
-                    <type>custom</type>
-                    <!-- manually defined mapping function r = c1*f*fun(theta/c2 + c3) -->
-                    <!-- More information here: https://en.wikipedia.org/wiki/Fisheye_lens#Mapping_function -->
-                    <custom_function>
-                        <c1>1.05</c1>   <!-- linear scaling -->
-                        <c2>4</c2>      <!-- angle scaling -->
-                        <f>1.0</f>      <!-- one more scaling parameter -->
-                        <fun>tan</fun>  <!-- one of sin,tan,id -->
-                    </custom_function>
-                    <!-- if it is set to `true` your horizontal FOV will ramain as defined -->
-                    <!-- othervise it depends on lens type and custom function, if there is one -->
-                    <scale_to_hfov>true</scale_to_hfov>
-                    <!-- clip everything that is outside of this angle -->
-                    <cutoff_angle>3.1415</cutoff_angle>
-                    <!-- resolution of the cubemap texture, the higher it is - the sharper is your image -->
-                    <env_texture_size>512</env_texture_size>
-                </lens>
-            </camera>
-            <plugin name="right_fisheye_camera_controller" filename="libgazebo_ros_camera.so">
-                <alwaysOn>true</alwaysOn>
-                <updateRate>0.0</updateRate>
-                <cameraName>right_fisheye_camera</cameraName>
-                <imageTopicName>image_raw</imageTopicName>
-                <cameraInfoTopicName>camera_info</cameraInfoTopicName>
-                <frameName>camera_left_link</frameName>
-                <hackBaseline>0.07</hackBaseline>
-                <distortionK1>0.0</distortionK1>
-                <distortionK2>0.0</distortionK2>
-                <distortionK3>0.0</distortionK3>
-                <distortionT1>0.0</distortionT1>
-                <distortionT2>0.0</distortionT2>
-            </plugin>
-            <always_on>1</always_on>
-            <update_rate>30</update_rate>
-        </sensor>
     </gazebo>
     <!-- Hokuyo LIDAR for simulation -->

File: leobot_description/robot/robot.urdf.xacro (robot description, xacro)
@@ -57,22 +57,42 @@
     <link name="camera_stick_link">
         <visual>
-            <xacro:box_geometry width="${camera_stick_width}" height="${camera_stick_height}" depth="${camera_stick_length}"/>
+            <xacro:box_geometry width="${camera_stick_width}" height="${camera_stick_height}"
+                                depth="${camera_stick_length}"/>
             <xacro:yellow_material/>
         </visual>
-        <xacro:box_collision width="${camera_stick_width}" height="${camera_stick_height}" depth="${camera_stick_length}"/>
-        <xacro:box_inertia   width="${camera_stick_width}" height="${camera_stick_height}" depth="${camera_stick_length}" mass="${camera_stick_mass}"/>
+        <xacro:box_collision width="${camera_stick_width}" height="${camera_stick_height}"
+                             depth="${camera_stick_length}"/>
+        <xacro:box_inertia   width="${camera_stick_width}" height="${camera_stick_height}"
+                             depth="${camera_stick_length}" mass="${camera_stick_mass}"/>
     </link>
-    <joint name="head_camera_stick_joint" type="continuous">
+    <joint name="head_camera_stick_joint" type="revolute">
         <origin rpy="${pi/2} ${pi/2} ${pi}"
                 xyz="0 ${camera_stick_length/2 - head_height/2} ${head_width/2 + camera_stick_width/2}"/>
         <parent link="head_link"/>
         <child link="camera_stick_link"/>
+        <limit effort="10" velocity="10" lower="${-pi/2}" upper="${pi/2}" />
     </joint>
-    <xacro:fish_camera prefix="left"  parent_link_name="camera_stick_link" parent_height="${camera_stick_height}" parent_width="${camera_stick_width}" side="1"/>
-    <xacro:fish_camera prefix="right" parent_link_name="camera_stick_link" parent_height="${camera_stick_height}" parent_width="${camera_stick_width}" side="-1"/>
+    <transmission name="head_transmission">
+        <type>transmission_interface/SimpleTransmission</type>
+        <joint name="head_camera_stick_joint">
+            <hardwareInterface>hardware_interface/EffortJointInterface</hardwareInterface>
+        </joint>
+        <actuator name="head_camera_stick_joint">
+            <hardwareInterface>EffortJointInterface</hardwareInterface>
+            <mechanicalReduction>1</mechanicalReduction>
+        </actuator>
+    </transmission>
+    <xacro:simple_camera prefix="left"  parent_link_name="camera_stick_link" parent_height="${camera_stick_height}"
+                  parent_width="${camera_stick_width}" side="1"/>
+    <xacro:simple_camera prefix="right" parent_link_name="camera_stick_link" parent_height="${camera_stick_height}"
+                  parent_width="${camera_stick_width}" side="-1"/>
     <xacro:lidar_hokuyo parent_link_name="base_link" parent_height="${base_length}"/>
-    <xacro:mecanum_wheel prefix="FL" wheel_type="2" side="1"  position="1"  parent_length="${base_width}" parent_height="${base_length}" parent_width="${base_height}"/>
-    <xacro:mecanum_wheel prefix="FR" wheel_type="1" side="-1" position="1"  parent_length="${base_width}" parent_height="${base_length}" parent_width="${base_height}"/>
-    <xacro:mecanum_wheel prefix="RL" wheel_type="1" side="1"  position="-1" parent_length="${base_width}" parent_height="${base_length}" parent_width="${base_height}"/>
-    <xacro:mecanum_wheel prefix="RR" wheel_type="2" side="-1" position="-1" parent_length="${base_width}" parent_height="${base_length}" parent_width="${base_height}"/>
+    <xacro:mecanum_wheel prefix="FL" wheel_type="2" side="1"  position="1"  parent_length="${base_width}"
+                         parent_height="${base_length}" parent_width="${base_height}"/>
+    <xacro:mecanum_wheel prefix="FR" wheel_type="1" side="-1" position="1"  parent_length="${base_width}"
+                         parent_height="${base_length}" parent_width="${base_height}"/>
+    <xacro:mecanum_wheel prefix="RL" wheel_type="1" side="1"  position="-1" parent_length="${base_width}"
+                         parent_height="${base_length}" parent_width="${base_height}"/>
+    <xacro:mecanum_wheel prefix="RR" wheel_type="2" side="-1" position="-1" parent_length="${base_width}"
+                         parent_height="${base_length}" parent_width="${base_height}"/>
 </robot>

File: leobot_description/urdf/sensors/camera.urdf.xacro (robot description, xacro)
@@ -1,4 +1,5 @@
 <robot xmlns:xacro="http://ros.org/wiki/xacro">
     <xacro:property name="camera_radius" value="0.025"/>
+    <xacro:property name="camera_size" value="0.03"/>
     <xacro:property name="camera_mass"   value="0.1"/>
     <xacro:macro name="fish_camera" params="prefix parent_link_name parent_height side parent_width">
@@ -18,3 +19,20 @@
         </joint>
     </xacro:macro>
+    <xacro:macro name="simple_camera" params="prefix parent_link_name parent_height side parent_width">
+        <link name="${prefix}_camera_link">
+            <visual>
+              <xacro:box_geometry width="${camera_size}" height="${camera_size}" depth="${camera_size}"/>
+              <xacro:green_material/>
+            </visual>
+            <xacro:box_collision width="${camera_size}" height="${camera_size}" depth="${camera_size}"/>
+            <xacro:box_inertia mass="${camera_mass}" width="${camera_size}" height="${camera_size}"
+                               depth="${camera_size}"/>
+        </link>
+        <joint name="${prefix}_camera_joint" type="fixed">
+            <origin xyz="${(-camera_size - parent_width) / 2} ${side * (parent_height - camera_size / 2) / 2} 0"
+                    rpy="${-pi / 2} ${pi / 2} ${pi / 2}"/>
+            <parent link="${parent_link_name}"/>
+            <child link="${prefix}_camera_link"/>
+        </joint>
+    </xacro:macro>
 </robot>

Commit message: Add footprint, remove unneeded line and topic

File: leobot_description/robot/leobot.gazebo.xacro (robot description, xacro)
@@ -223,5 +223,4 @@
     <gazebo>
     <plugin name="object_controller" filename="libgazebo_ros_planar_move.so">
-      <commandTopic>/wheel_diff_drive_controller/cmd_vel</commandTopic>
       <commandTopic>/teleop_twist_keyboard/cmd_vel</commandTopic>
       <commandTopic>/joy_teleop/cmd_vel</commandTopic>
@@ -229,5 +228,5 @@
       <odometryFrame>odom</odometryFrame>
       <odometryRate>10.0</odometryRate>
-      <robotBaseFrame>FL_wheel_link</robotBaseFrame>
+      <robotBaseFrame>base_footprint</robotBaseFrame>
     </plugin>
   </gazebo>

File: leobot_description/robot/robot.urdf.xacro (robot description, xacro)
@@ -9,4 +9,7 @@
     <xacro:property name="base_height" value="0.5"/>
     <xacro:property name="base_mass"   value="10"/>
+    <xacro:property name="base_footprint_length" value="0.001"/>
+    <xacro:property name="base_footprint_height" value="0.001"/>
+    <xacro:property name="base_footprint_width" value="0.001"/>
     <xacro:property name="neck_width"  value="0.04"/>
     <xacro:property name="neck_length" value="0.04"/>
@@ -29,4 +32,16 @@
         <xacro:box_inertia   width="${base_width}" height="${base_height}" depth="${base_length}" mass="${base_mass}"/>
     </link>
+    <link name="base_footprint">
+        <visual>
+            <xacro:box_geometry width="${base_footprint_width}" height="${base_footprint_height}" depth="${base_footprint_length}"/>
+            <xacro:green_material/>
+        </visual>
+        <xacro:box_collision width="${base_footprint_width}" height="${base_footprint_height}" depth="${base_footprint_length}"/>
+    </link>
+    <joint name="base_footprint_joint" type="fixed">
+        <origin rpy="0 0 0" xyz="0 0 ${mecanum_radius - motor_holder_radius*3 }"/>
+        <parent link="base_footprint"/>
+        <child link="base_link"/>
+    </joint>
     <link name="neck_link">
         <visual>

Commit message: Added planar move plugin for robot control in simulation.

File: leobot_description/robot/leobot.gazebo.xacro (robot description, xacro)
@@ -29,29 +29,21 @@
     </gazebo>
     <gazebo reference="FL_wheel_link">
-        <mu1 value="1.0"/>
-        <mu2 value="1.0"/>
-        <kp value="10000000.0"/>
-        <kd value="1.0"/>
+        <mu1>0.0</mu1>
+        <mu2>0.0</mu2>
         <material>Gazebo/Blue</material>
     </gazebo>
     <gazebo reference="FR_wheel_link">
-        <mu1 value="1.0"/>
-        <mu2 value="1.0"/>
-        <kp value="10000000.0"/>
-        <kd value="1.0"/>
+        <mu1>0.0</mu1>
+        <mu2>0.0</mu2>
         <material>Gazebo/Blue</material>
     </gazebo>
     <gazebo reference="RL_wheel_link">
-        <mu1 value="1.0"/>
-        <mu2 value="1.0"/>
-        <kp value="10000000.0"/>
-        <kd value="1.0"/>
+        <mu1>0.0</mu1>
+        <mu2>0.0</mu2>
         <material>Gazebo/Blue</material>
     </gazebo>
     <gazebo reference="RR_wheel_link">
-        <mu1 value="1.0"/>
-        <mu2 value="1.0"/>
-        <kp value="10000000.0"/>
-        <kd value="1.0"/>
+        <mu1>0.0</mu1>
+        <mu2>0.0</mu2>
         <material>Gazebo/Blue</material>
     </gazebo>
@@ -176,3 +168,12 @@
         </sensor>
     </gazebo>
+    <gazebo>
+        <plugin name="object_controller" filename="libgazebo_ros_planar_move.so">
+            <commandTopic>/wheel_diff_drive_controller/cmd_vel</commandTopic>
+            <odometryTopic>odom</odometryTopic>
+            <odometryFrame>odom</odometryFrame>
+            <odometryRate>10.0</odometryRate>
+            <robotBaseFrame>base_footprint</robotBaseFrame>
+        </plugin>
+    </gazebo>
 </robot>

File: leobot_description/robot/robot.urdf.xacro (robot description, xacro)
@@ -21,4 +21,10 @@
     <xacro:property name="camera_stick_height" value="0.02"/>
     <xacro:property name="camera_stick_mass"   value="0.2"/>
+    <link name="base_footprint"/>
+    <joint name="base_footprint_joint" type="fixed">
+        <origin rpy="0 0 0" xyz="0 0 ${base_height / 2 + mecanum_radius - motor_holder_radius - 0.01 }"/>
+        <parent link="base_footprint"/>
+        <child link="base_link"/>
+    </joint>
     <link name="base_link">
         <visual>
@@ -85,7 +91,7 @@
     </transmission>
     <xacro:simple_camera prefix="left"  parent_link_name="camera_stick_link" parent_height="${camera_stick_height}"
-                  parent_length="${camera_stick_length}" side="1"/>
+                         parent_length="${camera_stick_length}" side="1"/>
     <xacro:simple_camera prefix="right" parent_link_name="camera_stick_link" parent_height="${camera_stick_height}"
-                  parent_length="${camera_stick_length}" side="-1"/>
+                         parent_length="${camera_stick_length}" side="-1"/>
     <xacro:lidar_hokuyo parent_link_name="base_link" parent_height="${base_height}"/>
     <xacro:mecanum_wheel prefix="FL" wheel_type="2" side="1" position="1" parent_length="${base_length}"
