Commit message: Refactored docs structure. Added Gazebo plugin for force based move. Need to adjust friction and mecanum wheel direction.

File: leobot_description/robot/leobot.gazebo.xacro (robot description, xacro)
@@ -7,24 +7,27 @@
         </plugin>
     </gazebo>
+    <gazebo reference="base_footprint">
+        <gravity>true</gravity>
+        <mu1>0.0</mu1>
+        <mu2>0.0</mu2>
+        <kp>1000000.0</kp>
+        <kd>100.0</kd>
+        <minDepth>0.001</minDepth>
+        <maxVel>1.0</maxVel>
+    </gazebo>
     <gazebo reference="base_link">
-        <mu1 value="1.0"/>
-        <mu2 value="1.0"/>
-        <kp value="10000000.0"/>
-        <kd value="1.0"/>
         <material>Gazebo/White</material>
     </gazebo>
     <gazebo reference="head_link">
-        <mu1 value="1.0"/>
-        <mu2 value="1.0"/>
-        <kp value="10000000.0"/>
-        <kd value="1.0"/>
         <material>Gazebo/White</material>
     </gazebo>
     <gazebo reference="neck_link">
-        <mu1 value="1.0"/>
-        <mu2 value="1.0"/>
-        <kp value="10000000.0"/>
-        <kd value="1.0"/>
         <material>Gazebo/White</material>
+    </gazebo>
+    <gazebo reference="camera_stick_link">
+        <material>Gazebo/Yellow</material>
+    </gazebo>
+    <gazebo reference="imu_link">
+        <material>Gazebo/Green</material>
     </gazebo>
     <gazebo reference="FL_wheel_link">
@@ -169,11 +172,53 @@
     </gazebo>
     <gazebo>
-        <plugin name="object_controller" filename="libgazebo_ros_planar_move.so">
-            <commandTopic>/wheel_diff_drive_controller/cmd_vel</commandTopic>
+        <plugin name="imu_controller" filename="libhector_gazebo_ros_imu.so">
+            <robotNamespace>/</robotNamespace>
+            <updateRate>50.0</updateRate>
+            <bodyName>base_footprint</bodyName>
+            <frameId>imu_link</frameId>
+            <topicName>imu/data</topicName>
+            <accelDrift>0.005 0.005 0.005</accelDrift>
+            <accelGaussianNoise>0.005 0.005 0.005</accelGaussianNoise>
+            <rateDrift>0.00005 0.00005 0.00005</rateDrift>
+            <rateGaussianNoise>0.00005 0.00005 0.00005</rateGaussianNoise>
+            <headingDrift>0.005</headingDrift>
+            <headingGaussianNoise>0.005</headingGaussianNoise>
+        </plugin>
+    </gazebo>
+    <gazebo>
+        <plugin name="gazebo_ros_force_based_move" filename="libgazebo_ros_force_based_move.so">
+            <robotNamespace>/</robotNamespace>
+            <commandTopic>/mecanum_velocity_controller/cmd_vel</commandTopic>
             <odometryTopic>odom</odometryTopic>
             <odometryFrame>odom</odometryFrame>
-            <odometryRate>10.0</odometryRate>
+            <odometryRate>25.0</odometryRate>
             <robotBaseFrame>base_footprint</robotBaseFrame>
+            <cmdVelTimeOut>0.25</cmdVelTimeOut>
+            <!-- Don't publish a transform: the controller does it. -->
+            <publishOdometryTf>0</publishOdometryTf>
+            <yaw_velocity_p_gain>1.0</yaw_velocity_p_gain>
+            <x_velocity_p_gain>1.0</x_velocity_p_gain>
+            <y_velocity_p_gain>1.0</y_velocity_p_gain>
         </plugin>
     </gazebo>
+    <!--<gazebo>-->
+         <!--<plugin name="ridgeback_ros_force_based_move" filename="libridgeback_ros_force_based_move.so">-->
+            <!--<robotNamespace>/</robotNamespace>-->
+            <!--<commandTopic>/mecanum_velocity_controller/cmd_vel</commandTopic>-->
+            <!--<odometryTopic>odom</odometryTopic>-->
+            <!--<odometryFrame>odom</odometryFrame>-->
+            <!--<odometryRate>25.0</odometryRate>-->
+            <!--<robotBaseFrame>base_link</robotBaseFrame>-->
+            <!--&lt;!&ndash;<robotBaseFrame>base_footprint</robotBaseFrame>&ndash;&gt;-->
+            <!--<cmdVelTimeOut>0.25</cmdVelTimeOut>-->
+            <!--&lt;!&ndash; Don't publish a transform: the controller does it. &ndash;&gt;-->
+            <!--<publishOdometryTf>0</publishOdometryTf>-->
+            <!--&lt;!&ndash;<yaw_velocity_p_gain>1.0</yaw_velocity_p_gain>&ndash;&gt;-->
+            <!--&lt;!&ndash;<x_velocity_p_gain>1.0</x_velocity_p_gain>&ndash;&gt;-->
+            <!--&lt;!&ndash;<y_velocity_p_gain>1.0</y_velocity_p_gain>&ndash;&gt;-->
+            <!--<yaw_velocity_p_gain>500.0</yaw_velocity_p_gain>-->
+            <!--<x_velocity_p_gain>10000.0</x_velocity_p_gain>-->
+            <!--<y_velocity_p_gain>10000.0</y_velocity_p_gain>-->
+        <!--</plugin>-->
+    <!--</gazebo>-->
 </robot>

File: leobot_description/robot/robot.urdf.xacro (robot description, xacro)
@@ -9,4 +9,6 @@
     <xacro:property name="base_height" value="0.3"/>
     <xacro:property name="base_mass"   value="10"/>
+    <xacro:property name="imu_link_size" value="0.01"/>
+    <xacro:property name="imu_link_mass" value="0.01"/>
     <xacro:property name="neck_width"  value="0.04"/>
     <xacro:property name="neck_length" value="0.04"/>
@@ -23,5 +25,5 @@
     <link name="base_footprint"/>
     <joint name="base_footprint_joint" type="fixed">
-        <origin rpy="0 0 0" xyz="0 0 ${base_height / 2 + mecanum_radius - motor_holder_radius - 0.01 }"/>
+        <origin rpy="0 0 0" xyz="0 0 ${base_height / 2 + mecanum_radius - motor_holder_radius - 0.05 }"/>
         <parent link="base_footprint"/>
         <child link="base_link"/>
@@ -30,5 +32,5 @@
         <visual>
             <xacro:box_geometry width="${base_width}" length="${base_length}" height="${base_height}"/>
-            <xacro:green_material/>
+            <xacro:navajo_white_material/>
         </visual>
         <xacro:box_collision width="${base_width}" length="${base_length}" height="${base_height}"/>
@@ -86,8 +88,20 @@
         </joint>
         <actuator name="head_camera_stick_joint">
-            <hardwareInterface>EffortJointInterface</hardwareInterface>
             <mechanicalReduction>1</mechanicalReduction>
         </actuator>
     </transmission>
+    <link name="imu_link">
+        <visual>
+            <xacro:cube_geometry size="${imu_link_size}"/>
+            <xacro:green_material/>
+        </visual>
+        <xacro:cube_collision size="${imu_link_size}"/>
+        <xacro:cube_inertia size="${imu_link_size}" mass="${imu_link_mass}"/>
+    </link>
+    <joint name="base_imu_link_joint" type="fixed">
+        <origin rpy="0 0 0" xyz="${(base_width - imu_link_size) / 2} 0 ${(base_height + imu_link_size) / 2}"/>
+        <parent link="base_link"/>
+        <child link="imu_link"/>
+    </joint>
     <xacro:simple_camera prefix="left"  parent_link_name="camera_stick_link" parent_height="${camera_stick_height}"
                          parent_length="${camera_stick_length}" side="1"/>

File: leobot_description/urdf/common.urdf.xacro (robot description, xacro)
@@ -84,3 +84,13 @@
         </collision>
     </xacro:macro>
+    <xacro:macro name="cube_geometry" params="size">
+        <xacro:box_geometry width="${size}" length="${size}" height="${size}"/>
+    </xacro:macro>
+    <xacro:macro name="cube_collision" params="size">
+        <xacro:box_collision width="${size}" length="${size}" height="${size}"/>
+    </xacro:macro>
+    <xacro:macro name="cube_inertia" params="mass size x:=0 y:=0 z:=0 roll:=0 pitch:=0 yaw:=0">
+        <xacro:box_inertia mass="${mass}" width="${size}" length="${size}" height="${size}" x="${x}" y="${y}" z="${z}"
+                           roll="${roll}" pitch="${pitch}" yaw="${yaw}"/>
+    </xacro:macro>
 </robot>

File: leobot_description/urdf/sensors/camera.urdf.xacro (robot description, xacro)
@@ -22,10 +22,9 @@
         <link name="${prefix}_camera_link">
             <visual>
-              <xacro:box_geometry width="${camera_size}" length="${camera_size}" height="${camera_size}"/>
+              <xacro:cube_geometry size="${camera_size}"/>
               <xacro:green_material/>
             </visual>
-            <xacro:box_collision width="${camera_size}" length="${camera_size}" height="${camera_size}"/>
-            <xacro:box_inertia mass="${camera_mass}" width="${camera_size}" length="${camera_size}"
-                               height="${camera_size}"/>
+            <xacro:cube_collision size="${camera_size}"/>
+            <xacro:cube_inertia mass="${camera_mass}" size="${camera_size}"/>
         </link>
         <joint name="${prefix}_camera_joint" type="fixed">

File: leobot_description/urdf/sensors/hokuyo.urdf.xacro (robot description, xacro)
@@ -7,5 +7,5 @@
             <visual>
                 <xacro:cylinder_geometry height="${hokuyo_height}" radius="${hokuyo_radius}"/>
-                <xacro:navajo_white_material/>
+                <xacro:green_material/>
             </visual>
             <xacro:cylinder_collision height="${hokuyo_height}" radius="${hokuyo_radius}"/>

File: leobot_description/urdf/wheels.urdf.xacro (robot description, xacro)
@@ -44,7 +44,5 @@
             </joint>
             <actuator name="${prefix}_wheel_motor">
-                <hardwareInterface>hardware_interface/VelocityJointInterface</hardwareInterface>
-                <mechanicalReduction>131</mechanicalReduction>
-                <motorTorqueConstant>4.4</motorTorqueConstant>
+                <mechanicalReduction>1</mechanicalReduction>
             </actuator>
         </transmission>

Commit message: Working simulation with stop on no commands

File: leobot_description/robot/leobot.gazebo.xacro (robot description, xacro)
@@ -9,10 +9,4 @@
     <gazebo reference="base_footprint">
         <gravity>true</gravity>
-        <mu1>0.0</mu1>
-        <mu2>0.0</mu2>
-        <kp>1000000.0</kp>
-        <kd>100.0</kd>
-        <minDepth>0.001</minDepth>
-        <maxVel>1.0</maxVel>
     </gazebo>
     <gazebo reference="base_link">
@@ -187,5 +181,5 @@
     </gazebo>
     <gazebo>
-        <plugin name="gazebo_ros_force_based_move" filename="libgazebo_ros_force_based_move.so">
+         <plugin name="ridgeback_ros_force_based_move" filename="libridgeback_ros_force_based_move.so">
             <robotNamespace>/</robotNamespace>
             <commandTopic>/mecanum_velocity_controller/cmd_vel</commandTopic>
@@ -197,28 +191,8 @@
             <!-- Don't publish a transform: the controller does it. -->
             <publishOdometryTf>0</publishOdometryTf>
-            <yaw_velocity_p_gain>1.0</yaw_velocity_p_gain>
-            <x_velocity_p_gain>1.0</x_velocity_p_gain>
-            <y_velocity_p_gain>1.0</y_velocity_p_gain>
+            <yaw_velocity_p_gain>100.0</yaw_velocity_p_gain>
+            <x_velocity_p_gain>100.0</x_velocity_p_gain>
+            <y_velocity_p_gain>100.0</y_velocity_p_gain>
         </plugin>
     </gazebo>
-    <!--<gazebo>-->
-         <!--<plugin name="ridgeback_ros_force_based_move" filename="libridgeback_ros_force_based_move.so">-->
-            <!--<robotNamespace>/</robotNamespace>-->
-            <!--<commandTopic>/mecanum_velocity_controller/cmd_vel</commandTopic>-->
-            <!--<odometryTopic>odom</odometryTopic>-->
-            <!--<odometryFrame>odom</odometryFrame>-->
-            <!--<odometryRate>25.0</odometryRate>-->
-            <!--<robotBaseFrame>base_link</robotBaseFrame>-->
-            <!--&lt;!&ndash;<robotBaseFrame>base_footprint</robotBaseFrame>&ndash;&gt;-->
-            <!--<cmdVelTimeOut>0.25</cmdVelTimeOut>-->
-            <!--&lt;!&ndash; Don't publish a transform: the controller does it. &ndash;&gt;-->
-            <!--<publishOdometryTf>0</publishOdometryTf>-->
-            <!--&lt;!&ndash;<yaw_velocity_p_gain>1.0</yaw_velocity_p_gain>&ndash;&gt;-->
-            <!--&lt;!&ndash;<x_velocity_p_gain>1.0</x_velocity_p_gain>&ndash;&gt;-->
-            <!--&lt;!&ndash;<y_velocity_p_gain>1.0</y_velocity_p_gain>&ndash;&gt;-->
-            <!--<yaw_velocity_p_gain>500.0</yaw_velocity_p_gain>-->
-            <!--<x_velocity_p_gain>10000.0</x_velocity_p_gain>-->
-            <!--<y_velocity_p_gain>10000.0</y_velocity_p_gain>-->
-        <!--</plugin>-->
-    <!--</gazebo>-->
 </robot>

File: leobot_description/robot/robot.urdf.xacro (robot description, xacro)
@@ -25,5 +25,5 @@
     <link name="base_footprint"/>
     <joint name="base_footprint_joint" type="fixed">
-        <origin rpy="0 0 0" xyz="0 0 ${base_height / 2 + mecanum_radius - motor_holder_radius - 0.05 }"/>
+        <origin rpy="0 0 0" xyz="0 0 ${base_height / 2 + mecanum_radius - motor_holder_radius}"/>
         <parent link="base_footprint"/>
         <child link="base_link"/>

File: leobot_description/urdf/wheels.urdf.xacro (robot description, xacro)
@@ -18,5 +18,5 @@
         <joint name="${prefix}_motor_holder_base_joint" type="fixed">
             <origin rpy="${pi/2} 0 0"
-                    xyz="${position * (parent_width/2 - motor_holder_radius*2)} ${side * (parent_length/2 + motor_holder_height/2)} ${(-parent_height/2 + motor_holder_radius*2)}"/>
+                    xyz="${position * (parent_width/2 - motor_holder_radius*2)} ${side * (parent_length/2 + motor_holder_height/2)} ${-parent_height/2 + motor_holder_radius}"/>
             <parent link="base_link"/>
             <child link="${prefix}_motor_holder"/>
